File: hw/rev1/audio_iface_rev1.kicad_pcb (KiCad board)
At the start: 2 copper layers, 122 parts, among them J101 CONN_2, J102 CONN_2, J103 CONN_2, J104 CONN_2, J105 CONN_2, J501 CONN_6, J601 CONN_2, Q201 BC550, Q202 BC550, U101 USBMICROCONN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

Commit message: More routing
Parts:
- C209, C214, C215, C219, C608, R101: moved to B.Cu
- moved SB301 90.4 mm to (189.2, 115.2), turned to 270 degrees
- moved R101 83.0 mm to (161.6, 86.3), turned to 270 degrees
- moved C209 70.5 mm to (174.2, 96.1)
- moved C608 56.9 mm to (161.9, 93.0)
- moved C219 16.3 mm to (158.9, 88.1), turned to 180 degrees
- moved C215 11.6 mm to (167.0, 97.2), turned to 180 degrees
- moved C218 5.72 mm to (171.6, 98.9)
- moved J105 5.36 mm to (187.4, 86.0)
- moved J104 5.36 mm to (183.9, 85.9)
- moved C221 1.77 mm to (173.8, 91.3), turned to 270 degrees
- moved C206 1.64 mm to (156.6, 99.0)
- moved J101 1.34 mm to (159.7, 86.2)
- moved C214 0.72 mm to (165.6, 97.1), turned to 270 degrees
- moved R213 0.69 mm to (167.6, 96.4)
- moved R206 0.68 mm to (160.4, 98.3), turned to 90 degrees
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Routing:
- net AGND_IN: track 14.4 -> 75.7 mm, vias 6 -> 25
- net +5VA: track 10.2 -> 41.2 mm, vias 1 -> 5
- net VCOM_VRT: track 8.67 -> 20.9 mm, vias 0 -> 1
- net N-0000052: track 0.00 -> 8.47 mm, vias 0 -> 2
- net N-0000035: track 2.83 -> 9.32 mm, vias 0 -> 2
- net N-0000049: track 12.9 -> 17.9 mm
- net N-0000040: track 0.00 -> 2.93 mm
- net N-0000048: track 0.00 -> 2.46 mm
- net N-0000050: track 0.00 -> 2.28 mm
- net /Audio In/EXT_IN: track 0.00 -> 2.12 mm
- net N-0000033: track 1.25 -> 3.28 mm, vias 0 -> 1
- net N-0000051: track 0.00 -> 1.96 mm
- net /CODEC/AINR+: track 0.00 -> 1.95 mm
- net N-0000031: track 0.00 -> 1.71 mm
- net N-0000032: track 1.23 -> 2.83 mm, vias 0 -> 1
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- added copper zone on B.Cu, net AGND_IN
