File: hw/rev2/micro.sch (KiCad schematic (older format))
At the start: 21 parts, among them J501 CONN_6, U501 K20X7_QFP64, X501 XTAL

Commit message: Lots of things: --Added RGB LED on timer outputs --Input: Moved capacitively coupled feedback nodes from vgnd to gnd --Output: LTC6242 for filtering to amplifier --Power: 2-stage supply for analog: USB 5V boost to 6V, LDO to 5V   Digital still using LDO from USB 5V and not caring about anyone   Bonus! Can completely shut off analog portion of board --Layout and routing: All of it TODO: final checks on layout and LVS (vs simulation) HEAD2HEAD2HEAD! TODO: adjust silkscreen, add logo TODO: debate adding 12.288MHz dedicated crystal
Parts:
- removed D501, D?: LED, ~, symbol LED
- added D1: LTST-C19FD1WT, ~, symbol LED3
- added R30: RES, ~, symbol RES
- gave numbers to parts that had none: 3
- renumbered C501 to C29, C502 to C30, C503 to C31, C504 to C32, C507 to C33, C509 to C34, C510 to C35, C511 to C36, J501 to J8, R501 to R20, R504 to R23, TP503 to TP4, TP501 to TP5, TP502 to TP6, U501 to U4, X501 to X1
Connections:
- net labels added: ANALOG_EN
- wire segments 111 -> 86

Commit message: Added extra oscillator JIC. Moved labels and made it pretty. Also fixed a missing capacitron
Parts:
- added C71: 10n, ~, symbol CAP
- added X2: ASFLM2-12.288MHZ, symbol OSC_W_EN
Connections:
- wire segments 86 -> 99
Changed lines of the file:
@@
 Sheet 4 6
 Title "Android DPOAE Interface"
-Date "3 may 2014"
+Date "6 may 2014"
 Rev "2a"
 Comp "Sana AudioPulse"
@@
 HP_~SD
 $Comp
-L +3V #PWR028
+L +3V #PWR35
 U 1 1 524A6D6E
 P 4050 4200
-F 0 "#PWR028" H 4050 4160 30  0001 C CNN
+F 0 "#PWR35" H 4050 4160 30  0001 C CNN
 F 1 "+3V" H 4050 4310 30  0000 C CNN
 F 2 "" H 4050 4200 60  0000 C CNN
@@
 $EndComp
 $Comp
-L DGND #PWR029
+L DGND #PWR32
 U 1 1 524A769B
 P 2900 4950
-F 0 "#PWR029" H 2900 4950 40  0001 C CNN
+F 0 "#PWR32" H 2900 4950 40  0001 C CNN
 F 1 "DGND" H 2900 4880 40  0000 C CNN
 F 2 "" H 2900 4950 60  0000 C CNN
@@
 $EndComp
 $Comp
-L DGND #PWR030
+L DGND #PWR33
 U 1 1 524D9525
 P 3750 6650
-F 0 "#PWR030" H 3750 6650 40  0001 C CNN
+F 0 "#PWR33" H 3750 6650 40  0001 C CNN
 F 1 "DGND" H 3750 6580 40  0000 C CNN
 F 2 "" H 3750 6650 60  0000 C CNN
@@
 $EndComp
 $Comp
-L +3V #PWR031
+L +3V #PWR36
 U 1 1 5251A974
 P 4900 1350
-F 0 "#PWR031" H 4900 1310 30  0001 C CNN
+F 0 "#PWR36" H 4900 1310 30  0001 C CNN
 F 1 "+3V" H 4900 1460 30  0000 C CNN
 F 2 "" H 4900 1350 60  0000 C CNN
@@
 $EndComp
 $Comp
-L DGND #PWR032
+L DGND #PWR37
 U 1 1 5251A9DC
 P 4900 1650
-F 0 "#PWR032" H 4900 1650 40  0001 C CNN
+F 0 "#PWR37" H 4900 1650 40  0001 C CNN
 F 1 "DGND" H 4900 1580 40  0000 C CNN
 F 2 "" H 4900 1650 60  0000 C CNN
@@
 $EndComp
 $Comp
-L DGND #PWR033
+L DGND #PWR41
 U 1 1 5251B8ED
 P 8300 6650
-F 0 "#PWR033" H 8300 6650 40  0001 C CNN
+F 0 "#PWR41" H 8300 6650 40  0001 C CNN
 F 1 "DGND" H 8300 6580 40  0000 C CNN
 F 2 "" H 8300 6650 60  0000 C CNN
@@
 PGA0_D-
 $Comp
-L USB_5V #PWR034
+L USB_5V #PWR34
 U 1 1 535048A3
 P 3850 3600
-F 0 "#PWR034" H 3850 3560 30  0001 C CNN
+F 0 "#PWR34" H 3850 3560 30  0001 C CNN
 F 1 "USB_5V" H 3850 3710 30  0000 C CNN
 F 2 "~" H 3850 3600 60  0000 C CNN
@@
 $EndComp
 $Comp
-L DGND #PWR035
+L DGND #PWR42
 U 1 1 5352B535
 P 8500 6650
-F 0 "#PWR035" H 8500 6650 40  0001 C CNN
+F 0 "#PWR42" H 8500 6650 40  0001 C CNN
 F 1 "DGND" H 8500 6580 40  0000 C CNN
 F 2 "" H 8500 6650 60  0000 C CNN
@@
 	7250 4100 5950 4100
 Wire Wire Line
-	7250 4200 5950 4200
+	5950 4200 7250 4200
 Wire Wire Line
 	6400 5600 5950 5600
@@
 Connection ~ 6700 2700
 $Comp
-L +3V #PWR036
+L +3V #PWR39
 U 1 1 53570C75
 P 6700 2000
-F 0 "#PWR036" H 6700 1960 30  0001 C CNN
+F 0 "#PWR39" H 6700 1960 30  0001 C CNN
 F 1 "+3V" H 6700 2110 30  0000 C CNN
 F 2 "" H 6700 2000 60  0000 C CNN
@@
 $EndComp
 $Comp
-L DGND #PWR037
+L DGND #PWR43
 U 1 1 5363BE47
 P 8700 6650
-F 0 "#PWR037" H 8700 6650 40  0001 C CNN
+F 0 "#PWR43" H 8700 6650 40  0001 C CNN
 F 1 "DGND" H 8700 6580 40  0000 C CNN
 F 2 "" H 8700 6650 60  0000 C CNN
@@
 Wire Wire Line
 	8500 5500 5950 5500
+$Comp
+L OSC_W_EN X2
+U 1 1 53695566
+P 6750 4550
+F 0 "X2" H 6900 4400 60  0000 C CNN
+F 1 "ASFLM2-12.288MHZ" H 6750 4700 60  0000 C CNN
+F 2 "" H 6750 4550 60  0000 C CNN
+F 3 "" H 6750 4550 60  0000 C CNN
+	1    6750 4550
+	1    0    0    -1
+$EndComp
+Wire Wire Line
+	7050 4600 7200 4600
+Wire Wire Line
+	7200 4600 7200 4200
+Connection ~ 7200 4200
+$Comp
+L +3V #PWR40
+U 1 1 536955E4
+P 7300 4350
+F 0 "#PWR40" H 7300 4310 30  0001 C CNN
+F 1 "+3V" H 7300 4460 30  0000 C CNN
+F 2 "" H 7300 4350 60  0000 C CNN
+F 3 "" H 7300 4350 60  0000 C CNN
+	1    7300 4350
+	1    0    0    -1
+$EndComp
+Wire Wire Line
+	7300 4350 7300 4500
+Wire Wire Line
+	7300 4500 7050 4500
+$Comp
+L DGND #PWR38
+U 1 1 5369565E
+P 6350 4850
+F 0 "#PWR38" H 6350 4850 40  0001 C CNN
+F 1 "DGND" H 6350 4780 40  0000 C CNN
+F 2 "" H 6350 4850 60  0000 C CNN
+F 3 "" H 6350 4850 60  0000 C CNN
+	1    6350 4850
+	1    0    0    -1
+$EndComp
+Wire Wire Line
+	6350 4600 6350 4850
+Wire Wire Line
+	6350 4600 6450 4600
+Wire Wire Line
+	5950 3200 6250 3200
+Wire Wire Line
+	6250 3200 6250 4500
+Wire Wire Line
+	6250 4500 6450 4500
+$Comp
+L CAP C71
+U 1 1 53697AF9
+P 7400 4550
+F 0 "C71" H 7420 4520 50  0000 L TNN
+F 1 "10n" H 7425 4570 30  0000 L BNN
+F 2 "~" H 7400 4550 60  0000 C CNN
+F 3 "~" H 7400 4550 60  0000 C CNN
+	1    7400 4550
+	0    -1   -1   0
+$EndComp
+Wire Wire Line
+	6350 4750 7400 4750
+Wire Wire Line
+	7400 4750 7400 4650
+Connection ~ 6350 4750
+Wire Wire Line
+	7400 4450 7400 4400
+Wire Wire Line
+	7400 4400 7300 4400
+Connection ~ 7300 4400
 $EndSCHEMATC

Commit message: Rev 2a sent off for manufacturing: Slot added instead of drill hole at audio IO end Drill added near center Fixed huge error in HP amp schematic/layout Got rid of more labels Got rid of redundant UART port. Not sure how that happened twice... Got rid of DC blocking before CODEC inputs
Parts:
- removed TP5: TP_PTB3, ~, symbol TP
- removed TP6: TP_PTB16, ~, symbol TP
Connections:
- net labels removed: UART_RX, UART_TX
- wire segments 99 -> 97
Changed lines of the file:
@@
 Sheet 4 6
 Title "Android DPOAE Interface"
-Date "6 may 2014"
-Rev "2a"
+Date "29 jun 2014"
+Rev "2b"
 Comp "Sana AudioPulse"
 Comment1 "Ben Nahill <bnahill@gmail.com>"
@@
 $EndComp
 $Comp
-L TP TP6
-U 1 1 5251B77F
-P 8200 3000
-F 0 "TP6" H 8200 2900 60  0000 C CNN
-F 1 "TP_PTB16" H 8200 3100 60  0000 C CNN
-F 2 "~" H 8200 3000 60  0000 C CNN
-F 3 "~" H 8200 3000 60  0000 C CNN
-	1    8200 3000
-	1    0    0    -1
-$EndComp
-$Comp
 L RES R23
 U 1 1 5251B82C
@@
 F 3 "" H 8300 6650 60  0000 C CNN
 	1    8300 6650
-	1    0    0    -1
-$EndComp
-$Comp
-L TP TP5
-U 1 1 5251B955
-P 7800 3100
-F 0 "TP5" H 7800 3000 60  0000 C CNN
-F 1 "TP_PTB3" H 7800 3200 60  0000 C CNN
-F 2 "~" H 7800 3100 60  0000 C CNN
-F 3 "~" H 7800 3100 60  0000 C CNN
-	1    7800 3100
 	1    0    0    -1
 $EndComp
@@
 	6400 6000 5950 6000
 Wire Wire Line
-	8100 3000 5950 3000
-Wire Wire Line
-	5950 3100 7700 3100
-Wire Wire Line
 	3850 3700 3850 3600
 Connection ~ 3850 3700
@@
 Wire Wire Line
 	8500 6650 8500 6500
-Text Label 6900 3100 0    60   ~ 0
-UART_TX
-Text Label 6900 3000 0    60   ~ 0
-UART_RX
 Text HLabel 7250 2600 2    60   BiDi ~ 0
 I2C_SCL

Commit message: Added values for LED resistors
Parts:
- R23: value RES -> 220
- R24: value RES -> 7.5
- R30: value RES -> 39
Changed lines of the file:
@@
 LIBS:valves
 LIBS:audio_iface_rev2-cache
-EELAYER 27 0
+EELAYER 25 0
 EELAYER END
 $Descr A 11000 8500
@@
 P 8300 5850
 F 0 "R23" H 8370 5815 50  0000 L TNN
-F 1 "RES" H 8300 5905 30  0000 C BNN
+F 1 "220" H 8300 5905 30  0000 C BNN
 F 2 "~" H 8300 5850 60  0000 C CNN
 F 3 "~" H 8300 5850 60  0000 C CNN
@@
 P 8500 5850
 F 0 "R24" H 8570 5815 50  0000 L TNN
-F 1 "RES" H 8500 5905 30  0000 C BNN
+F 1 "7.5" H 8500 5905 30  0000 C BNN
 F 2 "~" H 8500 5850 60  0000 C CNN
 F 3 "~" H 8500 5850 60  0000 C CNN
@@
 P 8700 5850
 F 0 "R30" H 8770 5815 50  0000 L TNN
-F 1 "RES" H 8700 5905 30  0000 C BNN
+F 1 "39" H 8700 5905 30  0000 C BNN
 F 2 "~" H 8700 5850 60  0000 C CNN
 F 3 "~" H 8700 5850 60  0000 C CNN

Commit message: Added serial flash module to schematic and began layout
Connections:
- net labels added: SPI1_CS_FLASH, SPI1_SIN
- wire segments 97 -> 132
Changed lines of the file:
@@
 LIBS:valves
 LIBS:audio_iface_rev2-cache
-EELAYER 25 0
+EELAYER 27 0
 EELAYER END
 $Descr A 11000 8500
@@
 Sheet 4 6
 Title "Android DPOAE Interface"
-Date "29 jun 2014"
+Date "12 may 2015"
 Rev "2b"
 Comp "Sana AudioPulse"
@@
 $EndComp
 Wire Wire Line
-	3300 2600 3300 4550
-Wire Wire Line
-	2750 4800 4700 4800
+	3300 2600 3300 4400
+Wire Wire Line
+	3300 4400 3300 4550
+Wire Wire Line
+	2750 4800 2900 4800
+Wire Wire Line
+	2900 4800 3300 4800
+Wire Wire Line
+	3300 4800 3450 4800
+Wire Wire Line
+	3450 4800 3750 4800
+Wire Wire Line
+	3750 4800 4050 4800
+Wire Wire Line
+	4050 4800 4600 4800
+Wire Wire Line
+	4600 4800 4700 4800
 Connection ~ 4050 4800
 Wire Wire Line
@@
 Connection ~ 3450 4800
 Wire Wire Line
-	4150 6700 4450 6700
-Wire Wire Line
-	4150 6500 4700 6500
+	4150 6700 4300 6700
+Wire Wire Line
+	4300 6700 4450 6700
+Wire Wire Line
+	4150 6500 4300 6500
+Wire Wire Line
+	4300 6500 4700 6500
 Connection ~ 4300 6700
 Connection ~ 4300 6500
@@
 	3950 6500 3850 6500
 Wire Wire Line
-	3850 6500 3850 6700
+	3850 6500 3850 6600
+Wire Wire Line
+	3850 6600 3850 6700
 Wire Wire Line
 	3850 6700 3950 6700
@@
 	7250 4100 5950 4100
 Wire Wire Line
-	5950 4200 7250 4200
+	5950 4200 7200 4200
+Wire Wire Line
+	7200 4200 7250 4200
 Wire Wire Line
 	6400 5600 5950 5600
@@
 	4700 4700 4600 4700
 Wire Wire Line
-	4600 4700 4600 5200
+	4600 4700 4600 4800
+Wire Wire Line
+	4600 4800 4600 4900
+Wire Wire Line
+	4600 4900 4600 5000
+Wire Wire Line
+	4600 5000 4600 5100
+Wire Wire Line
+	4600 5100 4600 5200
 Wire Wire Line
 	4600 4900 4700 4900
@@
 	4700 4000 4600 4000
 Wire Wire Line
-	4600 3800 4600 4500
+	4600 3800 4600 4000
+Wire Wire Line
+	4600 4000 4600 4100
+Wire Wire Line
+	4600 4100 4600 4200
+Wire Wire Line
+	4600 4200 4600 4300
+Wire Wire Line
+	4600 4300 4600 4400
+Wire Wire Line
+	4600 4400 4600 4500
 Wire Wire Line
 	4600 4100 4700 4100
@@
 	4450 6600 4700 6600
 Wire Wire Line
-	4050 4200 4050 4550
+	4050 4200 4050 4400
+Wire Wire Line
+	4050 4400 4050 4550
 Wire Wire Line
 	4050 4800 4050 4750
 Wire Wire Line
-	2900 4050 2900 4950
+	2900 4050 2900 4800
+Wire Wire Line
+	2900 4800 2900 4950
 Connection ~ 2900 4800
 Connection ~ 3300 4800
@@
 Connection ~ 3850 3700
 Wire Wire Line
-	2750 3700 4700 3700
+	2750 3700 2900 3700
+Wire Wire Line
+	2900 3700 3850 3700
+Wire Wire Line
+	3850 3700 4700 3700
 Wire Wire Line
 	8500 6000 8500 6100
@@
 I2C_SDA
 Wire Wire Line
-	5950 2700 7250 2700
-Wire Wire Line
-	5950 2600 7250 2600
+	5950 2700 6700 2700
+Wire Wire Line
+	6700 2700 7250 2700
+Wire Wire Line
+	5950 2600 6850 2600
+Wire Wire Line
+	6850 2600 7250 2600
 $Comp
 L RES R21
@@
 $EndComp
 Wire Wire Line
-	6700 2000 6700 2150
+	6700 2000 6700 2050
+Wire Wire Line
+	6700 2050 6700 2150
 Wire Wire Line
 	6700 2050 6850 2050
@@
 Connection ~ 6700 2050
 Wire Wire Line
-	3300 4400 4700 4400
+	3300 4400 3450 4400
+Wire Wire Line
+	3450 4400 3750 4400
+Wire Wire Line
+	3750 4400 4050 4400
+Wire Wire Line
+	4050 4400 4600 4400
+Wire Wire Line
+	4600 4400 4700 4400
 Text HLabel 6250 5300 2    60   Output ~ 0
 ANALOG_EN
@@
 $EndComp
 Wire Wire Line
-	7300 4350 7300 4500
+	7300 4350 7300 4400
+Wire Wire Line
+	7300 4400 7300 4500
 Wire Wire Line
 	7300 4500 7050 4500
@@
 $EndComp
 Wire Wire Line
-	6350 4600 6350 4850
+	6350 4600 6350 4750
+Wire Wire Line
+	6350 4750 6350 4850
 Wire Wire Line
 	6350 4600 6450 4600
 Wire Wire Line
-	5950 3200 6250 3200
-Wire Wire Line
-	6250 3200 6250 4500
-Wire Wire Line
-	6250 4500 6450 4500
+	5950 3200 6150 3200
+Wire Wire Line
+	6150 3200 6150 4500
+Wire Wire Line
+	6150 4500 6450 4500
 $Comp
 L CAP C71
@@
 	7400 4400 7300 4400
 Connection ~ 7300 4400
+Text HLabel 6250 4300 2    60   Input ~ 0
+SPI1_SIN
+Wire Wire Line
+	6250 4300 5950 4300
+Text HLabel 6250 3600 2    60   Output ~ 0
+SPI1_CS_FLASH
+Wire Wire Line
+	6250 3600 5950 3600
 $EndSCHEMATC

Commit message: Added SMA connectors, still need to recreate keepouts
Connections:
- wire segments 132 -> 99
Changed lines of the file:
@@
 Sheet 4 6
 Title "Android DPOAE Interface"
-Date "12 may 2015"
+Date "13 may 2015"
 Rev "2b"
 Comp "Sana AudioPulse"
@@
 HP_~SD
 $Comp
-L +3V #PWR35
+L +3V #PWR38
 U 1 1 524A6D6E
 P 4050 4200
-F 0 "#PWR35" H 4050 4160 30  0001 C CNN
+F 0 "#PWR38" H 4050 4160 30  0001 C CNN
 F 1 "+3V" H 4050 4310 30  0000 C CNN
 F 2 "" H 4050 4200 60  0000 C CNN
@@
 $EndComp
 $Comp
-L DGND #PWR32
+L DGND #PWR35
 U 1 1 524A769B
 P 2900 4950
-F 0 "#PWR32" H 2900 4950 40  0001 C CNN
+F 0 "#PWR35" H 2900 4950 40  0001 C CNN
 F 1 "DGND" H 2900 4880 40  0000 C CNN
 F 2 "" H 2900 4950 60  0000 C CNN
@@
 $EndComp
 $Comp
-L DGND #PWR33
+L DGND #PWR36
 U 1 1 524D9525
 P 3750 6650
-F 0 "#PWR33" H 3750 6650 40  0001 C CNN
+F 0 "#PWR36" H 3750 6650 40  0001 C CNN
 F 1 "DGND" H 3750 6580 40  0000 C CNN
 F 2 "" H 3750 6650 60  0000 C CNN
@@
 $EndComp
 $Comp
-L +3V #PWR36
+L +3V #PWR39
 U 1 1 5251A974
 P 4900 1350
-F 0 "#PWR36" H 4900 1310 30  0001 C CNN
+F 0 "#PWR39" H 4900 1310 30  0001 C CNN
 F 1 "+3V" H 4900 1460 30  0000 C CNN
 F 2 "" H 4900 1350 60  0000 C CNN
@@
 $EndComp
 $Comp
-L DGND #PWR37
+L DGND #PWR40
 U 1 1 5251A9DC
 P 4900 1650
-F 0 "#PWR37" H 4900 1650 40  0001 C CNN
+F 0 "#PWR40" H 4900 1650 40  0001 C CNN
 F 1 "DGND" H 4900 1580 40  0000 C CNN
 F 2 "" H 4900 1650 60  0000 C CNN
@@
 $EndComp
 $Comp
-L DGND #PWR41
+L DGND #PWR44
 U 1 1 5251B8ED
 P 8300 6650
-F 0 "#PWR41" H 8300 6650 40  0001 C CNN
+F 0 "#PWR44" H 8300 6650 40  0001 C CNN
 F 1 "DGND" H 8300 6580 40  0000 C CNN
 F 2 "" H 8300 6650 60  0000 C CNN
@@
 PGA0_D-
 $Comp
-L USB_5V #PWR34
+L USB_5V #PWR37
 U 1 1 535048A3
 P 3850 3600
-F 0 "#PWR34" H 3850 3560 30  0001 C CNN
+F 0 "#PWR37" H 3850 3560 30  0001 C CNN
 F 1 "USB_5V" H 3850 3710 30  0000 C CNN
 F 2 "~" H 3850 3600 60  0000 C CNN
@@
 $EndComp
 $Comp
-L DGND #PWR42
+L DGND #PWR45
 U 1 1 5352B535
 P 8500 6650
-F 0 "#PWR42" H 8500 6650 40  0001 C CNN
+F 0 "#PWR45" H 8500 6650 40  0001 C CNN
 F 1 "DGND" H 8500 6580 40  0000 C CNN
 F 2 "" H 8500 6650 60  0000 C CNN
@@
 $EndComp
 Wire Wire Line
-	3300 2600 3300 4400
-Wire Wire Line
-	3300 4400 3300 4550
-Wire Wire Line
-	2750 4800 2900 4800
-Wire Wire Line
-	2900 4800 3300 4800
-Wire Wire Line
-	3300 4800 3450 4800
-Wire Wire Line
-	3450 4800 3750 4800
-Wire Wire Line
-	3750 4800 4050 4800
-Wire Wire Line
-	4050 4800 4600 4800
-Wire Wire Line
-	4600 4800 4700 4800
+	3300 2600 3300 4550
+Wire Wire Line
+	2750 4800 4700 4800
 Connection ~ 4050 4800
 Wire Wire Line
@@
 Connection ~ 3450 4800
 Wire Wire Line
-	4150 6700 4300 6700
-Wire Wire Line
-	4300 6700 4450 6700
-Wire Wire Line
-	4150 6500 4300 6500
-Wire Wire Line
-	4300 6500 4700 6500
+	4150 6700 4450 6700
+Wire Wire Line
+	4150 6500 4700 6500
 Connection ~ 4300 6700
 Connection ~ 4300 6500
@@
 	3950 6500 3850 6500
 Wire Wire Line
-	3850 6500 3850 6600
-Wire Wire Line
-	3850 6600 3850 6700
+	3850 6500 3850 6700
 Wire Wire Line
 	3850 6700 3950 6700
@@
 	7250 4100 5950 4100
 Wire Wire Line
-	5950 4200 7200 4200
-Wire Wire Line
-	7200 4200 7250 4200
+	5950 4200 7250 4200
 Wire Wire Line
 	6400 5600 5950 5600
@@
 	4700 4700 4600 4700
 Wire Wire Line
-	4600 4700 4600 4800
-Wire Wire Line
-	4600 4800 4600 4900
-Wire Wire Line
-	4600 4900 4600 5000
-Wire Wire Line
-	4600 5000 4600 5100
-Wire Wire Line
-	4600 5100 4600 5200
+	4600 4700 4600 5200
 Wire Wire Line
 	4600 4900 4700 4900
@@
 	4700 4000 4600 4000
 Wire Wire Line
-	4600 3800 4600 4000
-Wire Wire Line
-	4600 4000 4600 4100
-Wire Wire Line
-	4600 4100 4600 4200
-Wire Wire Line
-	4600 4200 4600 4300
-Wire Wire Line
-	4600 4300 4600 4400
-Wire Wire Line
-	4600 4400 4600 4500
+	4600 3800 4600 4500
 Wire Wire Line
 	4600 4100 4700 4100
@@
 	4450 6600 4700 6600
 Wire Wire Line
-	4050 4200 4050 4400
-Wire Wire Line
-	4050 4400 4050 4550
+	4050 4200 4050 4550
 Wire Wire Line
 	4050 4800 4050 4750
 Wire Wire Line
-	2900 4050 2900 4800
-Wire Wire Line
-	2900 4800 2900 4950
+	2900 4050 2900 4950
 Connection ~ 2900 4800
 Connection ~ 3300 4800
@@
 Connection ~ 3850 3700
 Wire Wire Line
-	2750 3700 2900 3700
-Wire Wire Line
-	2900 3700 3850 3700
-Wire Wire Line
-	3850 3700 4700 3700
+	2750 3700 4700 3700
 Wire Wire Line
 	8500 6000 8500 6100
@@
 I2C_SDA
 Wire Wire Line
-	5950 2700 6700 2700
-Wire Wire Line
-	6700 2700 7250 2700
-Wire Wire Line
-	5950 2600 6850 2600
-Wire Wire Line
-	6850 2600 7250 2600
+	5950 2700 7250 2700
+Wire Wire Line
+	5950 2600 7250 2600
 $Comp
 L RES R21
@@
 Connection ~ 6700 2700
 $Comp
-L +3V #PWR39
+L +3V #PWR42
 U 1 1 53570C75
 P 6700 2000
-F 0 "#PWR39" H 6700 1960 30  0001 C CNN
+F 0 "#PWR42" H 6700 1960 30  0001 C CNN
 F 1 "+3V" H 6700 2110 30  0000 C CNN
 F 2 "" H 6700 2000 60  0000 C CNN
@@
 $EndComp
 Wire Wire Line
-	6700 2000 6700 2050
-Wire Wire Line
-	6700 2050 6700 2150
+	6700 2000 6700 2150
 Wire Wire Line
 	6700 2050 6850 2050
@@
 Connection ~ 6700 2050
 Wire Wire Line
-	3300 4400 3450 4400
-Wire Wire Line
-	3450 4400 3750 4400
-Wire Wire Line
-	3750 4400 4050 4400
-Wire Wire Line
-	4050 4400 4600 4400
-Wire Wire Line
-	4600 4400 4700 4400
+	3300 4400 4700 4400
 Text HLabel 6250 5300 2    60   Output ~ 0
 ANALOG_EN
@@
 $EndComp
 $Comp
-L DGND #PWR43
+L DGND #PWR46
 U 1 1 5363BE47
 P 8700 6650
-F 0 "#PWR43" H 8700 6650 40  0001 C CNN
+F 0 "#PWR46" H 8700 6650 40  0001 C CNN
 F 1 "DGND" H 8700 6580 40  0000 C CNN
 F 2 "" H 8700 6650 60  0000 C CNN
@@
 Connection ~ 7200 4200
 $Comp
-L +3V #PWR40
+L +3V #PWR43
 U 1 1 536955E4
 P 7300 4350
-F 0 "#PWR40" H 7300 4310 30  0001 C CNN
+F 0 "#PWR43" H 7300 4310 30  0001 C CNN
 F 1 "+3V" H 7300 4460 30  0000 C CNN
 F 2 "" H 7300 4350 60  0000 C CNN
@@
 $EndComp
 Wire Wire Line
-	7300 4350 7300 4400
-Wire Wire Line
-	7300 4400 7300 4500
+	7300 4350 7300 4500
 Wire Wire Line
 	7300 4500 7050 4500
 $Comp
-L DGND #PWR38
+L DGND #PWR41
 U 1 1 5369565E
 P 6350 4850
-F 0 "#PWR38" H 6350 4850 40  0001 C CNN
+F 0 "#PWR41" H 6350 4850 40  0001 C CNN
 F 1 "DGND" H 6350 4780 40  0000 C CNN
 F 2 "" H 6350 4850 60  0000 C CNN
@@
 $EndComp
 Wire Wire Line
-	6350 4600 6350 4750
-Wire Wire Line
-	6350 4750 6350 4850
+	6350 4600 6350 4850
 Wire Wire Line
 	6350 4600 6450 4600

Commit message: Started board upgrade to 4 layers and better signal isolation
Parts:
- removed J8: CONN_6, ~, symbol CONN_6
- added P3: CONN_01X06, lib:HDR_6X1_50MIL, symbol CONN_01X06
- C29, C31: footprint ~ -> lib:SMD0603
- C30, C32, C33, C34, C35, C36, C71, R20, R21, R22, R23, R24, R30: footprint ~ -> lib:SMD0402
- D1: footprint ~ -> lib:LED-6PLCC
- TP4: footprint ~ -> lib:TP_HOLE
- U4: footprint (none) -> lib:FREESCALE_QFP64
- X1: footprint ~ -> lib:TXC_7A
- X2: footprint (none) -> lib:ASFLM
Connections:
- net labels added: GNDD
- net labels removed: DGND
