File: hw/rev2/micro.sch (KiCad schematic (older format))
At the start: 25 parts, among them P3 CONN_01X06, U4 SAM_S70N_TFBGA, X1 XTAL, X2 ASFLM2-12.288MHZ

Commit message: Replaced 8MHz xtal with 16
Parts:
- X1: value XTAL -> 7A-16.000MAAJ-T
Changed lines of the file:
@@
 P 8000 4350
 F 0 "X1" H 8000 4290 40  0000 C TNN
-F 1 "XTAL" H 8000 4410 40  0000 C BNN
+F 1 "7A-16.000MAAJ-T" H 8000 4410 40  0000 C BNN
 F 2 "lib:TXC_7A" H 8000 4350 60  0001 C CNN
 F 3 "~" H 8000 4350 60  0000 C CNN

Commit message: Added 3V regulator, started wiring
Parts:
- added C73, C74, C77, C78, C79, C80, C81: 100n, lib:SMD0402, symbol CAP
- C34: value 10n -> 100n
Connections:
- net labels added: LED1, LED2, LED3
- wire segments 102 -> 122
Changed lines of the file:
@@
 L CAP C34
 U 1 1 524A6DA1
-P 5100 1250
-F 0 "C34" H 5120 1220 50  0000 L TNN
-F 1 "10n" H 5125 1270 30  0000 L BNN
-F 2 "lib:SMD0402" H 5100 1250 60  0001 C CNN
-F 3 "~" H 5100 1250 60  0000 C CNN
-	1    5100 1250
+P 5550 1250
+F 0 "C34" H 5570 1220 50  0000 L TNN
+F 1 "100n" H 5575 1270 30  0000 L BNN
+F 2 "lib:SMD0402" H 5550 1250 60  0001 C CNN
+F 3 "~" H 5550 1250 60  0000 C CNN
+	1    5550 1250
 	0    -1   -1   0
 $EndComp
@@
 	8150 4350 8400 4350
 Wire Wire Line
-	5100 1000 5100 1150
-Wire Wire Line
-	5100 1400 5100 1350
-Wire Wire Line
 	9500 5250 9050 5250
 Wire Wire Line
@@
 $EndComp
 Wire Wire Line
-	6150 1800 6150 2050
+	6150 1800 6150 2250
 Wire Wire Line
 	6150 1850 7100 1850
@@
 $EndComp
 Wire Wire Line
-	4650 1400 5100 1400
+	4650 1400 5550 1400
 Wire Wire Line
 	4850 1400 4850 1500
@@
 Connection ~ 4950 1400
 Wire Wire Line
-	4650 1000 5100 1000
+	4650 1000 5550 1000
 Wire Wire Line
 	4900 1000 4900 950
@@
 Text Label 9450 5700 2    60   ~ 0
 CLK_EN
+Wire Wire Line
+	2900 7350 2750 7350
+Text Label 3400 3300 2    60   ~ 0
+LED2
+Wire Wire Line
+	3400 3300 3500 3300
+Text Label 8500 5500 1    60   ~ 0
+LED2
+Wire Wire Line
+	8500 5500 8500 5700
+Text Label 8300 5500 1    60   ~ 0
+LED1
+Wire Wire Line
+	8300 5500 8300 5700
+Text Label 2750 7350 2    60   ~ 0
+LED1
+Wire Wire Line
+	2900 7050 2750 7050
+Text Label 2750 7050 2    60   ~ 0
+LED3
+Text Label 8700 5500 1    60   ~ 0
+LED3
+Wire Wire Line
+	8700 5500 8700 5700
+Wire Wire Line
+	5550 1400 5550 1350
+Wire Wire Line
+	5550 1000 5550 1150
+$Comp
+L CAP C73
+U 1 1 58241E42
+P 5100 1250
+F 0 "C73" H 5120 1220 50  0000 L TNN
+F 1 "100n" H 5125 1270 30  0000 L BNN
+F 2 "lib:SMD0402" H 5100 1250 60  0001 C CNN
+F 3 "~" H 5100 1250 60  0000 C CNN
+	1    5100 1250
+	0    -1   -1   0
+$EndComp
+Wire Wire Line
+	5100 1400 5100 1350
+Wire Wire Line
+	5100 1000 5100 1150
+$Comp
+L CAP C74
+U 1 1 58241E6F
+P 5250 1250
+F 0 "C74" H 5270 1220 50  0000 L TNN
+F 1 "100n" H 5275 1270 30  0000 L BNN
+F 2 "lib:SMD0402" H 5250 1250 60  0001 C CNN
+F 3 "~" H 5250 1250 60  0000 C CNN
+	1    5250 1250
+	0    -1   -1   0
+$EndComp
+Wire Wire Line
+	5250 1400 5250 1350
+Wire Wire Line
+	5250 1000 5250 1150
+Connection ~ 5100 1000
+Connection ~ 5250 1000
+Connection ~ 5250 1400
+Connection ~ 5100 1400
+$Comp
+L CAP C77
+U 1 1 582421FD
+P 5400 1250
+F 0 "C77" H 5420 1220 50  0000 L TNN
+F 1 "100n" H 5425 1270 30  0000 L BNN
+F 2 "lib:SMD0402" H 5400 1250 60  0001 C CNN
+F 3 "~" H 5400 1250 60  0000 C CNN
+	1    5400 1250
+	0    -1   -1   0
+$EndComp
+Wire Wire Line
+	5400 1400 5400 1350
+Wire Wire Line
+	5400 1000 5400 1150
+Connection ~ 5400 1000
+Connection ~ 5400 1400
+$Comp
+L CAP C81
+U 1 1 58242974
+P 6600 2350
+F 0 "C81" H 6620 2320 50  0000 L TNN
+F 1 "100n" H 6625 2370 30  0000 L BNN
+F 2 "lib:SMD0402" H 6600 2350 60  0001 C CNN
+F 3 "~" H 6600 2350 60  0000 C CNN
+	1    6600 2350
+	0    -1   -1   0
+$EndComp
+Wire Wire Line
+	6600 2050 6600 2250
+$Comp
+L CAP C78
+U 1 1 5824297B
+P 6150 2350
+F 0 "C78" H 6170 2320 50  0000 L TNN
+F 1 "100n" H 6175 2370 30  0000 L BNN
+F 2 "lib:SMD0402" H 6150 2350 60  0001 C CNN
+F 3 "~" H 6150 2350 60  0000 C CNN
+	1    6150 2350
+	0    -1   -1   0
+$EndComp
+$Comp
+L CAP C79
+U 1 1 58242982
+P 6300 2350
+F 0 "C79" H 6320 2320 50  0000 L TNN
+F 1 "100n" H 6325 2370 30  0000 L BNN
+F 2 "lib:SMD0402" H 6300 2350 60  0001 C CNN
+F 3 "~" H 6300 2350 60  0000 C CNN
+	1    6300 2350
+	0    -1   -1   0
+$EndComp
+Wire Wire Line
+	6300 2050 6300 2250
+$Comp
+L CAP C80
+U 1 1 58242989
+P 6450 2350
+F 0 "C80" H 6470 2320 50  0000 L TNN
+F 1 "100n" H 6475 2370 30  0000 L BNN
+F 2 "lib:SMD0402" H 6450 2350 60  0001 C CNN
+F 3 "~" H 6450 2350 60  0000 C CNN
+	1    6450 2350
+	0    -1   -1   0
+$EndComp
+Wire Wire Line
+	6450 2050 6450 2250
+Connection ~ 6600 2050
+Connection ~ 6450 2050
+Connection ~ 6300 2050
+$Comp
+L GNDD #PWR047
+U 1 1 58242A92
+P 6150 2550
+F 0 "#PWR047" H 6150 2300 50  0001 C CNN
+F 1 "GNDD" H 6150 2400 50  0000 C CNN
+F 2 "" H 6150 2550 50  0000 C CNN
+F 3 "" H 6150 2550 50  0000 C CNN
+	1    6150 2550
+	1    0    0    -1
+$EndComp
+Wire Wire Line
+	6150 2550 6150 2450
+Wire Wire Line
+	6150 2500 6600 2500
+Wire Wire Line
+	6300 2500 6300 2450
+Connection ~ 6150 2500
+Wire Wire Line
+	6450 2500 6450 2450
+Connection ~ 6300 2500
+Wire Wire Line
+	6600 2500 6600 2450
+Connection ~ 6450 2500
+Connection ~ 6150 2050
 $EndSCHEMATC

Commit message: Fully routed
Parts:
- removed TP4: TP_PTE0, lib:TP_HOLE, symbol TP
Connections:
- wire segments 122 -> 125
Other:
- note added: "PWMC0_H0"
- note added: "PWMC0_H1"
Changed lines of the file:
@@
 Comment4 ""
 $EndDescr
-Text HLabel 9050 4900 2    60   Output ~ 0
+Text HLabel 4100 5950 2    60   Output ~ 0
 HP_~SD
 $Comp
@@
 Text Label 8350 1450 0    60   ~ 0
 ~RESET
-Text HLabel 9050 5000 2    60   Output ~ 0
+Text HLabel 4600 4100 2    60   Output ~ 0
 CODEC_PDN
 Text Notes 2550 3000 0    40   ~ 0
@@
 	0    -1   -1   0
 $EndComp
-$Comp
-L TP TP4
-U 1 1 5251BBAF
-P 9600 5250
-F 0 "TP4" H 9600 5150 60  0000 C CNN
-F 1 "TP_PTE0" H 9600 5350 60  0000 C CNN
-F 2 "lib:TP_HOLE" H 9600 5250 60  0001 C CNN
-F 3 "~" H 9600 5250 60  0000 C CNN
-	1    9600 5250
-	1    0    0    -1
-$EndComp
 Text HLabel 4100 6450 2    60   Output ~ 0
 SPI1_CS_CODEC
@@
 	1    0    0    -1
 $EndComp
-Text HLabel 9150 5450 2    60   Output ~ 0
+Text HLabel 4100 7250 2    60   Output ~ 0
 ANALOG_EN
 $Comp
@@
 Wire Wire Line
 	8150 4350 8400 4350
-Wire Wire Line
-	9500 5250 9050 5250
 Wire Wire Line
 	8500 6000 8500 6100
@@
 Text Label 1700 2600 2    60   ~ 0
 CLK_EN
-Text Label 9450 5700 2    60   ~ 0
+Text Label 8200 3650 2    60   ~ 0
 CLK_EN
 Wire Wire Line
-	2900 7350 2750 7350
-Text Label 3400 3300 2    60   ~ 0
+	2900 6950 2100 6950
+Text Label 2100 6950 2    60   ~ 0
 LED2
 Wire Wire Line
-	3400 3300 3500 3300
+	3050 3300 3500 3300
 Text Label 8500 5500 1    60   ~ 0
 LED2
@@
 Wire Wire Line
 	8300 5500 8300 5700
-Text Label 2750 7350 2    60   ~ 0
+Text Label 3050 3300 2    60   ~ 0
 LED1
 Wire Wire Line
-	2900 7050 2750 7050
-Text Label 2750 7050 2    60   ~ 0
+	3500 4300 3050 4300
+Text Label 3050 4300 2    60   ~ 0
 LED3
 Text Label 8700 5500 1    60   ~ 0
@@
 $EndComp
 Wire Wire Line
-	6150 2550 6150 2450
+	6150 2450 6150 2550
 Wire Wire Line
 	6150 2500 6600 2500
@@
 Connection ~ 6450 2500
 Connection ~ 6150 2050
+Wire Wire Line
+	4100 7250 3700 7250
+Text Notes 2850 6950 2    40   ~ 0
+PWMC0_H0
+Text Notes 3500 4300 2    40   ~ 0
+PWMC0_H1
+Text Notes 3500 3300 2    40   ~ 0
+PWMC0_H1
+Wire Wire Line
+	4100 5950 3700 5950
+Wire Wire Line
+	4600 4100 4300 4100
+Wire Wire Line
+	8200 3650 8400 3650
 $EndSCHEMATC
