File: hw/rev2/micro.sch (KiCad schematic (older format))
At the start: 21 parts, among them P3 CONN_01X06, U4 K20X7_QFP64, X1 XTAL, X2 ASFLM2-12.288MHZ

Commit message: Most of a schematic
Parts:
- removed C29: 2.2u, lib:SMD0603, symbol CAP
- removed C30: 0.1u, lib:SMD0402, symbol CAP
- removed C34: 10n, lib:SMD0402, symbol CAP
- removed C35, C36: CAP, lib:SMD0402, symbol CAP
- removed D1: LTST-C19FD1WT, lib:LED-6PLCC, symbol LED3
- removed P3: CONN_01X06, lib:HDR_6X1_50MIL, symbol CONN_01X06
- removed R20: 10k, lib:SMD0402, symbol RES
- removed R30: 39, lib:SMD0402, symbol RES
- removed TP4: TP_PTE0, lib:TP_HOLE, symbol TP
- removed U4: K20X7_QFP64, lib:FREESCALE_QFP64, symbol K20X7_QFP64
- removed X1: XTAL, lib:TXC_7A, symbol XTAL
- removed X2: ASFLM2-12.288MHZ, lib:ASFLM, symbol OSC_W_EN
- added C1, C2, C3, C4, C5, C6, C8: 2.2u, Capacitors_SMD:C_0603, symbol symbols:CAP
- added C10, C9: 22u, Capacitors_SMD:C_1210, symbol symbols:CAP
- added C11, C7: 100n, Capacitors_SMD:C_0402, symbol symbols:CAP
- added C12, C14: 1u, Capacitors_SMD:C_0402, symbol symbols:CAP
- added C13: 10u, Capacitors_SMD:C_0805, symbol symbols:CAP
- added C15, C16, C17, C18, C19, C20: 0.1u, Capacitors_SMD:C_0402, symbol symbols:CAP
- added D1: LG L29K-F2J1-24-Z, LEDs:LED_0603, symbol Device:LED
- added D2: LS L29K-H1J2-1-Z, LEDs:LED_0603, symbol Device:LED
- added J1: Amphenol 20021122, symbol Connector:Conn_ARM_JTAG_SWD_10
- added R1: 100k, Resistors_SMD:R_0402, symbol Device:R_Small
- added R2: 820, Resistors_SMD:R_0402, symbol Device:R_Small
- added R4: 12k (1%), Resistors_SMD:R_0402, symbol symbols:RES
- added R5, R6: 2k, Resistors_SMD:R_0402, symbol Device:R_Small
- added R7: 100k, Resistors_SMD:R_0402, symbol symbols:RES
- added TP2, TP3, TP4, TP5, TP6: TP, Wire_Pads:SolderWirePad_single_1mmDrill, symbol symbols:TP
- added U1: STM32H743VITx, Housings_QFP:LQFP-100_14x14mm_Pitch0.5mm, symbol MCU_ST_STM32H7:STM32H743VITx
- added U2: USB3300-EZK, Housings_DFN_QFN:QFN-32-1EP_5x5mm_Pitch0.5mm, symbol Interface_USB:USB3300-EZK
- added U3: ADAU1772, Housings_DFN_QFN:QFN-40-1EP_6x6mm_Pitch0.5mm, symbol symbols:ADAU1772
- added X1: DSC6011JE1A-024.0000, Oscillators:Oscillator_SMD_SeikoEpson_SG210-4pin_2.5x2.0mm, symbol symbols:OSC_W_EN
- added X2: DSC6011CI2A-012.2880, Oscillators:Oscillator_SMD_EuroQuartz_XO32-4pin_3.2x2.5mm, symbol symbols:OSC_W_EN
- C31: footprint lib:SMD0603 -> Capacitors_SMD:C_0603; symbol CAP -> symbols:CAP
- C32, C33: footprint lib:SMD0402 -> Capacitors_SMD:C_0402; symbol CAP -> symbols:CAP
- C71: value 10n -> 100n; footprint lib:SMD0402 -> Capacitors_SMD:C_0402; symbol CAP -> symbols:CAP
- R21, R22, R24: footprint lib:SMD0402 -> Resistors_SMD:R_0402; symbol RES -> symbols:RES
- R23: value 220 -> 7.5; footprint lib:SMD0402 -> Resistors_SMD:R_0402; symbol RES -> symbols:RES
Connections:
- net labels added: +1V8, +3V3, +3V3A, CODEC_LRCLK, CODEC_SDI, CODEC_~PD, GNDA, HP_LN, HP_LP, HP_RN, HP_RP, MCLK, MCLK_EN, MIC0_IN, MIC1_IN, USB_CLKOUT, USB_D0, USB_D1, USB_D2, USB_D3, USB_D4, USB_D5, USB_D6, USB_D7, USB_DIR, USB_ID, USB_NXT, USB_RESET, USB_STP, USB_VBUS
- net labels removed: CODEC_LRCK, CODEC_MCLK, CODEC_PDN, CODEC_SDIN, HP_~SD, PGA0_D+, PGA0_D-, SPI1_CS_CODEC, SPI1_CS_FLASH, SPI1_SCK, SPI1_SIN, SPI1_SOUT, UART0_RX, UART0_TX, USB_5V
- wire segments 99 -> 302
- no-connect marks 2 -> 9
Other:
- note added: "Green"
- note added: "Red"
- note removed: ">Fs*48"
- note removed: "Fs*2"
- note removed: "Fs*256: 25.476MHz (for 96kHz)"

Commit message: Schematic roughly complete
Parts:
- added C22, C26, C28: 100n, Capacitors_SMD:C_0402, symbol symbols:CAP
- added C23: 4.7u, Capacitors_SMD:C_0805, symbol symbols:CAP
- J3: renamed from J1; footprint (none) -> Pin_Headers:Pin_Header_Straight_2x05_Pitch1.27mm
- renumbered C31 to C10, C32 to C11, C33 to C12, C7 to C13, C8 to C14, C9 to C15, C10 to C16, C11 to C17, C12 to C18, C13 to C19, C14 to C20, C15 to C21, C16 to C24, C17 to C25, C18 to C27, C19 to C29, C20 to C30, C71 to C31, C1 to C4, C2 to C5, C3 to C6, C4 to C7, C5 to C8, C6 to C9, R23 to R1, R7 to R10, R24 to R2, R1 to R3, R21 to R4, R22 to R5, R2 to R6, R4 to R7, R5 to R8, R6 to R9, U1 to U2, U2 to U3, U3 to U4
Connections:
- wire segments 302 -> 314

Commit message: Placement!
Parts:
- U4: footprint Housings_DFN_QFN:QFN-40-1EP_6x6mm_Pitch0.5mm -> lib:QFN-40-1EP_6x6mm_Pitch0.5mm
Connections:
- net labels added: 1V8_USB, USB_D_N, USB_D_P
- net labels removed: USB_D+, USB_D-
- wire segments 314 -> 315
Changed lines of the file:
@@
 EESchema Schematic File Version 4
 LIBS:audio_iface_rev2-cache
-EELAYER 26 0
+EELAYER 29 0
 EELAYER END
 $Descr B 17000 11000
@@
 $EndComp
 Text HLabel 9950 3100 0    60   BiDi ~ 0
-USB_D+
+USB_D_P
 Text HLabel 9950 3200 0    60   BiDi ~ 0
-USB_D-
+USB_D_N
 Text Label 2100 4150 0    60   ~ 0
 SWDIO
@@
 L symbols:CAP C31
 U 1 1 53697AF9
-P 14750 3050
-F 0 "C31" H 14770 3020 50  0000 L TNN
-F 1 "100n" H 14775 3070 30  0000 L BNN
-F 2 "Capacitors_SMD:C_0402" H 14750 3050 60  0001 C CNN
-F 3 "~" H 14750 3050 60  0000 C CNN
-	1    14750 3050
+P 15100 3050
+F 0 "C31" H 15120 3020 50  0000 L TNN
+F 1 "100n" H 15125 3070 30  0000 L BNN
+F 2 "Capacitors_SMD:C_0402" H 15100 3050 60  0001 C CNN
+F 3 "~" H 15100 3050 60  0000 C CNN
+	1    15100 3050
 	0    -1   -1   0
 $EndComp
@@
 	10250 3000 10600 3000
 $Comp
-L symbols:ADAU1772 U4
-U 1 1 5C11F03E
-P 12850 6950
-F 0 "U4" H 12850 5714 50  0000 C CNN
-F 1 "ADAU1772" H 12850 5623 50  0000 C CNN
-F 2 "Housings_DFN_QFN:QFN-40-1EP_6x6mm_Pitch0.5mm" H 12850 6950 50  0001 C CNN
-F 3 "http://www.analog.com/media/en/technical-documentation/data-sheets/ADAU1701.pdf" H 12850 6950 50  0001 C CNN
-	1    12850 6950
-	1    0    0    -1
-$EndComp
-$Comp
 L power:+1V8 #PWR027
 U 1 1 5C02D6F4
@@
 Text Label 14900 2850 0    50   ~ 0
 MCLK
-Wire Wire Line
-	14900 2850 14750 2850
 $Comp
 L power:GNDD #PWR032
@@
 	13850 2750 14100 2750
 Wire Wire Line
-	13900 3200 14750 3200
-Wire Wire Line
-	14750 3200 14750 3150
+	15100 3200 15100 3150
 Connection ~ 13900 3200
 Wire Wire Line
 	13900 3200 13900 2850
-Wire Wire Line
-	14750 2950 14750 2850
-Connection ~ 14750 2850
-Wire Wire Line
-	14750 2850 14700 2850
 Wire Wire Line
 	6950 7100 8100 7100
@@
 	1    0    0    -1
 $EndComp
-$Comp
-L power:+1V8 #PWR016
-U 1 1 5C17162D
-P 9900 3600
-F 0 "#PWR016" H 9900 3450 50  0001 C CNN
-F 1 "+1V8" H 9915 3773 50  0000 C CNN
-F 2 "" H 9900 3600 50  0001 C CNN
-F 3 "" H 9900 3600 50  0001 C CNN
-	1    9900 3600
-	1    0    0    -1
-$EndComp
 Wire Wire Line
 	9900 3600 9900 3650
@@
 U 1 1 5C280446
 P 1300 4150
+AR Path="/5C280446" Ref="J3"  Part="1"
+AR Path="/523BF424/5C280446" Ref="J3"  Part="1"
 F 0 "J3" H 1650 3600 50  0000 R CNN
 F 1 "Amphenol 20021122" V 850 4600 50  0000 R CNN
@@
 	13750 7900 13550 7900
 Connection ~ 12900 8300
-Wire Wire Line
-	12900 8300 12900 8100
 Wire Wire Line
 	13550 7800 13750 7800
@@
 Text Label 7450 6600 0    50   ~ 0
 USB_RESET
+Wire Wire Line
+	14700 2850 14900 2850
+Wire Wire Line
+	15100 2750 15100 2950
+Connection ~ 15100 2750
+Wire Wire Line
+	13900 3200 15100 3200
+Text Label 9900 3600 0    50   ~ 0
+1V8_USB
+Text Label 12450 2900 0    50   ~ 0
+1V8_USB
+Wire Wire Line
+	12900 8300 12900 8100
+$Comp
+L symbols:ADAU1772 U4
+U 1 1 5C11F03E
+P 12850 6950
+F 0 "U4" H 12850 5714 50  0000 C CNN
+F 1 "ADAU1772" H 12850 5623 50  0000 C CNN
+F 2 "lib:QFN-40-1EP_6x6mm_Pitch0.5mm" H 12850 6950 50  0001 C CNN
+F 3 "http://www.analog.com/media/en/technical-documentation/data-sheets/ADAU1701.pdf" H 12850 6950 50  0001 C CNN
+	1    12850 6950
+	1    0    0    -1
+$EndComp
+Wire Wire Line
+	12700 8100 12700 8300
+Wire Wire Line
+	12700 8300 12900 8300
 $EndSCHEMATC

Commit message: Much more routing
Parts:
- C10, C14, C4, C5, C6, C7, C8, C9: footprint Capacitors_SMD:C_0603 -> Capacitor_SMD:C_0603_1608Metric_Pad1.05x0.95mm_HandSolder
- C11, C12, C13, C17, C18, C20, C21, C22, C24, C25, C26, C27, C28, C29, C30, C31: footprint Capacitors_SMD:C_0402 -> Capacitor_SMD:C_0402_1005Metric
- C15, C16: footprint Capacitors_SMD:C_1210 -> Capacitor_SMD:C_1210_3225Metric
- C19, C23: footprint Capacitors_SMD:C_0805 -> Capacitor_SMD:C_0805_2012Metric_Pad1.15x1.40mm_HandSolder
- D1, D2: footprint LEDs:LED_0603 -> LED_SMD:LED_0603_1608Metric_Pad1.05x0.95mm_HandSolder
- J3: footprint Pin_Headers:Pin_Header_Straight_2x05_Pitch1.27mm -> Connector_PinHeader_1.27mm:PinHeader_2x05_P1.27mm_Vertical
- R1, R10, R2, R3, R4, R5, R6, R7, R8, R9: footprint Resistors_SMD:R_0402 -> Resistor_SMD:R_0402_1005Metric
- U2: footprint Housings_QFP:LQFP-100_14x14mm_Pitch0.5mm -> Package_QFP:LQFP-100_14x14mm_P0.5mm
- U3: footprint Housings_DFN_QFN:QFN-32-1EP_5x5mm_Pitch0.5mm -> Package_DFN_QFN:QFN-32-1EP_5x5mm_P0.5mm_EP3.1x3.1mm_ThermalVias
- U4: footprint lib:QFN-40-1EP_6x6mm_Pitch0.5mm -> Package_DFN_QFN:QFN-40-1EP_6x6mm_P0.5mm_EP4.6x4.6mm_ThermalVias
- X1: footprint Oscillators:Oscillator_SMD_SeikoEpson_SG210-4pin_2.5x2.0mm -> Oscillator:Oscillator_SMD_SeikoEpson_SG210-4Pin_2.5x2.0mm_HandSoldering
- X2: footprint Oscillators:Oscillator_SMD_EuroQuartz_XO32-4pin_3.2x2.5mm -> Oscillator:Oscillator_SMD_EuroQuartz_XO32-4Pin_3.2x2.5mm_HandSoldering
Connections:
- wire segments 315 -> 317

Commit message: Design nearly complete. One more check.
Parts:
- C10, C11, C12, C13, C14, C15, C16, C17, C18, C19, C20, C21, C22, C23, C24, C25, C26, C27, C28, C29, C30, C31, C4, C5, C6, C7, C8, C9: symbol symbols:CAP -> Device:C_Small
- R1, R10, R2, R4, R5, R7: symbol symbols:RES -> Device:R_Small
Connections:
- net labels removed: +3V
- wire segments 317 -> 318
- no-connect marks 9 -> 66
