File: hw/rev2/audio_iface_rev2.sch (KiCad schematic (older format))
At the start: 10 parts, among them J101 CONN_2, J102 CONN_2, J103 CONN_2, J104 CONN_2, J105 CONN_2, J106 CONN_2, J107 USBMICROCONN

Commit message: Lots of things: --Added RGB LED on timer outputs --Input: Moved capacitively coupled feedback nodes from vgnd to gnd --Output: LTC6242 for filtering to amplifier --Power: 2-stage supply for analog: USB 5V boost to 6V, LDO to 5V   Digital still using LDO from USB 5V and not caring about anyone   Bonus! Can completely shut off analog portion of board --Layout and routing: All of it TODO: final checks on layout and LVS (vs simulation) HEAD2HEAD2HEAD! TODO: adjust silkscreen, add logo TODO: debate adding 12.288MHz dedicated crystal
Parts:
- added R2, R3: 22R, ~, symbol RES
- gave numbers to parts that had none: 1
- renumbered J101 to J1, J102 to J2, J107 to J3, J103 to J4, J106 to J5, J104 to J6, J105 to J7, R101 to R1, TP102 to TP1
Connections:
- wire segments 80 -> 85
Changed lines of the file:
@@
 Sheet 1 6
 Title "Android DPOAE Interface"
-Date "22 apr 2014"
+Date "3 may 2014"
 Rev "2a"
 Comp "Sana AudioPulse"
@@
 $EndSheet
 $Comp
-L CONN_2 J101
+L CONN_2 J1
 U 1 1 523BE918
 P 1600 3000
-F 0 "J101" V 1550 3000 40  0000 C CNN
+F 0 "J1" V 1550 3000 40  0000 C CNN
 F 1 "CONN_2" V 1650 3000 40  0000 C CNN
 F 2 "~" H 1600 3000 60  0000 C CNN
@@
 $EndComp
 $Comp
-L RES R101
+L RES R1
 U 1 1 523BEA36
 P 2050 2650
-F 0 "R101" H 2120 2615 50  0000 L TNN
+F 0 "R1" H 2120 2615 50  0000 L TNN
 F 1 "3.9k (1%)" H 2050 2705 30  0000 C BNN
 F 2 "" H 2050 2650 60  0000 C CNN
@@
 F18 "I2C_SCL" B R 6100 4800 60
 F19 "I2C_SDA" B R 6100 4900 60
+F20 "ANALOG_EN" O L 4800 5500 60
 $EndSheet
 $Comp
-L USBMICROCONN J107
+L USBMICROCONN J3
 U 1 1 523BF69D
 P 2950 5750
-F 0 "J107" H 3000 5350 60  0001 C CNN
+F 0 "J3" H 3000 5350 60  0001 C CNN
 F 1 "USBMICROCONN" H 3000 5350 60  0000 C CNN
 F 2 "" H 2950 5750 60  0000 C CNN
@@
 $EndComp
 $Comp
-L CONN_2 J102
+L CONN_2 J2
 U 1 1 52486D64
 P 1600 3400
-F 0 "J102" V 1550 3400 40  0000 C CNN
+F 0 "J2" V 1550 3400 40  0000 C CNN
 F 1 "CONN_2" V 1650 3400 40  0000 C CNN
 F 2 "~" H 1600 3400 60  0000 C CNN
@@
 $EndComp
 $Comp
-L AGND_IN #PWR02
+L AGND_IN #PWR01
 U 1 1 52486D6B
 P 2050 3600
-F 0 "#PWR02" H 2050 3600 40  0001 C CNN
+F 0 "#PWR01" H 2050 3600 40  0001 C CNN
 F 1 "AGND_IN" H 2050 3530 50  0000 C CNN
 F 2 "" H 2050 3600 60  0000 C CNN
@@
 $EndComp
 $Comp
-L DGND #PWR03
+L DGND #PWR02
 U 1 1 524E1634
 P 3300 6100
-F 0 "#PWR03" H 3300 6100 40  0001 C CNN
+F 0 "#PWR02" H 3300 6100 40  0001 C CNN
 F 1 "DGND" H 3300 6030 40  0000 C CNN
 F 2 "" H 3300 6100 60  0000 C CNN
@@
 $EndComp
 $Comp
-L CONN_2 J104
+L CONN_2 J6
 U 1 1 524E6315
 P 9400 3000
-F 0 "J104" V 9350 3000 40  0000 C CNN
+F 0 "J6" V 9350 3000 40  0000 C CNN
 F 1 "CONN_2" V 9450 3000 40  0000 C CNN
 F 2 "~" H 9400 3000 60  0000 C CNN
@@
 $EndComp
 $Comp
-L CONN_2 J105
+L CONN_2 J7
 U 1 1 524E6F43
 P 9400 3500
-F 0 "J105" V 9350 3500 40  0000 C CNN
+F 0 "J7" V 9350 3500 40  0000 C CNN
 F 1 "CONN_2" V 9450 3500 40  0000 C CNN
 F 2 "~" H 9400 3500 60  0000 C CNN
@@
 F0 "Power" 50
 F1 "power.sch" 50
+F2 "ANALOG_EN" I L 4600 950 60
 $EndSheet
 $Comp
-L CONN_2 J103
+L CONN_2 J4
 U 1 1 5251A6D0
 P 7750 5250
-F 0 "J103" V 7700 5250 40  0000 C CNN
+F 0 "J4" V 7700 5250 40  0000 C CNN
 F 1 "CONN_2" V 7800 5250 40  0000 C CNN
 F 2 "~" H 7750 5250 60  0000 C CNN
@@
 $EndComp
 $Comp
-L TP TP102
+L TP TP1
 U 1 1 5251B035
 P 3600 6200
-F 0 "TP102" H 3600 6100 60  0000 C CNN
+F 0 "TP1" H 3600 6100 60  0000 C CNN
 F 1 "TP_USB_ID" H 3600 6300 60  0000 C CNN
 F 2 "~" H 3600 6200 60  0000 C CNN
@@
 	0    1    1    0
 $EndComp
-Text Notes 3650 5950 0    60   ~ 0
+Text Notes 3850 5950 3    60   ~ 0
 Floating for USB device
 $Comp
-L +5VA #PWR06
+L +5VA #PWR03
 U 1 1 525790A9
 P 2050 2400
-F 0 "#PWR06" H 2050 2530 20  0001 C CNN
+F 0 "#PWR03" H 2050 2530 20  0001 C CNN
 F 1 "+5VA" H 2050 2500 30  0000 C CNN
 F 2 "" H 2050 2400 60  0000 C CNN
@@
 $EndComp
 $Comp
-L CONN_2 J106
+L CONN_2 J5
 U 1 1 52581553
 P 7750 6150
-F 0 "J106" V 7700 6150 40  0000 C CNN
+F 0 "J5" V 7700 6150 40  0000 C CNN
 F 1 "CONN_2" V 7800 6150 40  0000 C CNN
 F 2 "~" H 7750 6150 60  0000 C CNN
@@
 	6700 4700 6700 3500
 Wire Wire Line
-	3200 5700 4800 5700
-Wire Wire Line
-	4800 5800 3200 5800
-Wire Wire Line
 	3300 6100 3300 6000
 Wire Wire Line
@@
 	8600 3400 9050 3400
 $Comp
-L USB_5V #PWR?
+L USB_5V #PWR04
 U 1 1 5350403E
 P 3600 5500
-F 0 "#PWR?" H 3600 5460 30  0001 C CNN
+F 0 "#PWR04" H 3600 5460 30  0001 C CNN
 F 1 "USB_5V" H 3600 5610 30  0000 C CNN
 F 2 "~" H 3600 5500 60  0000 C CNN
@@
 	8600 3100 8600 3750
 $Comp
-L AGND_OUT #PWR?
+L AGND_OUT #PWR05
 U 1 1 53573760
 P 8600 3750
-F 0 "#PWR?" H 8600 3750 40  0001 C CNN
+F 0 "#PWR05" H 8600 3750 40  0001 C CNN
 F 1 "AGND_OUT" H 8600 3680 50  0000 C CNN
 F 2 "~" H 8600 3750 60  0000 C CNN
@@
 Connection ~ 8600 3400
 $Comp
-L CAP C?
+L CAP C1
 U 1 1 535741F7
 P 2300 3100
-F 0 "C?" H 2320 3070 50  0000 L TNN
+F 0 "C1" H 2320 3070 50  0000 L TNN
 F 1 "10n" H 2325 3120 30  0000 L BNN
 F 2 "~" H 2300 3100 60  0000 C CNN
@@
 Text Notes 2100 3250 0    60   ~ 0
 DNP
+$Comp
+L RES R2
+U 1 1 5357CAB5
+P 3850 5700
+F 0 "R2" H 3920 5665 50  0000 L TNN
+F 1 "22R" H 3850 5755 30  0000 C BNN
+F 2 "~" H 3850 5700 60  0000 C CNN
+F 3 "~" H 3850 5700 60  0000 C CNN
+	1    3850 5700
+	1    0    0    -1
+$EndComp
+$Comp
+L RES R3
+U 1 1 5357CCFF
+P 4200 5800
+F 0 "R3" H 4270 5765 50  0000 L TNN
+F 1 "22R" H 4200 5855 30  0000 C BNN
+F 2 "~" H 4200 5800 60  0000 C CNN
+F 3 "~" H 4200 5800 60  0000 C CNN
+	1    4200 5800
+	1    0    0    -1
+$EndComp
+Wire Wire Line
+	4350 5800 4800 5800
+Wire Wire Line
+	4800 5700 4000 5700
+Wire Wire Line
+	4050 5800 3200 5800
+Wire Wire Line
+	3200 5700 3700 5700
+Wire Wire Line
+	4800 5500 4100 5500
+Wire Wire Line
+	4100 5500 4100 950
+Wire Wire Line
+	4100 950  4600 950
 $EndSCHEMATC

Commit message: Added serial flash module to schematic and began layout
Parts:
- added C?: 0.1u, SMD0402, symbol CAP
- added C?: 1u, SMD0402, symbol CAP
- added R?: 100k, ~, symbol RES
- added U?: MT29FXX01A, ~, symbol MT29FXX01A
Connections:
- net labels added: +3V, GND
- wire segments 85 -> 114

Commit message: Added SMA connectors, still need to recreate keepouts
Parts:
- removed J1, J6, J7: CONN_2, ~, symbol CONN_2
- added J1, J6, J7: COAX, ~, symbol COAX
- gave numbers to parts that had none: 4
Connections:
- wire segments 114 -> 116

Commit message: Started board upgrade to 4 layers and better signal isolation
Parts:
- removed J2, J4, J5: CONN_2, ~, symbol CONN_2
- added C74: 47p, lib:SMD0402, symbol CAP
- added C75: 10u, lib:SMD0805, symbol CAP
- added C76: 0.1u, lib:SMD0402, symbol CAP
- added FB1, FB2: BLM18PG221SN1D, lib:SMD0805, symbol FB
- added J2, P1, P2: CONN_01X02, lib:HDR_2X1_50MIL, symbol CONN_01X02
- C1, R2, R3, R39: footprint ~ -> lib:SMD0402
- C16, C73: footprint SMD0402 -> lib:SMD0402
- J1, J6, J7: footprint ~ -> lib:SMA_EDGE
- J3: footprint (none) -> lib:FCI_10118194
- R1: footprint (none) -> lib:SMD0402
- TP1: footprint ~ -> lib:TP_HOLE
- U9: footprint ~ -> MICRON_VFBGA63:MICRON_VFBGA63
Connections:
- net labels added: GNDD
- net labels removed: DGND
- wire segments 116 -> 120

Commit message: Routed out 4-layer variant--now need to do silkscreens and such
Parts:
- renumbered P1 to J4, P2 to J5
Changed lines of the file:
@@
 $EndComp
 $Comp
-L CONN_01X02 P2
+L CONN_01X02 J5
 U 1 1 57D4EFF8
 P 7600 6150
-F 0 "P2" H 7600 6300 50  0000 C CNN
+F 0 "J5" H 7600 6300 50  0000 C CNN
 F 1 "CONN_01X02" V 7700 6150 50  0000 C CNN
 F 2 "lib:HDR_2X1_50MIL" H 7600 6150 50  0001 C CNN
@@
 $EndComp
 $Comp
-L CONN_01X02 P1
+L CONN_01X02 J4
 U 1 1 57D5084F
 P 7600 5250
-F 0 "P1" H 7600 5400 50  0000 C CNN
+F 0 "J4" H 7600 5400 50  0000 C CNN
 F 1 "CONN_01X02" V 7700 5250 50  0000 C CNN
 F 2 "lib:HDR_2X1_50MIL" H 7600 5250 50  0001 C CNN
