File: hw/rev2/audio_iface_rev2.sch (KiCad schematic (older format))
At the start: 14 parts, among them J1 COAX, J2 CONN_01X02, J3 USBMICROCONN, J4 CONN_01X02, J6 COAX, J7 COAX

Commit message: Fully routed
Connections:
- wire segments 86 -> 85
Changed lines of the file:
@@
 	6200 3800 6100 3800
-Wire Wire Line
-	6100 5700 7800 5700
 Wire Wire Line
 	6300 5700 6300 3700
@@
 Wire Wire Line
 	4100 950  4600 950
-Wire Wire Line
-	7800 5700 7800 5200
-Connection ~ 6300 5700
 Wire Wire Line
 	8600 3850 9950 3850
@@
 Text Label 2450 5700 0    60   ~ 0
 USB_D_N
+Wire Wire Line
+	6300 5700 6100 5700
 $EndSCHEMATC

Commit message: Simplified input processing, reduced amp count by 2
Parts:
- removed J2: CONN_01X02, lib:HDR_2X1_50MIL, symbol CONN_01X02
Connections:
- wire segments 85 -> 82
Changed lines of the file:
@@
 F5 "EXT_DIFF_N" O R 3700 3300 60
 F6 "EXT_DIFF_P" O R 3700 3200 60
-F7 "EXT_IN" I L 2500 3300 60
 $EndSheet
 $Sheet
@@
 L AGND_IN #PWR01
 U 1 1 52486D6B
-P 2050 3600
-F 0 "#PWR01" H 2050 3600 40  0001 C CNN
-F 1 "AGND_IN" H 2050 3530 50  0000 C CNN
-F 2 "" H 2050 3600 60  0000 C CNN
-F 3 "" H 2050 3600 60  0000 C CNN
-	1    2050 3600
+P 2300 3400
+F 0 "#PWR01" H 2300 3400 40  0001 C CNN
+F 1 "AGND_IN" H 2300 3330 50  0000 C CNN
+F 2 "" H 2300 3400 60  0000 C CNN
+F 3 "" H 2300 3400 60  0000 C CNN
+	1    2300 3400
 	1    0    0    -1
 $EndComp
@@
 	4800 3300 3700 3300
 Wire Wire Line
-	2050 3400 2050 3600
-Wire Wire Line
-	1950 3400 2300 3400
-Wire Wire Line
-	1950 3300 2500 3300
-Wire Wire Line
 	4800 4700 4700 4700
 Wire Wire Line
@@
 Wire Wire Line
 	8600 3100 8600 4000
-Connection ~ 2050 3400
 Wire Wire Line
 	2300 3400 2300 3200
@@
 $EndComp
 $Comp
-L CONN_01X02 J2
-U 1 1 57D51C49
-P 1750 3350
-F 0 "J2" H 1750 3500 50  0000 C CNN
-F 1 "CONN_01X02" V 1850 3350 50  0000 C CNN
-F 2 "lib:HDR_2X1_50MIL" H 1750 3350 50  0001 C CNN
-F 3 "" H 1750 3350 50  0000 C CNN
-	1    1750 3350
-	-1   0    0    1
-$EndComp
-$Comp

Commit message: Lots of layout and grounding changes. DRC good
Connections:
- net labels added: GND
- net labels removed: GNDD
Changed lines of the file:
@@
 	0    1    1    0
-$EndComp
-$Comp
-L AGND_IN #PWR01
-U 1 1 52486D6B
-P 2300 3400
-F 0 "#PWR01" H 2300 3400 40  0001 C CNN
-F 1 "AGND_IN" H 2300 3330 50  0000 C CNN
-F 2 "" H 2300 3400 60  0000 C CNN
-F 3 "" H 2300 3400 60  0000 C CNN
-	1    2300 3400
-	1    0    0    -1
 $EndComp
 $Sheet
@@
 Floating for USB device
 $Comp
-L +5VA #PWR02
+L +5VA #PWR01
 U 1 1 525790A9
 P 2050 2400
-F 0 "#PWR02" H 2050 2530 20  0001 C CNN
+F 0 "#PWR01" H 2050 2530 20  0001 C CNN
 F 1 "+5VA" H 2050 2500 30  0000 C CNN
 F 2 "" H 2050 2400 60  0000 C CNN
@@
 $EndSheet
 $Comp
-L USB_5V #PWR03
+L USB_5V #PWR02
 U 1 1 5350403E
 P 3950 4900
-F 0 "#PWR03" H 3950 4860 30  0001 C CNN
+F 0 "#PWR02" H 3950 4860 30  0001 C CNN
 F 1 "USB_5V" H 3950 5010 30  0000 C CNN
 F 2 "~" H 3950 4900 60  0000 C CNN
 F 3 "~" H 3950 4900 60  0000 C CNN
 	1    3950 4900
-	1    0    0    -1
-$EndComp
-$Comp
-L AGND_OUT #PWR04
-U 1 1 53573760
-P 8600 4000
-F 0 "#PWR04" H 8600 4000 40  0001 C CNN
-F 1 "AGND_OUT" H 8600 3930 50  0000 C CNN
-F 2 "~" H 8600 4000 60  0000 C CNN
-F 3 "~" H 8600 4000 60  0000 C CNN
-	1    8600 4000
 	1    0    0    -1
 $EndComp
@@
 	-1   0    0    -1
 $EndComp
-$Comp
-L AGND_IN #PWR05
-U 1 1 5552EDD2
-P 1050 3800
-F 0 "#PWR05" H 1050 3800 40  0001 C CNN
-F 1 "AGND_IN" H 1050 3730 50  0000 C CNN
-F 2 "" H 1050 3800 60  0000 C CNN
-F 3 "" H 1050 3800 60  0000 C CNN
-	1    1050 3800
-	1    0    0    -1
-$EndComp
 Wire Wire Line
 	1050 3800 1050 3150
-$Comp
-L GNDD #PWR06
-U 1 1 57D4EA5B
-P 3300 6500
-F 0 "#PWR06" H 3300 6250 50  0001 C CNN
-F 1 "GNDD" H 3300 6350 50  0000 C CNN
-F 2 "" H 3300 6500 50  0000 C CNN
-F 3 "" H 3300 6500 50  0000 C CNN
-	1    3300 6500
-	1    0    0    -1
-$EndComp
 $Comp
 L CONN_01X02 J4
@@
 	3400 5000 3400 5050
 Connection ~ 3400 5000
-$Comp
-L GNDD #PWR07
-U 1 1 57D676D1
-P 3400 5500
-F 0 "#PWR07" H 3400 5250 50  0001 C CNN
-F 1 "GNDD" H 3400 5350 50  0000 C CNN
-F 2 "" H 3400 5500 50  0000 C CNN
-F 3 "" H 3400 5500 50  0000 C CNN
-	1    3400 5500
-	1    0    0    -1
-$EndComp
 Wire Wire Line
 	3400 5250 3400 5500
@@
 Wire Wire Line
 	6300 5700 6100 5700
+$Comp
+L AGND_OUT #PWR03
+U 1 1 582A8666
+P 8600 4000
+F 0 "#PWR03" H 8600 4000 40  0001 C CNN
+F 1 "AGND_OUT" H 8600 3930 50  0000 C CNN
+F 2 "" H 8600 4000 60  0000 C CNN
+F 3 "" H 8600 4000 60  0000 C CNN
+	1    8600 4000
+	1    0    0    -1
+$EndComp
+$Comp
+L AGND_IN #PWR04
+U 1 1 582A9203
+P 2300 3400
+F 0 "#PWR04" H 2300 3400 40  0001 C CNN
+F 1 "AGND_IN" H 2300 3330 50  0000 C CNN
+F 2 "" H 2300 3400 60  0000 C CNN
+F 3 "" H 2300 3400 60  0000 C CNN
+	1    2300 3400
+	1    0    0    -1
+$EndComp
+$Comp
+L AGND_IN #PWR05
+U 1 1 582A960F
+P 1050 3800
+F 0 "#PWR05" H 1050 3800 40  0001 C CNN
+F 1 "AGND_IN" H 1050 3730 50  0000 C CNN
+F 2 "" H 1050 3800 60  0000 C CNN
+F 3 "" H 1050 3800 60  0000 C CNN
+	1    1050 3800
+	1    0    0    -1
+$EndComp
+$Comp
+L GND #PWR06
+U 1 1 582A9A8A
+P 3300 6500
+F 0 "#PWR06" H 3300 6250 50  0001 C CNN
+F 1 "GND" H 3300 6350 50  0000 C CNN
+F 2 "" H 3300 6500 50  0000 C CNN
+F 3 "" H 3300 6500 50  0000 C CNN
+	1    3300 6500
+	1    0    0    -1
+$EndComp
+$Comp
+L GND #PWR07
+U 1 1 582AA252
+P 3400 5500
+F 0 "#PWR07" H 3400 5250 50  0001 C CNN
+F 1 "GND" H 3400 5350 50  0000 C CNN
+F 2 "" H 3400 5500 50  0000 C CNN
+F 3 "" H 3400 5500 50  0000 C CNN
+	1    3400 5500
+	1    0    0    -1
+$EndComp
 $EndSCHEMATC

Commit message: Fixed power connections for S70--submitted PCB
Parts:
- FB1, FB2: footprint lib:SMD0805 -> lib:SMD0603
Changed lines of the file:
@@
 LIBS:contrib
 LIBS:valves
+LIBS:audio_iface_rev2-cache
 EELAYER 25 0
 EELAYER END
@@
 F 0 "FB1" H 3370 6215 50  0000 L TNN
 F 1 "BLM18PG221SN1D" H 3235 6325 30  0000 C BNN
-F 2 "lib:SMD0805" H 3280 6270 60  0001 C CNN
+F 2 "lib:SMD0603" H 3280 6270 60  0001 C CNN
 F 3 "" H 3280 6270 60  0000 C CNN
 	1    3300 6250
@@
 F 0 "FB2" H 3670 4965 50  0000 L TNN
 F 1 "BLM18PG221SN1D" H 3535 5075 30  0000 C BNN
-F 2 "lib:SMD0805" H 3580 5020 60  0001 C CNN
+F 2 "lib:SMD0603" H 3580 5020 60  0001 C CNN
 F 3 "" H 3580 5020 60  0000 C CNN
 	1    3600 5000

Commit message: Finished schematic and layout with STM32F7
Parts:
- removed TP1: TP_USB_ID, lib:TP_HOLE, symbol TP
Connections:
- wire segments 82 -> 83
Other:
- note removed: "Floating for USB device"
Changed lines of the file:
@@
 F18 "ANALOG_EN" O L 4800 5500 60
 F19 "SPI1_SIN" I R 6100 5900 60
+F20 "USB_VBUS" I L 4800 6000 60
+F21 "USB_ID" B L 4800 5900 60
 $EndSheet
 $Comp
@@
 $EndSheet
 $Comp
-L TP TP1
-U 1 1 5251B035
-P 3600 6200
-F 0 "TP1" H 3600 6100 60  0000 C CNN
-F 1 "TP_USB_ID" H 3600 6300 60  0000 C CNN
-F 2 "lib:TP_HOLE" H 3600 6200 60  0001 C CNN
-F 3 "~" H 3600 6200 60  0000 C CNN
-	1    3600 6200
-	0    1    1    0
-$EndComp
-Text Notes 3850 5950 3    60   ~ 0
-Floating for USB device
-$Comp
-L +5VA #PWR2
+L +5VA #PWR01
 U 1 1 525790A9
 P 2050 2400
-F 0 "#PWR2" H 2050 2530 20  0001 C CNN
+F 0 "#PWR01" H 2050 2530 20  0001 C CNN
 F 1 "+5VA" H 2050 2500 30  0000 C CNN
 F 2 "" H 2050 2400 60  0000 C CNN
@@
 $EndSheet
 $Comp
-L USB_5V #PWR6
+L USB_5V #PWR02
 U 1 1 5350403E
-P 3950 4900
-F 0 "#PWR6" H 3950 4860 30  0001 C CNN
-F 1 "USB_5V" H 3950 5010 30  0000 C CNN
-F 2 "~" H 3950 4900 60  0000 C CNN
-F 3 "~" H 3950 4900 60  0000 C CNN
-	1    3950 4900
+P 4000 4900
+F 0 "#PWR02" H 4000 4860 30  0001 C CNN
+F 1 "USB_5V" H 4000 5010 30  0000 C CNN
+F 2 "~" H 4000 4900 60  0000 C CNN
+F 3 "~" H 4000 4900 60  0000 C CNN
+	1    4000 4900
 	1    0    0    -1
 $EndComp
@@
 	6700 4700 6700 3500
 Wire Wire Line
-	3300 6100 3300 6000
-Wire Wire Line
-	3300 6000 2300 6000
+	2800 6100 2800 6000
+Wire Wire Line
+	2800 6000 2300 6000
 Wire Wire Line
 	9050 2900 8100 2900
@@
 	6100 5300 7400 5300
 Wire Wire Line
-	3600 6100 3600 5900
-Wire Wire Line
-	3600 5900 2300 5900
+	2300 5900 4800 5900
 Wire Wire Line
 	6100 5600 6200 5600
@@
 L FB FB1
 U 1 1 57D53855
-P 3300 6250
-F 0 "FB1" H 3370 6215 50  0000 L TNN
-F 1 "BLM18PG221SN1D" H 3235 6325 30  0000 C BNN
-F 2 "lib:SMD0603" H 3280 6270 60  0001 C CNN
-F 3 "" H 3280 6270 60  0000 C CNN
-	1    3300 6250
+P 2800 6250
+F 0 "FB1" H 2870 6215 50  0000 L TNN
+F 1 "BLM18PG221SN1D" H 2735 6325 30  0000 C BNN
+F 2 "lib:SMD0603" H 2780 6270 60  0001 C CNN
+F 3 "" H 2780 6270 60  0000 C CNN
+	1    2800 6250
 	0    1    1    0
 $EndComp
 Wire Wire Line
-	3300 6500 3300 6400
+	2800 6500 2800 6400
 $Comp
 L CAP C75
 U 1 1 57D66AF8
-P 3400 5150
-F 0 "C75" H 3420 5120 50  0000 L TNN
-F 1 "10u" H 3425 5170 30  0000 L BNN
-F 2 "lib:SMD0805" H 3400 5150 60  0001 C CNN
-F 3 "" H 3400 5150 60  0000 C CNN
-	1    3400 5150
+P 3450 5150
+F 0 "C75" H 3470 5120 50  0000 L TNN
+F 1 "10u" H 3475 5170 30  0000 L BNN
+F 2 "lib:SMD0805" H 3450 5150 60  0001 C CNN
+F 3 "" H 3450 5150 60  0000 C CNN
+	1    3450 5150
 	0    1    1    0
 $EndComp
@@
 L FB FB2
 U 1 1 57D66D61
-P 3600 5000
-F 0 "FB2" H 3670 4965 50  0000 L TNN
-F 1 "BLM18PG221SN1D" H 3535 5075 30  0000 C BNN
-F 2 "lib:SMD0603" H 3580 5020 60  0001 C CNN
-F 3 "" H 3580 5020 60  0000 C CNN
-	1    3600 5000
+P 3650 5000
+F 0 "FB2" H 3720 4965 50  0000 L TNN
+F 1 "BLM18PG221SN1D" H 3585 5075 30  0000 C BNN
+F 2 "lib:SMD0603" H 3630 5020 60  0001 C CNN
+F 3 "" H 3630 5020 60  0000 C CNN
+	1    3650 5000
 	-1   0    0    1
 $EndComp
@@
 	2550 5600 2550 5000
 Wire Wire Line
-	2550 5000 3450 5000
-Wire Wire Line
-	3400 5000 3400 5050
-Connection ~ 3400 5000
-Wire Wire Line
-	3400 5250 3400 5500
+	2550 5000 3500 5000
+Wire Wire Line
+	3450 5000 3450 5050
+Connection ~ 3450 5000
+Wire Wire Line
+	3450 5250 3450 5500
 $Comp
 L CAP C76
 U 1 1 57D6798C
-P 3850 5150
-F 0 "C76" H 3870 5120 50  0000 L TNN
-F 1 "0.1u" H 3875 5170 30  0000 L BNN
-F 2 "lib:SMD0402" H 3850 5150 60  0001 C CNN
-F 3 "" H 3850 5150 60  0000 C CNN
-	1    3850 5150
+P 3900 5150
+F 0 "C76" H 3920 5120 50  0000 L TNN
+F 1 "0.1u" H 3925 5170 30  0000 L BNN
+F 2 "lib:SMD0402" H 3900 5150 60  0001 C CNN
+F 3 "" H 3900 5150 60  0000 C CNN
+	1    3900 5150
 	0    1    1    0
 $EndComp
 Wire Wire Line
-	3750 5000 3950 5000
-Wire Wire Line
-	3850 5000 3850 5050
-Wire Wire Line
-	3850 5250 3850 5450
-Wire Wire Line
-	3850 5450 3400 5450
-Connection ~ 3400 5450
-Wire Wire Line
-	3950 5000 3950 4900
-Connection ~ 3850 5000
+	3800 5000 4000 5000
+Wire Wire Line
+	3900 5000 3900 5050
+Wire Wire Line
+	3900 5250 3900 5450
+Wire Wire Line
+	3900 5450 3450 5450
+Connection ~ 3450 5450
+Wire Wire Line
+	4000 5000 4000 4900
+Connection ~ 3900 5000
 $Comp
 L TP TP14
@@
 	6300 5700 6100 5700
 $Comp
-L AGND_OUT #PWR7
+L AGND_OUT #PWR03
 U 1 1 582A8666
 P 8600 4000
-F 0 "#PWR7" H 8600 4000 40  0001 C CNN
+F 0 "#PWR03" H 8600 4000 40  0001 C CNN
 F 1 "AGND_OUT" H 8600 3930 50  0000 C CNN
 F 2 "" H 8600 4000 60  0000 C CNN
@@
 $EndComp
 $Comp
-L AGND_IN #PWR3
+L AGND_IN #PWR04
 U 1 1 582A9203
 P 2300 3400
-F 0 "#PWR3" H 2300 3400 40  0001 C CNN
+F 0 "#PWR04" H 2300 3400 40  0001 C CNN
 F 1 "AGND_IN" H 2300 3330 50  0000 C CNN
 F 2 "" H 2300 3400 60  0000 C CNN
@@
 $EndComp
 $Comp
-L AGND_IN #PWR1
+L AGND_IN #PWR05
 U 1 1 582A960F
 P 1050 3800
-F 0 "#PWR1" H 1050 3800 40  0001 C CNN
+F 0 "#PWR05" H 1050 3800 40  0001 C CNN
 F 1 "AGND_IN" H 1050 3730 50  0000 C CNN
 F 2 "" H 1050 3800 60  0000 C CNN
@@
 $EndComp
 $Comp
-L GND #PWR4
+L GND #PWR06
 U 1 1 582A9A8A
-P 3300 6500
-F 0 "#PWR4" H 3300 6250 50  0001 C CNN
-F 1 "GND" H 3300 6350 50  0000 C CNN
-F 2 "" H 3300 6500 50  0000 C CNN
-F 3 "" H 3300 6500 50  0000 C CNN
-	1    3300 6500
-	1    0    0    -1
-$EndComp
-$Comp
-L GND #PWR5
+P 2800 6500
+F 0 "#PWR06" H 2800 6250 50  0001 C CNN
+F 1 "GND" H 2800 6350 50  0000 C CNN
+F 2 "" H 2800 6500 50  0000 C CNN
+F 3 "" H 2800 6500 50  0000 C CNN
+	1    2800 6500
+	1    0    0    -1
+$EndComp
+$Comp
+L GND #PWR07
 U 1 1 582AA252
-P 3400 5500
-F 0 "#PWR5" H 3400 5250 50  0001 C CNN
-F 1 "GND" H 3400 5350 50  0000 C CNN
-F 2 "" H 3400 5500 50  0000 C CNN
-F 3 "" H 3400 5500 50  0000 C CNN
-	1    3400 5500
-	1    0    0    -1
-$EndComp
+P 3450 5500
+F 0 "#PWR07" H 3450 5250 50  0001 C CNN
+F 1 "GND" H 3450 5350 50  0000 C CNN
+F 2 "" H 3450 5500 50  0000 C CNN
+F 3 "" H 3450 5500 50  0000 C CNN
+	1    3450 5500
+	1    0    0    -1
+$EndComp
+Wire Wire Line
+	3200 6000 4800 6000
+Wire Wire Line
+	3200 6000 3200 5000
+Connection ~ 3200 5000
 $EndSCHEMATC
