File: hw/rev2/audio_iface_rev2.sch (KiCad schematic (older format))
At the start: 21 parts, among them J1 COAX, J2 CONN_01X02, J3 USBMICROCONN, J4 CONN_01X02, J5 CONN_01X02, J6 COAX, J7 COAX, U9 MT29FXX01A

Commit message: Submitted PCB revision
Parts:
- removed C74: 47p, lib:SMD0402, symbol CAP
- added TP14: TP, lib:TP_HOLE, symbol TP
Connections:
- wire segments 120 -> 118
Changed lines of the file:
@@
 $EndSheet
 $Comp
-L USB_5V #PWR7
+L USB_5V #PWR6
 U 1 1 5350403E
 P 3950 4900
-F 0 "#PWR7" H 3950 4860 30  0001 C CNN
+F 0 "#PWR6" H 3950 4860 30  0001 C CNN
 F 1 "USB_5V" H 3950 5010 30  0000 C CNN
 F 2 "~" H 3950 4900 60  0000 C CNN
@@
 $EndComp
 $Comp
-L AGND_OUT #PWR10
+L AGND_OUT #PWR9
 U 1 1 53573760
 P 8600 4000
-F 0 "#PWR10" H 8600 4000 40  0001 C CNN
+F 0 "#PWR9" H 8600 4000 40  0001 C CNN
 F 1 "AGND_OUT" H 8600 3930 50  0000 C CNN
 F 2 "~" H 8600 4000 60  0000 C CNN
@@
 $EndComp
 $Comp
-L +3V #PWR8
+L +3V #PWR7
 U 1 1 5551B31B
 P 8450 5350
-F 0 "#PWR8" H 8450 5310 30  0001 C CNN
+F 0 "#PWR7" H 8450 5310 30  0001 C CNN
 F 1 "+3V" H 8450 5460 30  0000 C CNN
 F 2 "~" H 8450 5350 60  0000 C CNN
@@
 $EndComp
 $Comp
-L GND #PWR9
+L GND #PWR8
 U 1 1 5551C3F8
 P 8450 6400
-F 0 "#PWR9" H 8450 6400 30  0001 C CNN
+F 0 "#PWR8" H 8450 6400 30  0001 C CNN
 F 1 "GND" H 8450 6330 30  0001 C CNN
 F 2 "" H 8450 6400 60  0000 C CNN
@@
 	1050 3800 1050 3150
 $Comp
-L GNDD #PWR5
+L GNDD #PWR4
 U 1 1 57D4EA5B
 P 3300 6500
-F 0 "#PWR5" H 3300 6250 50  0001 C CNN
+F 0 "#PWR4" H 3300 6250 50  0001 C CNN
 F 1 "GNDD" H 3300 6350 50  0000 C CNN
 F 2 "" H 3300 6500 50  0000 C CNN
@@
 Connection ~ 3400 5000
 $Comp
-L GNDD #PWR6
+L GNDD #PWR5
 U 1 1 57D676D1
 P 3400 5500
-F 0 "#PWR6" H 3400 5250 50  0001 C CNN
+F 0 "#PWR5" H 3400 5250 50  0001 C CNN
 F 1 "GNDD" H 3400 5350 50  0000 C CNN
 F 2 "" H 3400 5500 50  0000 C CNN
@@
 Connection ~ 3850 5000
 $Comp
-L CAP C74
-U 1 1 57D6B4C5
-P 2400 6300
-F 0 "C74" H 2420 6270 50  0000 L TNN
-F 1 "47p" H 2425 6320 30  0000 L BNN
-F 2 "lib:SMD0402" H 2400 6300 60  0001 C CNN
-F 3 "" H 2400 6300 60  0000 C CNN
-	1    2400 6300
-	0    1    1    0
-$EndComp
-Wire Wire Line
-	2300 6100 2400 6100
-Wire Wire Line
-	2400 6100 2400 6200
-$Comp
-L GNDD #PWR4
-U 1 1 57D6BD63
-P 2400 6500
-F 0 "#PWR4" H 2400 6250 50  0001 C CNN
-F 1 "GNDD" H 2400 6350 50  0000 C CNN
-F 2 "" H 2400 6500 50  0000 C CNN
-F 3 "" H 2400 6500 50  0000 C CNN
-	1    2400 6500
-	1    0    0    -1
-$EndComp
-Wire Wire Line
-	2400 6400 2400 6500
-Text Notes 2200 6250 0    60   ~ 0
-DNP
+L TP TP14
+U 1 1 57EDDF81
+P 1600 2500
+F 0 "TP14" H 1600 2400 60  0000 C CNN
+F 1 "TP" H 1600 2600 60  0000 C CNN
+F 2 "lib:TP_HOLE" H 1600 2500 60  0001 C CNN
+F 3 "~" H 1600 2500 60  0000 C CNN
+	1    1600 2500
+	0    -1   -1   0
+$EndComp
+Wire Wire Line
+	1600 2600 1600 2900
+Connection ~ 1600 2900
 $EndSCHEMATC

Commit message: Most of a schematic
Parts:
- removed C1: 10n, lib:SMD0402, symbol CAP
- removed C16: 0.1u, lib:SMD0402, symbol CAP
- removed C73: 1u, lib:SMD0402, symbol CAP
- removed J1, J6, J7: COAX, lib:SMA_EDGE, symbol COAX
- removed J2, J4, J5: CONN_01X02, lib:HDR_2X1_50MIL, symbol CONN_01X02
- removed J3: USBMICROCONN, lib:FCI_10118194, symbol USBMICROCONN
- removed R1: 3.9k (1%), lib:SMD0402, symbol RES
- removed R2, R3: 22R, lib:SMD0402, symbol RES
- removed R39: 100k, lib:SMD0402, symbol RES
- removed TP14: TP, lib:TP_HOLE, symbol TP
- removed U9: MT29FXX01A, MICRON_VFBGA63:MICRON_VFBGA63, symbol MT29FXX01A
- added C30: 2.2u, Capacitors_SMD:C_0603, symbol symbols:CAP
- added J3: USB_B_Micro, Connectors:USB_Micro-B_10103594-0001LF, symbol Connector:USB_B_Micro
- added U7: USBLC6-2SC6, TO_SOT_Packages_SMD:SOT-23-6, symbol Power_Protection:USBLC6-2SC6
- C75: value 10u -> 2.2u; footprint lib:SMD0805 -> Capacitors_SMD:C_0603; symbol CAP -> symbols:CAP
- C76: footprint lib:SMD0402 -> Capacitors_SMD:C_0402; symbol CAP -> symbols:CAP
- FB1, FB2: footprint lib:SMD0805 -> Inductors_SMD:L_0805; symbol FB -> symbols:FB
- TP1: footprint lib:TP_HOLE -> Wire_Pads:SolderWirePad_single_1mmDrill; symbol TP -> symbols:TP
Connections:
- net labels removed: +3V, +5VA, AGND_IN, AGND_OUT, GND
- wire segments 118 -> 61
Other:
- note removed: "DNP"

Commit message: Schematic roughly complete
Parts:
- added J2: Conn_01x08, Pin_Headers:Pin_Header_Straight_1x08_Pitch1.27mm, symbol Connector_Generic:Conn_01x08
- renumbered C30 to C1, C75 to C2, C76 to C3, J3 to J1, U7 to U1
Connections:
- net labels added: HP_LN, HP_LP, HP_RN, HP_RP, MIC0, MIC1
- wire segments 61 -> 74
Changed lines of the file:
@@
 Floating for USB device
 $Comp
-L symbols:USB_5V #PWR06
+L symbols:USB_5V #PWR05
 U 1 1 5350403E
 P 3950 4600
-F 0 "#PWR06" H 3950 4560 30  0001 C CNN
+F 0 "#PWR05" H 3950 4560 30  0001 C CNN
 F 1 "USB_5V" H 3950 4710 30  0000 C CNN
 F 2 "~" H 3950 4600 60  0000 C CNN
@@
 $EndComp
 Wire Wire Line
-	6500 4700 6700 4700
-Wire Wire Line
 	3350 6750 3350 6650
 Wire Wire Line
 	7400 5200 6500 5200
 Wire Wire Line
-	6800 4800 6500 4800
-Wire Wire Line
-	6500 4900 6900 4900
-Wire Wire Line
 	4100 950  4600 950
 $Comp
-L power:GNDD #PWR04
+L power:GNDD #PWR02
 U 1 1 57D4EA5B
 P 3350 7150
-F 0 "#PWR04" H 3350 6900 50  0001 C CNN
+F 0 "#PWR02" H 3350 6900 50  0001 C CNN
 F 1 "GNDD" H 3350 7000 50  0000 C CNN
 F 2 "" H 3350 7150 50  0000 C CNN
@@
 	3350 7150 3350 7050
 $Comp
-L symbols:CAP C75
+L symbols:CAP C2
 U 1 1 57D66AF8
 P 3400 4850
-F 0 "C75" H 3420 4820 50  0000 L TNN
+F 0 "C2" H 3420 4820 50  0000 L TNN
 F 1 "2.2u" H 3425 4870 30  0000 L BNN
 F 2 "Capacitors_SMD:C_0603" H 3400 4850 60  0001 C CNN
@@
 Connection ~ 3400 4700
 $Comp
-L power:GNDD #PWR05
+L power:GNDD #PWR03
 U 1 1 57D676D1
 P 3400 5150
-F 0 "#PWR05" H 3400 4900 50  0001 C CNN
+F 0 "#PWR03" H 3400 4900 50  0001 C CNN
 F 1 "GNDD" H 3400 5000 50  0000 C CNN
 F 2 "" H 3400 5150 50  0000 C CNN
@@
 	3400 4950 3400 5050
 $Comp
-L symbols:CAP C76
+L symbols:CAP C3
 U 1 1 57D6798C
 P 3850 4850
-F 0 "C76" H 3870 4820 50  0000 L TNN
+F 0 "C3" H 3870 4820 50  0000 L TNN
 F 1 "0.1u" H 3875 4870 30  0000 L BNN
 F 2 "Capacitors_SMD:C_0402" H 3850 4850 60  0001 C CNN
@@
 	4100 2700 4100 950
 $Comp
-L Connector:USB_B_Micro J3
+L Connector:USB_B_Micro J1
 U 1 1 5C51D316
 P 800 5800
-F 0 "J3" H 855 6267 50  0000 C CNN
+F 0 "J1" H 855 6267 50  0000 C CNN
 F 1 "USB_B_Micro" H 855 6176 50  0000 C CNN
 F 2 "Connectors:USB_Micro-B_10103594-0001LF" H 950 5750 50  0001 C CNN
@@
 	1250 5900 1250 5850
 $Comp
-L symbols:CAP C30
+L symbols:CAP C1
 U 1 1 5C59A595
 P 700 6400
-F 0 "C30" H 720 6370 50  0000 L TNN
+F 0 "C1" H 720 6370 50  0000 L TNN
 F 1 "2.2u" H 725 6420 30  0000 L BNN
 F 2 "Capacitors_SMD:C_0603" H 700 6400 60  0001 C CNN
@@
 	700  6500 700  6600
 $Comp
-L power:GNDD #PWR0143
+L power:GNDD #PWR01
 U 1 1 5C59BE8E
 P 700 6600
-F 0 "#PWR0143" H 700 6350 50  0001 C CNN
+F 0 "#PWR01" H 700 6350 50  0001 C CNN
 F 1 "GNDD" H 700 6450 50  0000 C CNN
 F 2 "" H 700 6600 50  0000 C CNN
@@
 $EndComp
 $Comp
-L Power_Protection:USBLC6-2SC6 U7
+L Power_Protection:USBLC6-2SC6 U1
 U 1 1 5C59C6CB
 P 2200 5750
-F 0 "U7" H 2200 6428 50  0000 C CNN
+F 0 "U1" H 2200 6428 50  0000 C CNN
 F 1 "USBLC6-2SC6" H 2200 6337 50  0000 C CNN
 F 2 "TO_SOT_Packages_SMD:SOT-23-6" H 1450 6150 50  0001 C CNN
@@
 Wire Wire Line
 	3400 5800 3400 6150
+Text Label 4500 3650 2    50   ~ 0
+MIC0
+Text Label 4500 3850 2    50   ~ 0
+MIC1
+$Comp
+L power:GNDD #PWR04
+U 1 1 5C51DAE2
+P 3700 4100
+F 0 "#PWR04" H 3700 3850 50  0001 C CNN
+F 1 "GNDD" H 3700 3950 50  0000 C CNN
+F 2 "" H 3700 4100 50  0000 C CNN
+F 3 "" H 3700 4100 50  0000 C CNN
+	1    3700 4100
+	-1   0    0    -1
+$EndComp
+Text Label 4500 4050 2    50   ~ 0
+HP_LP
+Text Label 4500 4150 2    50   ~ 0
+HP_LN
+Wire Wire Line
+	3700 3750 3700 3950
+Connection ~ 3700 3950
+Wire Wire Line
+	3700 3950 3700 4100
+Text Label 4500 4250 2    50   ~ 0
+HP_RP
+Text Label 4500 4350 2    50   ~ 0
+HP_RN
+$Comp
+L Connector_Generic:Conn_01x08 J2
+U 1 1 5C524BA8
+P 4850 3950
+F 0 "J2" H 4930 3942 50  0000 L CNN
+F 1 "Conn_01x08" H 4930 3851 50  0000 L CNN
+F 2 "Pin_Headers:Pin_Header_Straight_1x08_Pitch1.27mm" H 4850 3950 50  0001 C CNN
+F 3 "~" H 4850 3950 50  0001 C CNN
+	1    4850 3950
+	1    0    0    -1
+$EndComp
+Wire Wire Line
+	4500 3650 4650 3650
+Wire Wire Line
+	4500 3850 4650 3850
+Wire Wire Line
+	3700 3750 4650 3750
+Wire Wire Line
+	3700 3950 4650 3950
+Wire Wire Line
+	4500 4050 4650 4050
+Wire Wire Line
+	4500 4150 4650 4150
+Wire Wire Line
+	4500 4250 4650 4250
+Wire Wire Line
+	4500 4350 4650 4350
+Text Label 6950 4700 0    50   ~ 0
+HP_LP
+Text Label 6950 4800 0    50   ~ 0
+HP_LN
+Text Label 6950 4900 0    50   ~ 0
+HP_RP
+Text Label 6950 5000 0    50   ~ 0
+HP_RN
+Wire Wire Line
+	6500 4700 6950 4700
+Wire Wire Line
+	6500 4800 6950 4800
+Wire Wire Line
+	6500 4900 6950 4900
+Wire Wire Line
+	6950 5000 6500 5000
+Text Label 4800 4700 2    50   ~ 0
+MIC0
+Wire Wire Line
+	4800 4700 5200 4700
+Text Label 4800 4800 2    50   ~ 0
+MIC1
+Wire Wire Line
+	4800 4800 5200 4800
 $EndSCHEMATC

Commit message: Placement!
Changed lines of the file:
@@
 EESchema Schematic File Version 4
 LIBS:audio_iface_rev2-cache
-EELAYER 26 0
+EELAYER 29 0
 EELAYER END
 $Descr A 11000 8500
@@
 F0 "Microcontroller" 50
 F1 "micro.sch" 50
-F2 "USB_D+" B L 5200 5700 60
-F3 "USB_D-" B L 5200 5800 60
+F2 "USB_D_P" B L 5200 5700 60
+F3 "USB_D_N" B L 5200 5800 60
 F4 "USB_ID" B L 5200 5900 50
 F5 "USB_VBUS" B L 5200 5600 50
@@
 	1    0    0    -1
 $EndComp
-$Comp
-L Power_Protection:USBLC6-2SC6 U1
-U 1 1 5C59C6CB
-P 2200 5750
-F 0 "U1" H 2200 6428 50  0000 C CNN
-F 1 "USBLC6-2SC6" H 2200 6337 50  0000 C CNN
-F 2 "TO_SOT_Packages_SMD:SOT-23-6" H 1450 6150 50  0001 C CNN
-F 3 "http://www2.st.com/resource/en/datasheet/CD00050750.pdf" H 2400 6100 50  0001 C CNN
-	1    2200 5750
-	1    0    0    -1
-$EndComp
 Wire Wire Line
 	1150 5650 1150 5800
-Wire Wire Line
-	1250 5850 1700 5850
 Wire Wire Line
 	3400 5800 5200 5800
@@
 	3500 5600 5200 5600
 Wire Wire Line
-	1700 5850 1700 5650
-Connection ~ 1700 5850
-Wire Wire Line
 	2900 5450 2900 5200
 Wire Wire Line
@@
 Wire Wire Line
 	1550 5650 1550 5400
-Wire Wire Line
-	1550 5400 2700 5400
-Wire Wire Line
-	2700 5400 2700 5650
-Connection ~ 2700 5650
-Wire Wire Line
-	2700 5650 2700 5850
-Wire Wire Line
-	3400 6150 1700 6150
-Wire Wire Line
-	1700 6150 1700 5850
 Wire Wire Line
 	3400 5800 3400 6150
@@
 	-1   0    0    -1
 $EndComp
+Text Label 4500 4150 2    50   ~ 0
+HP_LP
 Text Label 4500 4050 2    50   ~ 0
-HP_LP
-Text Label 4500 4150 2    50   ~ 0
 HP_LN
 Wire Wire Line
@@
 Wire Wire Line
 	3700 3950 3700 4100
+Text Label 4500 4350 2    50   ~ 0
+HP_RP
 Text Label 4500 4250 2    50   ~ 0
-HP_RP
-Text Label 4500 4350 2    50   ~ 0
 HP_RN
 $Comp
@@
 Wire Wire Line
 	4800 4800 5200 4800
+Wire Wire Line
+	1250 5850 1700 5850
+Wire Wire Line
+	1650 6150 1650 5650
+Wire Wire Line
+	1650 5650 1700 5650
+Wire Wire Line
+	1650 6150 3400 6150
+$Comp
+L Power_Protection:USBLC6-2SC6 U1
+U 1 1 5C59C6CB
+P 2200 5750
+F 0 "U1" H 2200 6428 50  0000 C CNN
+F 1 "USBLC6-2SC6" H 2200 6337 50  0000 C CNN
+F 2 "TO_SOT_Packages_SMD:SOT-23-6" H 1450 6150 50  0001 C CNN
+F 3 "http://www2.st.com/resource/en/datasheet/CD00050750.pdf" H 2400 6100 50  0001 C CNN
+	1    2200 5750
+	1    0    0    -1
+$EndComp
+Wire Wire Line
+	2750 5400 2750 5850
+Wire Wire Line
+	2750 5850 2700 5850
+Wire Wire Line
+	1550 5400 2750 5400
 $EndSCHEMATC

Commit message: Much more routing
Parts:
- C1, C2: footprint Capacitors_SMD:C_0603 -> Capacitor_SMD:C_0603_1608Metric_Pad1.05x0.95mm_HandSolder
- FB1, FB2: footprint Inductors_SMD:L_0805 -> Inductor_SMD:L_0805_2012Metric_Pad1.15x1.40mm_HandSolder
- J1: footprint Connectors:USB_Micro-B_10103594-0001LF -> Connector_USB:USB_Micro-B_Molex-105017-0001
- J2: footprint Pin_Headers:Pin_Header_Straight_1x08_Pitch1.27mm -> Connector_PinHeader_1.27mm:PinHeader_1x08_P1.27mm_Vertical
- U1: footprint TO_SOT_Packages_SMD:SOT-23-6 -> Package_TO_SOT_SMD:SOT-23-6
Changed lines of the file:
@@
 EESchema Schematic File Version 4
 LIBS:audio_iface_rev2-cache
-EELAYER 29 0
+EELAYER 30 0
 EELAYER END
 $Descr A 11000 8500
@@
 F 0 "FB1" H 3420 6865 50  0000 L TNN
 F 1 "BLM18PG221SN1D" H 3285 6975 30  0000 C BNN
-F 2 "Inductors_SMD:L_0805" H 3330 6920 60  0001 C CNN
+F 2 "Inductor_SMD:L_0805_2012Metric_Pad1.15x1.40mm_HandSolder" H 3330 6920 60  0001 C CNN
 F 3 "" H 3330 6920 60  0000 C CNN
 	1    3350 6900
@@
 F 0 "C2" H 3420 4820 50  0000 L TNN
 F 1 "2.2u" H 3425 4870 30  0000 L BNN
-F 2 "Capacitors_SMD:C_0603" H 3400 4850 60  0001 C CNN
+F 2 "Capacitor_SMD:C_0603_1608Metric_Pad1.05x0.95mm_HandSolder" H 3400 4850 60  0001 C CNN
 F 3 "" H 3400 4850 60  0000 C CNN
 	1    3400 4850
@@
 F 0 "FB2" H 3670 4665 50  0000 L TNN
 F 1 "BLM18PG221SN1D" H 3535 4775 30  0000 C BNN
-F 2 "Inductors_SMD:L_0805" H 3580 4720 60  0001 C CNN
+F 2 "Inductor_SMD:L_0805_2012Metric_Pad1.15x1.40mm_HandSolder" H 3580 4720 60  0001 C CNN
 F 3 "" H 3580 4720 60  0000 C CNN
 	1    3600 4700
@@
 F 0 "J1" H 855 6267 50  0000 C CNN
 F 1 "USB_B_Micro" H 855 6176 50  0000 C CNN
-F 2 "Connectors:USB_Micro-B_10103594-0001LF" H 950 5750 50  0001 C CNN
+F 2 "Connector_USB:USB_Micro-B_Molex-105017-0001" H 950 5750 50  0001 C CNN
 F 3 "~" H 950 5750 50  0001 C CNN
 	1    800  5800
@@
 F 0 "C1" H 720 6370 50  0000 L TNN
 F 1 "2.2u" H 725 6420 30  0000 L BNN
-F 2 "Capacitors_SMD:C_0603" H 700 6400 60  0001 C CNN
+F 2 "Capacitor_SMD:C_0603_1608Metric_Pad1.05x0.95mm_HandSolder" H 700 6400 60  0001 C CNN
 F 3 "" H 700 6400 60  0000 C CNN
 	1    700  6400
@@
 F 0 "J2" H 4930 3942 50  0000 L CNN
 F 1 "Conn_01x08" H 4930 3851 50  0000 L CNN
-F 2 "Pin_Headers:Pin_Header_Straight_1x08_Pitch1.27mm" H 4850 3950 50  0001 C CNN
+F 2 "Connector_PinHeader_1.27mm:PinHeader_1x08_P1.27mm_Vertical" H 4850 3950 50  0001 C CNN
 F 3 "~" H 4850 3950 50  0001 C CNN
 	1    4850 3950
@@
 F 0 "U1" H 2200 6428 50  0000 C CNN
 F 1 "USBLC6-2SC6" H 2200 6337 50  0000 C CNN
-F 2 "TO_SOT_Packages_SMD:SOT-23-6" H 1450 6150 50  0001 C CNN
+F 2 "Package_TO_SOT_SMD:SOT-23-6" H 1450 6150 50  0001 C CNN
 F 3 "http://www2.st.com/resource/en/datasheet/CD00050750.pdf" H 2400 6100 50  0001 C CNN
 	1    2200 5750

Commit message: More routing
Connections:
- net labels added: AGND
Changed lines of the file:
@@
 Text Label 4500 3850 2    50   ~ 0
 MIC1
-$Comp
-L power:GNDD #PWR04
-U 1 1 5C51DAE2
-P 3700 4100
-F 0 "#PWR04" H 3700 3850 50  0001 C CNN
-F 1 "GNDD" H 3700 3950 50  0000 C CNN
-F 2 "" H 3700 4100 50  0000 C CNN
-F 3 "" H 3700 4100 50  0000 C CNN
-	1    3700 4100
-	-1   0    0    -1
-$EndComp
 Text Label 4500 4150 2    50   ~ 0
 HP_LP
@@
 Wire Wire Line
 	1550 5400 2750 5400
+$Comp
+L symbols:AGND #PWR?
+U 1 1 5D866BD1
+P 3700 4100
+F 0 "#PWR?" H 3700 4100 40  0001 C CNN
+F 1 "AGND" H 3695 4175 50  0000 C CNN
+F 2 "" H 3700 4100 60  0000 C CNN
+F 3 "" H 3700 4100 60  0000 C CNN
+	1    3700 4100
+	1    0    0    -1
+$EndComp
 $EndSCHEMATC

Commit message: Design nearly complete. One more check.
Parts:
- added H1, H2, H3, H4: MountingHole, MountingHole:MountingHole_2.2mm_M2, symbol Mechanical:MountingHole
- C1, C2: symbol symbols:CAP -> Device:C_Small
- C3: footprint Capacitors_SMD:C_0402 -> Capacitor_SMD:C_0402_1005Metric; symbol symbols:CAP -> Device:C_Small
Changed lines of the file:
@@
 Floating for USB device
 $Comp
-L symbols:USB_5V #PWR05
+L audio_iface_rev2-rescue:USB_5V-symbols #PWR05
 U 1 1 5350403E
 P 3950 4600
@@
 	3350 7150 3350 7050
 $Comp
-L symbols:CAP C2
+L Device:C_Small C2
 U 1 1 57D66AF8
 P 3400 4850
@@
 F 3 "" H 3400 4850 60  0000 C CNN
 	1    3400 4850
-	0    1    1    0
+	1    0    0    -1
 $EndComp
 $Comp
@@
 	3400 4950 3400 5050
 $Comp
-L symbols:CAP C3
+L Device:C_Small C3
 U 1 1 57D6798C
 P 3850 4850
 F 0 "C3" H 3870 4820 50  0000 L TNN
 F 1 "0.1u" H 3875 4870 30  0000 L BNN
-F 2 "Capacitors_SMD:C_0402" H 3850 4850 60  0001 C CNN
+F 2 "Capacitor_SMD:C_0402_1005Metric" H 3850 4850 60  0001 C CNN
 F 3 "" H 3850 4850 60  0000 C CNN
 	1    3850 4850
-	0    1    1    0
+	1    0    0    -1
 $EndComp
 Wire Wire Line
@@
 	1250 5900 1250 5850
 $Comp
-L symbols:CAP C1
+L Device:C_Small C1
 U 1 1 5C59A595
 P 700 6400
@@
 F 3 "" H 700 6400 60  0000 C CNN
 	1    700  6400
-	0    1    1    0
+	1    0    0    -1
 $EndComp
 Wire Wire Line
@@
 	1550 5400 2750 5400
 $Comp
-L symbols:AGND #PWR?
+L symbols:AGND #PWR0101
 U 1 1 5D866BD1
 P 3700 4100
-F 0 "#PWR?" H 3700 4100 40  0001 C CNN
+F 0 "#PWR0101" H 3700 4100 40  0001 C CNN
 F 1 "AGND" H 3695 4175 50  0000 C CNN
 F 2 "" H 3700 4100 60  0000 C CNN
@@
 	1    0    0    -1
 $EndComp
+$Comp
+L Mechanical:MountingHole H1
+U 1 1 5D8AAD8E
+P 1150 950
+F 0 "H1" H 1250 996 50  0000 L CNN
+F 1 "MountingHole" H 1250 905 50  0000 L CNN
+F 2 "MountingHole:MountingHole_2.2mm_M2" H 1150 950 50  0001 C CNN
+F 3 "~" H 1150 950 50  0001 C CNN
+	1    1150 950
+	1    0    0    -1
+$EndComp
+$Comp
+L Mechanical:MountingHole H3
+U 1 1 5D8AB8E4
+P 2000 950
+F 0 "H3" H 2100 996 50  0000 L CNN
+F 1 "MountingHole" H 2100 905 50  0000 L CNN
+F 2 "MountingHole:MountingHole_2.2mm_M2" H 2000 950 50  0001 C CNN
+F 3 "~" H 2000 950 50  0001 C CNN
+	1    2000 950
+	1    0    0    -1
+$EndComp
+$Comp
+L Mechanical:MountingHole H2
+U 1 1 5D8ABA4E
+P 1150 1200
+F 0 "H2" H 1250 1246 50  0000 L CNN
+F 1 "MountingHole" H 1250 1155 50  0000 L CNN
+F 2 "MountingHole:MountingHole_2.2mm_M2" H 1150 1200 50  0001 C CNN
+F 3 "~" H 1150 1200 50  0001 C CNN
+	1    1150 1200
+	1    0    0    -1
+$EndComp
+$Comp
+L Mechanical:MountingHole H4
+U 1 1 5D8ABCBE
+P 2000 1200
+F 0 "H4" H 2100 1246 50  0000 L CNN
+F 1 "MountingHole" H 2100 1155 50  0000 L CNN
+F 2 "MountingHole:MountingHole_2.2mm_M2" H 2000 1200 50  0001 C CNN
+F 3 "~" H 2000 1200 50  0001 C CNN
+	1    2000 1200
+	1    0    0    -1
+$EndComp

Commit message: Changed some connectors, added files
Parts:
- J2: value Conn_01x08 -> Conn_01x07; footprint Connector_PinHeader_1.27mm:PinHeader_1x08_P1.27mm_Vertical -> Connector_JST:JST_PH_S7B-PH-K_1x07_P2.00mm_Horizontal; symbol Connector_Generic:Conn_01x08 -> Connector_Generic:Conn_01x07
Connections:
- wire segments 74 -> 72
Changed lines of the file:
@@
 Text Label 4500 3850 2    50   ~ 0
 MIC1
+Text Label 4500 4050 2    50   ~ 0
+HP_LP
+Text Label 4500 3950 2    50   ~ 0
+HP_LN
+Text Label 4500 4250 2    50   ~ 0
+HP_RP
 Text Label 4500 4150 2    50   ~ 0
-HP_LP
-Text Label 4500 4050 2    50   ~ 0
-HP_LN
-Wire Wire Line
-	3700 3750 3700 3950
-Connection ~ 3700 3950
-Wire Wire Line
-	3700 3950 3700 4100
-Text Label 4500 4350 2    50   ~ 0
-HP_RP
-Text Label 4500 4250 2    50   ~ 0
 HP_RN
 $Comp
-L Connector_Generic:Conn_01x08 J2
+L Connector_Generic:Conn_01x07 J2
 U 1 1 5C524BA8
 P 4850 3950
 F 0 "J2" H 4930 3942 50  0000 L CNN
-F 1 "Conn_01x08" H 4930 3851 50  0000 L CNN
-F 2 "Connector_PinHeader_1.27mm:PinHeader_1x08_P1.27mm_Vertical" H 4850 3950 50  0001 C CNN
+F 1 "Conn_01x07" H 4930 3851 50  0000 L CNN
+F 2 "Connector_JST:JST_PH_S7B-PH-K_1x07_P2.00mm_Horizontal" H 4850 3950 50  0001 C CNN
 F 3 "~" H 4850 3950 50  0001 C CNN
 	1    4850 3950
@@
 	3700 3750 4650 3750
 Wire Wire Line
-	3700 3950 4650 3950
+	4500 3950 4650 3950
 Wire Wire Line
 	4500 4050 4650 4050
@@
 Wire Wire Line
 	4500 4250 4650 4250
-Wire Wire Line
-	4500 4350 4650 4350
 Text Label 6950 4700 0    50   ~ 0
 HP_LP
@@
 	1    0    0    -1
 $EndComp
+Wire Wire Line
+	3700 3750 3700 4100
 $EndSCHEMATC
