File: hw/rev2/power.sch (KiCad schematic (older format))
At the start: 24 parts, among them J601 CONN_2, U601 LP2992AILD-5.0

Commit message: Lots of things: --Added RGB LED on timer outputs --Input: Moved capacitively coupled feedback nodes from vgnd to gnd --Output: LTC6242 for filtering to amplifier --Power: 2-stage supply for analog: USB 5V boost to 6V, LDO to 5V   Digital still using LDO from USB 5V and not caring about anyone   Bonus! Can completely shut off analog portion of board --Layout and routing: All of it TODO: final checks on layout and LVS (vs simulation) HEAD2HEAD2HEAD! TODO: adjust silkscreen, add logo TODO: debate adding 12.288MHz dedicated crystal
Parts:
- removed R601: 22k, ~, symbol RES
- removed TP601: TP_5VEN, ~, symbol TP
- removed U?: TPS61252, symbol TPS61252
- added R29: 0R, ~, symbol RES
- added U5: TPS61252, ~, symbol TPS61252
- C42: renamed from C601; value 10u 16V -> 2.2u
- C43: renamed from C602; value 2.2u 16V -> 10u
- gave numbers to parts that had none: 10
- renumbered C603 to C41, C604 to C45, C605 to C46, C606 to C47, C607 to C48, C608 to C49, C609 to C50, J601 to J9, U601 to U6
Connections:
- net labels added: USB_5V
Other:
- note added: "DNP for external supply"

Commit message: Rev 2a sent off for manufacturing: Slot added instead of drill hole at audio IO end Drill added near center Fixed huge error in HP amp schematic/layout Got rid of more labels Got rid of redundant UART port. Not sure how that happened twice... Got rid of DC blocking before CODEC inputs
Parts:
- added TP5, TP6: TP, ~, symbol TP
- L1: value 1.5u -> MLZ2012A1R5WT000
Connections:
- wire segments 67 -> 68
Changed lines of the file:
@@
 Sheet 5 6
 Title ""
-Date "6 may 2014"
-Rev "2a"
+Date "29 jun 2014"
+Rev "2b"
 Comp ""
 Comment1 ""
@@
 P 3900 2150
 F 0 "L1" H 3970 2115 50  0000 L TNN
-F 1 "1.5u" H 3900 2205 30  0000 C BNN
+F 1 "MLZ2012A1R5WT000" H 3900 2205 30  0000 C BNN
 F 2 "~" H 3900 2150 60  0000 C CNN
 F 3 "~" H 3900 2150 60  0000 C CNN
@@
 	6350 4450 6900 4450
 Wire Wire Line
-	7800 4350 7800 4250
+	7800 4050 7800 4350
 Wire Wire Line
 	7500 4250 8400 4250
@@
 	10150 5150 10150 5400
 Connection ~ 9800 5150
+$Comp
+L TP TP5
+U 1 1 53AF6D72
+P 7800 3950
+F 0 "TP5" H 7800 3850 60  0000 C CNN
+F 1 "TP" H 7800 4050 60  0000 C CNN
+F 2 "~" H 7800 3950 60  0000 C CNN
+F 3 "~" H 7800 3950 60  0000 C CNN
+	1    7800 3950
+	0    -1   -1   0
+$EndComp
+$Comp
+L TP TP6
+U 1 1 53AF7518
+P 6550 3950
+F 0 "TP6" H 6550 3850 60  0000 C CNN
+F 1 "TP" H 6550 4050 60  0000 C CNN
+F 2 "~" H 6550 3950 60  0000 C CNN
+F 3 "~" H 6550 3950 60  0000 C CNN
+	1    6550 3950
+	0    -1   -1   0
+$EndComp
+Wire Wire Line
+	6550 4050 6550 4250
+Connection ~ 6550 4250
 $EndSCHEMATC

Commit message: Started board upgrade to 4 layers and better signal isolation
Parts:
- removed J9: CONN_2, ~, symbol CONN_2
- added J9: CONN_01X02, lib:HDR_2X1_50MIL, symbol CONN_01X02
- C37: footprint ~ -> lib:SMD1206_POL
- C38, C39, C40, C41, C42, C44, C45, C46, C47, R25, R26, R27, R28, R29: footprint ~ -> lib:SMD0402
- C43, C49, L1: footprint ~ -> lib:SMD0805
- C48: footprint ~ -> lib:SMD0603
- C50: footprint ~ -> lib:SMD1411_POL
- TP5, TP6: footprint ~ -> lib:TP_HOLE
- U5: footprint ~ -> lib:TPS61252_QFN8
- U6: footprint ~ -> lib:TI_WSON6
Connections:
- net labels added: GNDD
- net labels removed: DGND
- wire segments 68 -> 70

Commit message: Routed out 4-layer variant--now need to do silkscreens and such
Parts:
- added TP7: TP, lib:TP_HOLE, symbol TP
Connections:
- wire segments 70 -> 71
Changed lines of the file:
@@
 Connection ~ 6800 4950
 Wire Wire Line
-	6000 4950 8400 4950
+	6000 4950 8800 4950
 Wire Wire Line
 	4100 1200 4100 1600
@@
 Wire Wire Line
 	1750 2950 2950 2950
+$Comp
+L TP TP7
+U 1 1 57EB7321
+P 8800 4400
+F 0 "TP7" H 8800 4300 60  0000 C CNN
+F 1 "TP" H 8800 4500 60  0000 C CNN
+F 2 "lib:TP_HOLE" H 8800 4400 60  0001 C CNN
+F 3 "~" H 8800 4400 60  0000 C CNN
+	1    8800 4400
+	0    -1   -1   0
+$EndComp
+Wire Wire Line
+	8800 4950 8800 4500
+Connection ~ 8400 4950
 $EndSCHEMATC

Commit message: More routing
Parts:
- added TP12: TP, lib:TP_HOLE, symbol TP
Connections:
- wire segments 71 -> 72
Changed lines of the file:
@@
 $EndDescr
 $Comp
-L AGND_IN #PWR045
+L AGND_IN #PWR56
 U 1 1 524EE50E
 P 9000 5400
-F 0 "#PWR045" H 9000 5400 40  0001 C CNN
+F 0 "#PWR56" H 9000 5400 40  0001 C CNN
 F 1 "AGND_IN" H 9000 5330 50  0000 C CNN
 F 2 "~" H 9000 5400 60  0000 C CNN
@@
 $EndComp
 $Comp
-L AGND_OUT #PWR046
+L AGND_OUT #PWR58
 U 1 1 524EE514
 P 9800 5400
-F 0 "#PWR046" H 9800 5400 40  0001 C CNN
+F 0 "#PWR58" H 9800 5400 40  0001 C CNN
 F 1 "AGND_OUT" H 9800 5330 50  0000 C CNN
 F 2 "~" H 9800 5400 60  0000 C CNN
@@
 $EndComp
 $Comp
-L +5VA #PWR047
+L +5VA #PWR55
 U 1 1 524F286A
 P 8400 4150
-F 0 "#PWR047" H 8400 4280 20  0001 C CNN
+F 0 "#PWR55" H 8400 4280 20  0001 C CNN
 F 1 "+5VA" H 8400 4250 30  0000 C CNN
 F 2 "" H 8400 4150 60  0000 C CNN
@@
 $EndComp
 $Comp
-L GND #PWR048
+L GND #PWR52
 U 1 1 53512E5E
 P 4000 2750
-F 0 "#PWR048" H 4000 2750 30  0001 C CNN
+F 0 "#PWR52" H 4000 2750 30  0001 C CNN
 F 1 "GND" H 4000 2680 30  0001 C CNN
 F 2 "" H 4000 2750 60  0000 C CNN
@@
 $EndComp
 $Comp
-L GND #PWR049
+L GND #PWR51
 U 1 1 53513050
 P 2300 3000
-F 0 "#PWR049" H 2300 3000 30  0001 C CNN
+F 0 "#PWR51" H 2300 3000 30  0001 C CNN
 F 1 "GND" H 2300 2930 30  0001 C CNN
 F 2 "" H 2300 3000 60  0000 C CNN
@@
 $EndComp
 $Comp
-L +6V #PWR050
+L +6V #PWR50
 U 1 1 5351D85D
 P 1900 2150
-F 0 "#PWR050" H 1900 2110 30  0001 C CNN
+F 0 "#PWR50" H 1900 2110 30  0001 C CNN
 F 1 "+6V" H 1900 2260 30  0000 C CNN
 F 2 "~" H 1900 2150 60  0000 C CNN
@@
 $EndComp
 $Comp
-L +6V #PWR051
+L +6V #PWR53
 U 1 1 5351DA70
 P 5800 4200
-F 0 "#PWR051" H 5800 4160 30  0001 C CNN
+F 0 "#PWR53" H 5800 4160 30  0001 C CNN
 F 1 "+6V" H 5800 4310 30  0000 C CNN
 F 2 "~" H 5800 4200 60  0000 C CNN
@@
 $EndComp
 $Comp
-L USB_5V #PWR052
+L USB_5V #PWR49
 U 1 1 5357BECD
 P 1150 1050
-F 0 "#PWR052" H 1150 1010 30  0001 C CNN
+F 0 "#PWR49" H 1150 1010 30  0001 C CNN
 F 1 "USB_5V" H 1150 1160 30  0000 C CNN
 F 2 "~" H 1150 1050 60  0000 C CNN
@@
 Connection ~ 6800 4950
 Wire Wire Line
-	6000 4950 8800 4950
+	6000 4950 9200 4950
 Wire Wire Line
 	4100 1200 4100 1600
@@
 	6800 4350 6900 4350
 $Comp
-L GND #PWR053
+L GND #PWR59
 U 1 1 535D962B
 P 10150 5400
-F 0 "#PWR053" H 10150 5400 30  0001 C CNN
+F 0 "#PWR59" H 10150 5400 30  0001 C CNN
 F 1 "GND" H 10150 5330 30  0001 C CNN
 F 2 "" H 10150 5400 60  0000 C CNN
@@
 	1150 1200 4100 1200
 $Comp
-L GNDD #PWR054
+L GNDD #PWR57
 U 1 1 57D6373F
 P 9400 5400
-F 0 "#PWR054" H 9400 5150 50  0001 C CNN
+F 0 "#PWR57" H 9400 5150 50  0001 C CNN
 F 1 "GNDD" H 9400 5250 50  0000 C CNN
 F 2 "" H 9400 5400 50  0000 C CNN
@@
 $EndComp
 $Comp
-L GNDD #PWR055
+L GNDD #PWR54
 U 1 1 57D65DAE
 P 6550 5100
-F 0 "#PWR055" H 6550 4850 50  0001 C CNN
+F 0 "#PWR54" H 6550 4850 50  0001 C CNN
 F 1 "GNDD" H 6550 4950 50  0000 C CNN
 F 2 "" H 6550 5100 50  0000 C CNN
@@
 	8800 4950 8800 4500
 Connection ~ 8400 4950
+$Comp
+L TP TP12
+U 1 1 57EC7546
+P 9200 4400
+F 0 "TP12" H 9200 4300 60  0000 C CNN
+F 1 "TP" H 9200 4500 60  0000 C CNN
+F 2 "lib:TP_HOLE" H 9200 4400 60  0001 C CNN
+F 3 "~" H 9200 4400 60  0000 C CNN
+	1    9200 4400
+	0    -1   -1   0
+$EndComp
+Wire Wire Line
+	9200 4950 9200 4500
+Connection ~ 8800 4950
 $EndSCHEMATC
