File: hw/rev2/power.sch (KiCad schematic (older format))
At the start: 31 parts, among them J9 CONN_01X02, U5 TPS61252, U6 LP2992AILD-5.0, U9 FAN536xx

Commit message: Fixed power connections for S70--submitted PCB
Parts:
- C42: footprint lib:SMD0402 -> lib:SMD0603
- C48: footprint lib:SMD0603 -> lib:SMD0402
- FB5, FB6: footprint lib:SMD0805 -> lib:SMD0603
Changed lines of the file:
@@
 LIBS:contrib
 LIBS:valves
+LIBS:audio_iface_rev2-cache
 EELAYER 25 0
 EELAYER END
@@
 F 0 "C42" H 4870 2270 50  0000 L TNN
 F 1 "2.2u" H 4875 2320 30  0000 L BNN
-F 2 "lib:SMD0402" H 4850 2300 60  0001 C CNN
+F 2 "lib:SMD0603" H 4850 2300 60  0001 C CNN
 F 3 "~" H 4850 2300 60  0000 C CNN
 	1    4850 2300
@@
 F 0 "C48" H 8120 4420 50  0000 L TNN
 F 1 "0.1u 6.3V" H 8125 4470 30  0000 L BNN
-F 2 "lib:SMD0603" H 8100 4450 60  0001 C CNN
+F 2 "lib:SMD0402" H 8100 4450 60  0001 C CNN
 F 3 "~" H 8100 4450 60  0000 C CNN
 	1    8100 4450
@@
 F 0 "FB5" H 9270 5465 50  0000 L TNN
 F 1 "BLM18PG221SN1D" H 9135 5575 30  0000 C BNN
-F 2 "lib:SMD0805" H 9180 5520 60  0001 C CNN
+F 2 "lib:SMD0603" H 9180 5520 60  0001 C CNN
 F 3 "" H 9180 5520 60  0000 C CNN
 	1    9200 5500
@@
 F 0 "FB6" H 10020 5465 50  0000 L TNN
 F 1 "BLM18PG221SN1D" H 9885 5575 30  0000 C BNN
-F 2 "lib:SMD0805" H 9930 5520 60  0001 C CNN
+F 2 "lib:SMD0603" H 9930 5520 60  0001 C CNN
 F 3 "" H 9930 5520 60  0000 C CNN
 	1    9950 5500

Commit message: Modified feedback values on PCB
Parts:
- R25: value RES -> 100k
- R26: value RES -> 22k
Changed lines of the file:
@@
 $EndComp
 $Comp
-L +5VA #PWR59
+L +5VA #PWR045
 U 1 1 524F286A
 P 8400 4150
-F 0 "#PWR59" H 8400 4280 20  0001 C CNN
+F 0 "#PWR045" H 8400 4280 20  0001 C CNN
 F 1 "+5VA" H 8400 4250 30  0000 C CNN
 F 2 "" H 8400 4150 60  0000 C CNN
@@
 P 2500 2350
 F 0 "R25" H 2570 2315 50  0000 L TNN
-F 1 "RES" H 2500 2405 30  0000 C BNN
+F 1 "100k" H 2500 2405 30  0000 C BNN
 F 2 "lib:SMD0402" H 2500 2350 60  0001 C CNN
 F 3 "~" H 2500 2350 60  0000 C CNN
@@
 P 2500 2750
 F 0 "R26" H 2570 2715 50  0000 L TNN
-F 1 "RES" H 2500 2805 30  0000 C BNN
+F 1 "22k" H 2500 2805 30  0000 C BNN
 F 2 "lib:SMD0402" H 2500 2750 60  0001 C CNN
 F 3 "~" H 2500 2750 60  0000 C CNN
@@
 $EndComp
 $Comp
-L +6V #PWR52
+L +6V #PWR046
 U 1 1 5351D85D
 P 1900 2150
-F 0 "#PWR52" H 1900 2110 30  0001 C CNN
+F 0 "#PWR046" H 1900 2110 30  0001 C CNN
 F 1 "+6V" H 1900 2260 30  0000 C CNN
 F 2 "~" H 1900 2150 60  0000 C CNN
@@
 $EndComp
 $Comp
-L +6V #PWR57
+L +6V #PWR047
 U 1 1 5351DA70
 P 5800 4200
-F 0 "#PWR57" H 5800 4160 30  0001 C CNN
+F 0 "#PWR047" H 5800 4160 30  0001 C CNN
 F 1 "+6V" H 5800 4310 30  0000 C CNN
 F 2 "~" H 5800 4200 60  0000 C CNN
@@
 $EndComp
 $Comp
-L USB_5V #PWR49
+L USB_5V #PWR048
 U 1 1 5357BECD
 P 1150 1050
-F 0 "#PWR49" H 1150 1010 30  0001 C CNN
+F 0 "#PWR048" H 1150 1010 30  0001 C CNN
 F 1 "USB_5V" H 1150 1160 30  0000 C CNN
 F 2 "~" H 1150 1050 60  0000 C CNN
@@
 $EndComp
 $Comp
-L USB_5V #PWR55
+L USB_5V #PWR049
 U 1 1 58249708
 P 3600 5450
-F 0 "#PWR55" H 3600 5410 30  0001 C CNN
+F 0 "#PWR049" H 3600 5410 30  0001 C CNN
 F 1 "USB_5V" H 3600 5560 30  0000 C CNN
 F 2 "~" H 3600 5450 60  0000 C CNN
@@
 Connection ~ 1700 6100
 $Comp
-L +3V #PWR50
+L +3V #PWR050
 U 1 1 58249F3F
 P 1700 5350
-F 0 "#PWR50" H 1700 5310 30  0001 C CNN
+F 0 "#PWR050" H 1700 5310 30  0001 C CNN
 F 1 "+3V" H 1700 5460 30  0000 C CNN
 F 2 "" H 1700 5350 60  0000 C CNN
@@
 Connection ~ 10150 5500
 $Comp
-L AGND_OUT #PWR62
+L AGND_OUT #PWR051
 U 1 1 582A72C1
 P 10150 5650
-F 0 "#PWR62" H 10150 5650 40  0001 C CNN
+F 0 "#PWR051" H 10150 5650 40  0001 C CNN
 F 1 "AGND_OUT" H 10150 5580 50  0000 C CNN
 F 2 "" H 10150 5650 60  0000 C CNN
@@
 $EndComp
 $Comp
-L AGND_IN #PWR60
+L AGND_IN #PWR052
 U 1 1 582A73A4
 P 8950 5650
-F 0 "#PWR60" H 8950 5650 40  0001 C CNN
+F 0 "#PWR052" H 8950 5650 40  0001 C CNN
 F 1 "AGND_IN" H 8950 5580 50  0000 C CNN
 F 2 "" H 8950 5650 60  0000 C CNN
@@
 $EndComp
 $Comp
-L PWR_FLAG #FLG1
+L PWR_FLAG #FLG053
 U 1 1 582A7458
 P 8550 5400
-F 0 "#FLG1" H 8550 5495 50  0001 C CNN
+F 0 "#FLG053" H 8550 5495 50  0001 C CNN
 F 1 "PWR_FLAG" H 8550 5580 50  0000 C CNN
 F 2 "" H 8550 5400 50  0000 C CNN
@@
 	8550 5400 8550 5500
 $Comp
-L PWR_FLAG #FLG3
+L PWR_FLAG #FLG054
 U 1 1 582A76DA
 P 10450 5350
-F 0 "#FLG3" H 10450 5445 50  0001 C CNN
+F 0 "#FLG054" H 10450 5445 50  0001 C CNN
 F 1 "PWR_FLAG" H 10450 5530 50  0000 C CNN
 F 2 "" H 10450 5350 50  0000 C CNN
@@
 	10450 5500 10450 5350
 $Comp
-L GND #PWR61
+L GND #PWR055
 U 1 1 582A7A45
 P 9500 5600
-F 0 "#PWR61" H 9500 5350 50  0001 C CNN
+F 0 "#PWR055" H 9500 5350 50  0001 C CNN
 F 1 "GND" H 9500 5450 50  0000 C CNN
 F 2 "" H 9500 5600 50  0000 C CNN
@@
 $EndComp
 $Comp
-L PWR_FLAG #FLG2
+L PWR_FLAG #FLG056
 U 1 1 582A7AB7
 P 9700 5250
-F 0 "#FLG2" H 9700 5345 50  0001 C CNN
+F 0 "#FLG056" H 9700 5345 50  0001 C CNN
 F 1 "PWR_FLAG" H 9700 5430 50  0000 C CNN
 F 2 "" H 9700 5250 50  0000 C CNN
@@
 	9500 5500 9500 5600
 $Comp
-L GND #PWR58
+L GND #PWR057
 U 1 1 582AB277
 P 6550 5100
-F 0 "#PWR58" H 6550 4850 50  0001 C CNN
+F 0 "#PWR057" H 6550 4850 50  0001 C CNN
 F 1 "GND" H 6550 4950 50  0000 C CNN
 F 2 "" H 6550 5100 50  0000 C CNN
@@
 $EndComp
 $Comp
-L GND #PWR54
+L GND #PWR058
 U 1 1 582AB382
 P 3200 6150
-F 0 "#PWR54" H 3200 5900 50  0001 C CNN
+F 0 "#PWR058" H 3200 5900 50  0001 C CNN
 F 1 "GND" H 3200 6000 50  0000 C CNN
 F 2 "" H 3200 6150 50  0000 C CNN
@@
 $EndComp
 $Comp
-L GND #PWR51
+L GND #PWR059
 U 1 1 582AB4ED
 P 1700 6150
-F 0 "#PWR51" H 1700 5900 50  0001 C CNN
+F 0 "#PWR059" H 1700 5900 50  0001 C CNN
 F 1 "GND" H 1700 6000 50  0000 C CNN
 F 2 "" H 1700 6150 50  0000 C CNN
@@
 $EndComp
 $Comp
-L GND #PWR53
+L GND #PWR060
 U 1 1 582AB638
 P 2300 3000
-F 0 "#PWR53" H 2300 2750 50  0001 C CNN
+F 0 "#PWR060" H 2300 2750 50  0001 C CNN
 F 1 "GND" H 2300 2850 50  0000 C CNN
 F 2 "" H 2300 3000 50  0000 C CNN
@@
 $EndComp
 $Comp
-L GND #PWR56
+L GND #PWR061
 U 1 1 582AB903
 P 4000 2750
-F 0 "#PWR56" H 4000 2500 50  0001 C CNN
+F 0 "#PWR061" H 4000 2500 50  0001 C CNN
 F 1 "GND" H 4000 2600 50  0000 C CNN
 F 2 "" H 4000 2750 50  0000 C CNN

Commit message: Finished schematic and layout with STM32F7
Connections:
- net labels added: +3V3
- net labels removed: +3V
Changed lines of the file:
@@
 $EndComp
 $Comp
-L +5VA #PWR59
+L +5VA #PWR047
 U 1 1 524F286A
 P 8400 4150
-F 0 "#PWR59" H 8400 4280 20  0001 C CNN
+F 0 "#PWR047" H 8400 4280 20  0001 C CNN
 F 1 "+5VA" H 8400 4250 30  0000 C CNN
 F 2 "" H 8400 4150 60  0000 C CNN
@@
 $EndComp
 $Comp
-L +6V #PWR52
+L +6V #PWR048
 U 1 1 5351D85D
 P 1900 2150
-F 0 "#PWR52" H 1900 2110 30  0001 C CNN
+F 0 "#PWR048" H 1900 2110 30  0001 C CNN
 F 1 "+6V" H 1900 2260 30  0000 C CNN
 F 2 "~" H 1900 2150 60  0000 C CNN
@@
 $EndComp
 $Comp
-L +6V #PWR57
+L +6V #PWR049
 U 1 1 5351DA70
 P 5800 4200
-F 0 "#PWR57" H 5800 4160 30  0001 C CNN
+F 0 "#PWR049" H 5800 4160 30  0001 C CNN
 F 1 "+6V" H 5800 4310 30  0000 C CNN
 F 2 "~" H 5800 4200 60  0000 C CNN
@@
 $EndComp
 $Comp
-L USB_5V #PWR49
+L USB_5V #PWR050
 U 1 1 5357BECD
 P 1150 1050
-F 0 "#PWR49" H 1150 1010 30  0001 C CNN
+F 0 "#PWR050" H 1150 1010 30  0001 C CNN
 F 1 "USB_5V" H 1150 1160 30  0000 C CNN
 F 2 "~" H 1150 1050 60  0000 C CNN
@@
 $EndComp
 $Comp
-L USB_5V #PWR55
+L USB_5V #PWR051
 U 1 1 58249708
 P 3600 5450
-F 0 "#PWR55" H 3600 5410 30  0001 C CNN
+F 0 "#PWR051" H 3600 5410 30  0001 C CNN
 F 1 "USB_5V" H 3600 5560 30  0000 C CNN
 F 2 "~" H 3600 5450 60  0000 C CNN
@@
 	1550 6100 1700 6100
 Connection ~ 1700 6100
-$Comp
-L +3V #PWR50
-U 1 1 58249F3F
-P 1700 5350
-F 0 "#PWR50" H 1700 5310 30  0001 C CNN
-F 1 "+3V" H 1700 5460 30  0000 C CNN
-F 2 "" H 1700 5350 60  0000 C CNN
-F 3 "" H 1700 5350 60  0000 C CNN
-	1    1700 5350
-	1    0    0    -1
-$EndComp
 Connection ~ 1700 5700
 $Comp
@@
 Connection ~ 10150 5500
 $Comp
-L AGND_OUT #PWR62
+L AGND_OUT #PWR052
 U 1 1 582A72C1
 P 10150 5650
-F 0 "#PWR62" H 10150 5650 40  0001 C CNN
+F 0 "#PWR052" H 10150 5650 40  0001 C CNN
 F 1 "AGND_OUT" H 10150 5580 50  0000 C CNN
 F 2 "" H 10150 5650 60  0000 C CNN
@@
 $EndComp
 $Comp
-L AGND_IN #PWR60
+L AGND_IN #PWR053
 U 1 1 582A73A4
 P 8950 5650
-F 0 "#PWR60" H 8950 5650 40  0001 C CNN
+F 0 "#PWR053" H 8950 5650 40  0001 C CNN
 F 1 "AGND_IN" H 8950 5580 50  0000 C CNN
 F 2 "" H 8950 5650 60  0000 C CNN
@@
 $EndComp
 $Comp
-L PWR_FLAG #FLG1
+L PWR_FLAG #FLG054
 U 1 1 582A7458
 P 8550 5400
-F 0 "#FLG1" H 8550 5495 50  0001 C CNN
+F 0 "#FLG054" H 8550 5495 50  0001 C CNN
 F 1 "PWR_FLAG" H 8550 5580 50  0000 C CNN
 F 2 "" H 8550 5400 50  0000 C CNN
@@
 	8550 5400 8550 5500
 $Comp
-L PWR_FLAG #FLG3
+L PWR_FLAG #FLG055
 U 1 1 582A76DA
 P 10450 5350
-F 0 "#FLG3" H 10450 5445 50  0001 C CNN
+F 0 "#FLG055" H 10450 5445 50  0001 C CNN
 F 1 "PWR_FLAG" H 10450 5530 50  0000 C CNN
 F 2 "" H 10450 5350 50  0000 C CNN
@@
 	10450 5500 10450 5350
 $Comp
-L GND #PWR61
+L GND #PWR056
 U 1 1 582A7A45
 P 9500 5600
-F 0 "#PWR61" H 9500 5350 50  0001 C CNN
+F 0 "#PWR056" H 9500 5350 50  0001 C CNN
 F 1 "GND" H 9500 5450 50  0000 C CNN
 F 2 "" H 9500 5600 50  0000 C CNN
@@
 $EndComp
 $Comp
-L PWR_FLAG #FLG2
+L PWR_FLAG #FLG057
 U 1 1 582A7AB7
 P 9700 5250
-F 0 "#FLG2" H 9700 5345 50  0001 C CNN
+F 0 "#FLG057" H 9700 5345 50  0001 C CNN
 F 1 "PWR_FLAG" H 9700 5430 50  0000 C CNN
 F 2 "" H 9700 5250 50  0000 C CNN
@@
 	9500 5500 9500 5600
 $Comp
-L GND #PWR58
+L GND #PWR058
 U 1 1 582AB277
 P 6550 5100
-F 0 "#PWR58" H 6550 4850 50  0001 C CNN
+F 0 "#PWR058" H 6550 4850 50  0001 C CNN
 F 1 "GND" H 6550 4950 50  0000 C CNN
 F 2 "" H 6550 5100 50  0000 C CNN
@@
 $EndComp
 $Comp
-L GND #PWR54
+L GND #PWR059
 U 1 1 582AB382
 P 3200 6150
-F 0 "#PWR54" H 3200 5900 50  0001 C CNN
+F 0 "#PWR059" H 3200 5900 50  0001 C CNN
 F 1 "GND" H 3200 6000 50  0000 C CNN
 F 2 "" H 3200 6150 50  0000 C CNN
@@
 $EndComp
 $Comp
-L GND #PWR51
+L GND #PWR060
 U 1 1 582AB4ED
 P 1700 6150
-F 0 "#PWR51" H 1700 5900 50  0001 C CNN
+F 0 "#PWR060" H 1700 5900 50  0001 C CNN
 F 1 "GND" H 1700 6000 50  0000 C CNN
 F 2 "" H 1700 6150 50  0000 C CNN
@@
 $EndComp
 $Comp
-L GND #PWR53
+L GND #PWR061
 U 1 1 582AB638
 P 2300 3000
-F 0 "#PWR53" H 2300 2750 50  0001 C CNN
+F 0 "#PWR061" H 2300 2750 50  0001 C CNN
 F 1 "GND" H 2300 2850 50  0000 C CNN
 F 2 "" H 2300 3000 50  0000 C CNN
@@
 $EndComp
 $Comp
-L GND #PWR56
+L GND #PWR062
 U 1 1 582AB903
 P 4000 2750
-F 0 "#PWR56" H 4000 2500 50  0001 C CNN
+F 0 "#PWR062" H 4000 2500 50  0001 C CNN
 F 1 "GND" H 4000 2600 50  0000 C CNN
 F 2 "" H 4000 2750 50  0000 C CNN
@@
 Wire Wire Line
 	7500 4250 8400 4250
+$Comp
+L +3V3 #PWR063
+U 1 1 58CFA9D7
+P 1700 5350
+F 0 "#PWR063" H 1700 5200 50  0001 C CNN
+F 1 "+3V3" H 1700 5490 50  0000 C CNN
+F 2 "" H 1700 5350 50  0000 C CNN
+F 3 "" H 1700 5350 50  0000 C CNN
+	1    1700 5350
+	1    0    0    -1
+$EndComp
 $EndSCHEMATC
