File: hw/rev2/power.sch (KiCad schematic (older format))
At the start: 27 parts, among them J9 CONN_01X02, U5 TPS61252, U6 LP2992AILD-5.0

Commit message: Most of a schematic
Parts:
- removed C37: 22u, lib:SMD1206_POL, symbol CPOL
- removed C38: 100n, lib:SMD0402, symbol CAP
- removed C39, C44: 10n, lib:SMD0402, symbol CAP
- removed C40: 100p, lib:SMD0402, symbol CAP
- removed C41, C45: 10n 16V, lib:SMD0402, symbol CAP
- removed C42: 2.2u, lib:SMD0402, symbol CAP
- removed C43: 10u, lib:SMD0805, symbol CAP
- removed C46: 10n 6.3V, lib:SMD0402, symbol CAP
- removed C47: 0.1u 6.3V, lib:SMD0402, symbol CAP
- removed C48: 0.1u 6.3V, lib:SMD0603, symbol CAP
- removed C49: 10u 6.3V, lib:SMD0805, symbol CPOL
- removed C50: 100u 6.3V, lib:SMD1411_POL, symbol CPOL
- removed J9: CONN_01X02, lib:HDR_2X1_50MIL, symbol CONN_01X02
- removed L1: MLZ2012A1R5WT000, lib:SMD0805, symbol IND
- removed R25, R26: RES, lib:SMD0402, symbol RES
- removed R27: 20k, lib:SMD0402, symbol RES
- removed R28: 1Meg, lib:SMD0402, symbol RES
- removed R29: 0R, lib:SMD0402, symbol RES
- removed TP12, TP5, TP7: TP, lib:TP_HOLE, symbol TP
- removed U5: TPS61252, lib:TPS61252_QFN8, symbol TPS61252
- removed U6: LP2992AILD-5.0, lib:TI_WSON6, symbol LP2992_WSON
- added C21, C23, C24, C26, C27, C29: 2.2u, Capacitors_SMD:C_0603, symbol symbols:CAP
- added C22, C25, C28: 10u, Capacitors_SMD:C_0805, symbol symbols:CAP
- added J2: Screw_Terminal_01x02, TerminalBlocks_Phoenix:TerminalBlock_Phoenix_MPT-2.54mm_2pol, symbol Connector:Screw_Terminal_01x02
- added R8: 100k, Resistors_SMD:R_0402, symbol symbols:RES
- added R9: 0R, Resistors_SMD:R_0402, symbol symbols:RES
- added TP8, TP9: TP, Wire_Pads:SolderWirePad_single_1mmDrill, symbol symbols:TP
- added U4, U6: LP5907MFX-3.3, TO_SOT_Packages_SMD:SOT-23-5, symbol symbols:LP5907MFX-3.3
- added U5: LP5907MFX-1.8, TO_SOT_Packages_SMD:SOT-23-5, symbol Regulator_Linear:LP5907MFX-1.8
- TP7: renamed from TP6; footprint lib:TP_HOLE -> Wire_Pads:SolderWirePad_single_1mmDrill; symbol TP -> symbols:TP
Connections:
- net labels added: +1V8, +3V3, +3V3A, +5V, GNDA
- net labels removed: +5VA, +6V, AGND_IN, AGND_OUT
- wire segments 72 -> 74
Other:
- note removed: "DNP for external supply"
- note removed: "Join nets once layout is complete"

Commit message: Schematic roughly complete
Parts:
- renumbered C21 to C32, C22 to C33, C23 to C34, C24 to C35, C25 to C36, C26 to C37, C27 to C38, C28 to C39, C29 to C40, J2 to J4, R8 to R11, R9 to R12, U4 to U5, U5 to U6, U6 to U7
Changed lines of the file:
@@
 $EndComp
 $Comp
-L power:GNDD #PWR056
+L power:GNDD #PWR042
 U 1 1 57D6373F
 P 5100 5000
-F 0 "#PWR056" H 5100 4750 50  0001 C CNN
+F 0 "#PWR042" H 5100 4750 50  0001 C CNN
 F 1 "GNDD" H 5100 4850 50  0000 C CNN
 F 2 "" H 5100 5000 50  0000 C CNN
@@
 $EndComp
 $Comp
-L Connector:Screw_Terminal_01x02 J2
+L Connector:Screw_Terminal_01x02 J4
 U 1 1 5C6534CB
 P 3200 3000
-F 0 "J2" H 3280 2992 50  0000 L CNN
+F 0 "J4" H 3280 2992 50  0000 L CNN
 F 1 "Screw_Terminal_01x02" H 3280 2901 50  0000 L CNN
 F 2 "TerminalBlocks_Phoenix:TerminalBlock_Phoenix_MPT-2.54mm_2pol" H 3200 3000 50  0001 C CNN
@@
 $EndComp
 $Comp
-L power:+1V8 #PWR0127
+L power:+1V8 #PWR046
 U 1 1 5C663EE9
 P 7050 2700
-F 0 "#PWR0127" H 7050 2550 50  0001 C CNN
+F 0 "#PWR046" H 7050 2550 50  0001 C CNN
 F 1 "+1V8" H 7065 2873 50  0000 C CNN
 F 2 "" H 7050 2700 50  0001 C CNN
@@
 $EndComp
 $Comp
-L symbols:+3V3A #PWR0128
+L symbols:+3V3A #PWR040
 U 1 1 5C663FB0
 P 2900 5150
-F 0 "#PWR0128" H 2900 5000 50  0001 C CNN
+F 0 "#PWR040" H 2900 5000 50  0001 C CNN
 F 1 "+3V3A" H 2915 5323 50  0000 C CNN
 F 2 "" H 2900 5150 50  0001 C CNN
@@
 $EndComp
 $Comp
-L power:+3V3 #PWR0129
+L power:+3V3 #PWR050
 U 1 1 5C664069
 P 8650 4650
-F 0 "#PWR0129" H 8650 4500 50  0001 C CNN
+F 0 "#PWR050" H 8650 4500 50  0001 C CNN
 F 1 "+3V3" H 8665 4823 50  0000 C CNN
 F 2 "" H 8650 4650 50  0001 C CNN
@@
 $EndComp
 $Comp
-L Regulator_Linear:LP5907MFX-1.8 U5
+L Regulator_Linear:LP5907MFX-1.8 U6
 U 1 1 5C669DA9
 P 6450 3100
-F 0 "U5" H 6450 3467 50  0000 C CNN
+F 0 "U6" H 6450 3467 50  0000 C CNN
 F 1 "LP5907MFX-1.8" H 6450 3376 50  0000 C CNN
 F 2 "TO_SOT_Packages_SMD:SOT-23-5" H 6450 3450 50  0001 C CNN
@@
 $EndComp
 $Comp
-L symbols:LP5907MFX-3.3 U4
+L symbols:LP5907MFX-3.3 U5
 U 1 1 5C66F71D
 P 2250 5550
-F 0 "U4" H 2250 5917 50  0000 C CNN
+F 0 "U5" H 2250 5917 50  0000 C CNN
 F 1 "LP5907MFX-3.3" H 2250 5826 50  0000 C CNN
 F 2 "TO_SOT_Packages_SMD:SOT-23-5" H 2250 5900 50  0001 C CNN
@@
 $EndComp
 $Comp
-L symbols:LP5907MFX-3.3 U6
+L symbols:LP5907MFX-3.3 U7
 U 1 1 5C66F7B3
 P 8050 5050
-F 0 "U6" H 8050 5417 50  0000 C CNN
+F 0 "U7" H 8050 5417 50  0000 C CNN
 F 1 "LP5907MFX-3.3" H 8050 5326 50  0000 C CNN
 F 2 "TO_SOT_Packages_SMD:SOT-23-5" H 8050 5400 50  0001 C CNN
@@
 	2900 5450 2700 5450
 $Comp
-L symbols:CAP C22
+L symbols:CAP C33
 U 1 1 5C676BB9
 P 2700 5650
-F 0 "C22" H 2720 5620 50  0000 L TNN
+F 0 "C33" H 2720 5620 50  0000 L TNN
 F 1 "10u" H 2725 5670 30  0000 L BNN
 F 2 "Capacitors_SMD:C_0805" H 2700 5650 60  0001 C CNN
@@
 $EndComp
 $Comp
-L symbols:CAP C23
+L symbols:CAP C34
 U 1 1 5C676C4D
 P 2900 5650
-F 0 "C23" H 2920 5620 50  0000 L TNN
+F 0 "C34" H 2920 5620 50  0000 L TNN
 F 1 "2.2u" H 2925 5670 30  0000 L BNN
 F 2 "Capacitors_SMD:C_0603" H 2900 5650 60  0001 C CNN
@@
 	2700 5450 2550 5450
 $Comp
-L symbols:CAP C28
+L symbols:CAP C39
 U 1 1 5C681F57
 P 8450 5150
-F 0 "C28" H 8470 5120 50  0000 L TNN
+F 0 "C39" H 8470 5120 50  0000 L TNN
 F 1 "10u" H 8475 5170 30  0000 L BNN
 F 2 "Capacitors_SMD:C_0805" H 8450 5150 60  0001 C CNN
@@
 $EndComp
 $Comp
-L symbols:CAP C29
+L symbols:CAP C40
 U 1 1 5C681F5D
 P 8650 5150
-F 0 "C29" H 8670 5120 50  0000 L TNN
+F 0 "C40" H 8670 5120 50  0000 L TNN
 F 1 "2.2u" H 8675 5170 30  0000 L BNN
 F 2 "Capacitors_SMD:C_0603" H 8650 5150 60  0001 C CNN
@@
 Connection ~ 8650 4950
 $Comp
-L power:GNDA #PWR0130
+L power:GNDA #PWR037
 U 1 1 5C68602A
 P 2250 5950
-F 0 "#PWR0130" H 2250 5700 50  0001 C CNN
+F 0 "#PWR037" H 2250 5700 50  0001 C CNN
 F 1 "GNDA" H 2255 5777 50  0000 C CNN
 F 2 "" H 2250 5950 50  0001 C CNN
@@
 	1100 5200 1100 5450
 $Comp
-L symbols:CAP C21
+L symbols:CAP C32
 U 1 1 5C697450
 P 1600 5650
-F 0 "C21" H 1620 5620 50  0000 L TNN
+F 0 "C32" H 1620 5620 50  0000 L TNN
 F 1 "2.2u" H 1625 5670 30  0000 L BNN
 F 2 "Capacitors_SMD:C_0603" H 1600 5650 60  0001 C CNN
@@
 	1800 5550 1950 5550
 $Comp
-L symbols:RES R8
+L symbols:RES R11
 U 1 1 5C6A9EAC
 P 1800 5750
-F 0 "R8" H 1870 5715 50  0000 L TNN
+F 0 "R11" H 1870 5715 50  0000 L TNN
 F 1 "100k" H 1800 5805 30  0000 C BNN
 F 2 "Resistors_SMD:R_0402" H 1800 5750 60  0001 C CNN
@@
 Connection ~ 1800 5550
 $Comp
-L power:GND #PWR0131
+L power:GND #PWR035
 U 1 1 5C6AF054
 P 1600 6050
-F 0 "#PWR0131" H 1600 5800 50  0001 C CNN
+F 0 "#PWR035" H 1600 5800 50  0001 C CNN
 F 1 "GND" H 1605 5877 50  0000 C CNN
 F 2 "" H 1600 6050 50  0001 C CNN
@@
 	1100 5450 1600 5450
 $Comp
-L symbols:CAP C27
+L symbols:CAP C38
 U 1 1 5C6BF0EB
 P 7550 5200
-F 0 "C27" H 7570 5170 50  0000 L TNN
+F 0 "C38" H 7570 5170 50  0000 L TNN
 F 1 "2.2u" H 7575 5220 30  0000 L BNN
 F 2 "Capacitors_SMD:C_0603" H 7550 5200 60  0001 C CNN
@@
 	7700 4950 7750 4950
 $Comp
-L power:GND #PWR0132
+L power:GND #PWR048
 U 1 1 5C6C9CA2
 P 7550 5350
-F 0 "#PWR0132" H 7550 5100 50  0001 C CNN
+F 0 "#PWR048" H 7550 5100 50  0001 C CNN
 F 1 "GND" H 7555 5177 50  0000 C CNN
 F 2 "" H 7550 5350 50  0001 C CNN
@@
 Connection ~ 7550 4950
 $Comp
-L power:GND #PWR0133
+L power:GND #PWR049
 U 1 1 5C6D5457
 P 8050 5600
-F 0 "#PWR0133" H 8050 5350 50  0001 C CNN
+F 0 "#PWR049" H 8050 5350 50  0001 C CNN
 F 1 "GND" H 8055 5427 50  0000 C CNN
 F 2 "" H 8050 5600 50  0001 C CNN
@@
 	7050 3000 6850 3000
 $Comp
-L symbols:CAP C25
+L symbols:CAP C36
 U 1 1 5C6E6B78
 P 6850 3200
-F 0 "C25" H 6870 3170 50  0000 L TNN
+F 0 "C36" H 6870 3170 50  0000 L TNN
 F 1 "10u" H 6875 3220 30  0000 L BNN
 F 2 "Capacitors_SMD:C_0805" H 6850 3200 60  0001 C CNN
@@
 $EndComp
 $Comp
-L symbols:CAP C26
+L symbols:CAP C37
 U 1 1 5C6E6B7E
 P 7050 3200
-F 0 "C26" H 7070 3170 50  0000 L TNN
+F 0 "C37" H 7070 3170 50  0000 L TNN
 F 1 "2.2u" H 7075 3220 30  0000 L BNN
 F 2 "Capacitors_SMD:C_0603" H 7050 3200 60  0001 C CNN
@@
 Connection ~ 7050 3000
 $Comp
-L symbols:CAP C24
+L symbols:CAP C35
 U 1 1 5C6E6B89
 P 5950 3250
-F 0 "C24" H 5970 3220 50  0000 L TNN
+F 0 "C35" H 5970 3220 50  0000 L TNN
 F 1 "2.2u" H 5975 3270 30  0000 L BNN
 F 2 "Capacitors_SMD:C_0603" H 5950 3250 60  0001 C CNN
@@
 	6100 3000 6150 3000
 $Comp
-L power:GND #PWR0134
+L power:GND #PWR044
 U 1 1 5C6E6B95
 P 5950 3450
-F 0 "#PWR0134" H 5950 3200 50  0001 C CNN
+F 0 "#PWR044" H 5950 3200 50  0001 C CNN
 F 1 "GND" H 5955 3277 50  0000 C CNN
 F 2 "" H 5950 3450 50  0001 C CNN
@@
 $EndComp
 $Comp
-L symbols:USB_5V #PWR0135
+L symbols:USB_5V #PWR036
 U 1 1 5C6E6B9C
 P 2050 2850
-F 0 "#PWR0135" H 2050 2810 30  0001 C CNN
+F 0 "#PWR036" H 2050 2810 30  0001 C CNN
 F 1 "USB_5V" H 2050 2960 30  0000 C CNN
 F 2 "~" H 2050 2850 60  0000 C CNN
@@
 Connection ~ 5950 3000
 $Comp
-L power:GND #PWR0136
+L power:GND #PWR045
 U 1 1 5C6E6BA4
 P 6450 3650
-F 0 "#PWR0136" H 6450 3400 50  0001 C CNN
+F 0 "#PWR045" H 6450 3400 50  0001 C CNN
 F 1 "GND" H 6455 3477 50  0000 C CNN
 F 2 "" H 6450 3650 50  0001 C CNN
@@
 Connection ~ 6850 3500
 $Comp
-L symbols:RES R9
+L symbols:RES R12
 U 1 1 5C72514F
 P 2400 3000
-F 0 "R9" H 2470 2965 50  0000 L TNN
+F 0 "R12" H 2470 2965 50  0000 L TNN
 F 1 "0R" H 2400 3055 30  0000 C BNN
 F 2 "Resistors_SMD:R_0402" H 2400 3000 60  0001 C CNN
@@
 $EndComp
 $Comp
-L power:+5V #PWR0137
+L power:+5V #PWR038
 U 1 1 5C736202
 P 2650 2850
-F 0 "#PWR0137" H 2650 2700 50  0001 C CNN
+F 0 "#PWR038" H 2650 2700 50  0001 C CNN
 F 1 "+5V" H 2665 3023 50  0000 C CNN
 F 2 "" H 2650 2850 50  0001 C CNN
@@
 Connection ~ 2650 3000
 $Comp
-L power:GND #PWR0138
+L power:GND #PWR039
 U 1 1 5C750C65
 P 2650 3200
-F 0 "#PWR0138" H 2650 2950 50  0001 C CNN
+F 0 "#PWR039" H 2650 2950 50  0001 C CNN
 F 1 "GND" H 2655 3027 50  0000 C CNN
 F 2 "" H 2650 3200 50  0001 C CNN
@@
 	5950 2750 5950 3000
 $Comp
-L power:+5V #PWR0139
+L power:+5V #PWR043
 U 1 1 5C762562
 P 5950 2750
-F 0 "#PWR0139" H 5950 2600 50  0001 C CNN
+F 0 "#PWR043" H 5950 2600 50  0001 C CNN
 F 1 "+5V" H 5965 2923 50  0000 C CNN
 F 2 "" H 5950 2750 50  0001 C CNN
@@
 $EndComp
 $Comp
-L power:+5V #PWR0140
+L power:+5V #PWR034
 U 1 1 5C7625E8
 P 1100 5200
-F 0 "#PWR0140" H 1100 5050 50  0001 C CNN
+F 0 "#PWR034" H 1100 5050 50  0001 C CNN
 F 1 "+5V" H 1115 5373 50  0000 C CNN
 F 2 "" H 1100 5200 50  0001 C CNN
@@
 $EndComp
 $Comp
-L power:+5V #PWR0141
+L power:+5V #PWR047
 U 1 1 5C7628B7
 P 7550 4750
-F 0 "#PWR0141" H 7550 4600 50  0001 C CNN
+F 0 "#PWR047" H 7550 4600 50  0001 C CNN
 F 1 "+5V" H 7565 4923 50  0000 C CNN
 F 2 "" H 7550 4750 50  0001 C CNN
@@
 Connection ~ 8650 5450
 $Comp
-L power:GNDA #PWR0142
+L power:GNDA #PWR041
 U 1 1 5C799F30
 P 4700 5000
-F 0 "#PWR0142" H 4700 4750 50  0001 C CNN
+F 0 "#PWR041" H 4700 4750 50  0001 C CNN
 F 1 "GNDA" H 4705 4827 50  0000 C CNN
 F 2 "" H 4700 5000 50  0001 C CNN

Commit message: Much more routing
Parts:
- C32, C34, C35, C37, C38, C40: footprint Capacitors_SMD:C_0603 -> Capacitor_SMD:C_0603_1608Metric_Pad1.05x0.95mm_HandSolder
- C33, C36, C39: footprint Capacitors_SMD:C_0805 -> Capacitor_SMD:C_0805_2012Metric_Pad1.15x1.40mm_HandSolder
- J4: footprint TerminalBlocks_Phoenix:TerminalBlock_Phoenix_MPT-2.54mm_2pol -> Connector_PinHeader_2.54mm:PinHeader_1x02_P2.54mm_Vertical
- R11, R12: footprint Resistors_SMD:R_0402 -> Resistor_SMD:R_0402_1005Metric
- U5, U6, U7: footprint TO_SOT_Packages_SMD:SOT-23-5 -> Package_TO_SOT_SMD:SOT-23-5
Changed lines of the file:
@@
 EESchema Schematic File Version 4
 LIBS:audio_iface_rev2-cache
-EELAYER 29 0
+EELAYER 30 0
 EELAYER END
 $Descr A4 11693 8268
@@
 F 0 "J4" H 3280 2992 50  0000 L CNN
 F 1 "Screw_Terminal_01x02" H 3280 2901 50  0000 L CNN
-F 2 "TerminalBlocks_Phoenix:TerminalBlock_Phoenix_MPT-2.54mm_2pol" H 3200 3000 50  0001 C CNN
+F 2 "Connector_PinHeader_2.54mm:PinHeader_1x02_P2.54mm_Vertical" H 3200 3000 50  0001 C CNN
 F 3 "~" H 3200 3000 50  0001 C CNN
 	1    3200 3000
@@
 F 0 "U6" H 6450 3467 50  0000 C CNN
 F 1 "LP5907MFX-1.8" H 6450 3376 50  0000 C CNN
-F 2 "TO_SOT_Packages_SMD:SOT-23-5" H 6450 3450 50  0001 C CNN
+F 2 "Package_TO_SOT_SMD:SOT-23-5" H 6450 3450 50  0001 C CNN
 F 3 "http://www.ti.com/lit/ds/symlink/lp5907.pdf" H 6450 3600 50  0001 C CNN
 	1    6450 3100
@@
 F 0 "U5" H 2250 5917 50  0000 C CNN
 F 1 "LP5907MFX-3.3" H 2250 5826 50  0000 C CNN
-F 2 "TO_SOT_Packages_SMD:SOT-23-5" H 2250 5900 50  0001 C CNN
+F 2 "Package_TO_SOT_SMD:SOT-23-5" H 2250 5900 50  0001 C CNN
 F 3 "http://www.ti.com/lit/ds/symlink/lp5907.pdf" H 2250 6050 50  0001 C CNN
 	1    2250 5550
@@
 F 0 "U7" H 8050 5417 50  0000 C CNN
 F 1 "LP5907MFX-3.3" H 8050 5326 50  0000 C CNN
-F 2 "TO_SOT_Packages_SMD:SOT-23-5" H 8050 5400 50  0001 C CNN
+F 2 "Package_TO_SOT_SMD:SOT-23-5" H 8050 5400 50  0001 C CNN
 F 3 "http://www.ti.com/lit/ds/symlink/lp5907.pdf" H 8050 5550 50  0001 C CNN
 	1    8050 5050
@@
 F 0 "C33" H 2720 5620 50  0000 L TNN
 F 1 "10u" H 2725 5670 30  0000 L BNN
-F 2 "Capacitors_SMD:C_0805" H 2700 5650 60  0001 C CNN
+F 2 "Capacitor_SMD:C_0805_2012Metric_Pad1.15x1.40mm_HandSolder" H 2700 5650 60  0001 C CNN
 F 3 "~" H 2700 5650 60  0000 C CNN
 	1    2700 5650
@@
 F 0 "C34" H 2920 5620 50  0000 L TNN
 F 1 "2.2u" H 2925 5670 30  0000 L BNN
-F 2 "Capacitors_SMD:C_0603" H 2900 5650 60  0001 C CNN
+F 2 "Capacitor_SMD:C_0603_1608Metric_Pad1.05x0.95mm_HandSolder" H 2900 5650 60  0001 C CNN
 F 3 "~" H 2900 5650 60  0000 C CNN
 	1    2900 5650
@@
 F 0 "C39" H 8470 5120 50  0000 L TNN
 F 1 "10u" H 8475 5170 30  0000 L BNN
-F 2 "Capacitors_SMD:C_0805" H 8450 5150 60  0001 C CNN
+F 2 "Capacitor_SMD:C_0805_2012Metric_Pad1.15x1.40mm_HandSolder" H 8450 5150 60  0001 C CNN
 F 3 "~" H 8450 5150 60  0000 C CNN
 	1    8450 5150
@@
 F 0 "C40" H 8670 5120 50  0000 L TNN
 F 1 "2.2u" H 8675 5170 30  0000 L BNN
-F 2 "Capacitors_SMD:C_0603" H 8650 5150 60  0001 C CNN
+F 2 "Capacitor_SMD:C_0603_1608Metric_Pad1.05x0.95mm_HandSolder" H 8650 5150 60  0001 C CNN
 F 3 "~" H 8650 5150 60  0000 C CNN
 	1    8650 5150
@@
 F 0 "C32" H 1620 5620 50  0000 L TNN
 F 1 "2.2u" H 1625 5670 30  0000 L BNN
-F 2 "Capacitors_SMD:C_0603" H 1600 5650 60  0001 C CNN
+F 2 "Capacitor_SMD:C_0603_1608Metric_Pad1.05x0.95mm_HandSolder" H 1600 5650 60  0001 C CNN
 F 3 "~" H 1600 5650 60  0000 C CNN
 	1    1600 5650
@@
 F 0 "R11" H 1870 5715 50  0000 L TNN
 F 1 "100k" H 1800 5805 30  0000 C BNN
-F 2 "Resistors_SMD:R_0402" H 1800 5750 60  0001 C CNN
+F 2 "Resistor_SMD:R_0402_1005Metric" H 1800 5750 60  0001 C CNN
 F 3 "~" H 1800 5750 60  0000 C CNN
 	1    1800 5750
@@
 F 0 "C38" H 7570 5170 50  0000 L TNN
 F 1 "2.2u" H 7575 5220 30  0000 L BNN
-F 2 "Capacitors_SMD:C_0603" H 7550 5200 60  0001 C CNN
+F 2 "Capacitor_SMD:C_0603_1608Metric_Pad1.05x0.95mm_HandSolder" H 7550 5200 60  0001 C CNN
 F 3 "~" H 7550 5200 60  0000 C CNN
 	1    7550 5200
@@
 F 0 "C36" H 6870 3170 50  0000 L TNN
 F 1 "10u" H 6875 3220 30  0000 L BNN
-F 2 "Capacitors_SMD:C_0805" H 6850 3200 60  0001 C CNN
+F 2 "Capacitor_SMD:C_0805_2012Metric_Pad1.15x1.40mm_HandSolder" H 6850 3200 60  0001 C CNN
 F 3 "~" H 6850 3200 60  0000 C CNN
 	1    6850 3200
@@
 F 0 "C37" H 7070 3170 50  0000 L TNN
 F 1 "2.2u" H 7075 3220 30  0000 L BNN
-F 2 "Capacitors_SMD:C_0603" H 7050 3200 60  0001 C CNN
+F 2 "Capacitor_SMD:C_0603_1608Metric_Pad1.05x0.95mm_HandSolder" H 7050 3200 60  0001 C CNN
 F 3 "~" H 7050 3200 60  0000 C CNN
 	1    7050 3200
@@
 F 0 "C35" H 5970 3220 50  0000 L TNN
 F 1 "2.2u" H 5975 3270 30  0000 L BNN
-F 2 "Capacitors_SMD:C_0603" H 5950 3250 60  0001 C CNN
+F 2 "Capacitor_SMD:C_0603_1608Metric_Pad1.05x0.95mm_HandSolder" H 5950 3250 60  0001 C CNN
 F 3 "~" H 5950 3250 60  0000 C CNN
 	1    5950 3250
@@
 F 0 "R12" H 2470 2965 50  0000 L TNN
 F 1 "0R" H 2400 3055 30  0000 C BNN
-F 2 "Resistors_SMD:R_0402" H 2400 3000 60  0001 C CNN
+F 2 "Resistor_SMD:R_0402_1005Metric" H 2400 3000 60  0001 C CNN
 F 3 "~" H 2400 3000 60  0000 C CNN
 	1    2400 3000
