File: hw/rev2/power.sch (KiCad schematic (older format))
At the start: 18 parts, among them J4 Screw_Terminal_01x02, U5 LP5907MFX-3.3, U6 LP5907MFX-1.8, U7 LP5907MFX-3.3

Commit message: Design nearly complete. One more check.
Parts:
- C32, C33, C34, C35, C36, C37, C38, C39, C40: symbol symbols:CAP -> Device:C_Small
- R12: symbol symbols:RES -> Device:R_Small
Connections:
- net labels removed: GND
- wire segments 74 -> 75
Changed lines of the file:
@@
 	2900 5450 2700 5450
 $Comp
-L symbols:CAP C33
+L Device:C_Small C33
 U 1 1 5C676BB9
 P 2700 5650
@@
 F 3 "~" H 2700 5650 60  0000 C CNN
 	1    2700 5650
-	0    -1   -1   0
-$EndComp
-$Comp
-L symbols:CAP C34
+	-1   0    0    1
+$EndComp
+$Comp
+L Device:C_Small C34
 U 1 1 5C676C4D
 P 2900 5650
@@
 F 3 "~" H 2900 5650 60  0000 C CNN
 	1    2900 5650
-	0    -1   -1   0
+	-1   0    0    1
 $EndComp
 Wire Wire Line
@@
 	2700 5450 2550 5450
 $Comp
-L symbols:CAP C39
+L Device:C_Small C39
 U 1 1 5C681F57
 P 8450 5150
@@
 F 3 "~" H 8450 5150 60  0000 C CNN
 	1    8450 5150
-	0    -1   -1   0
-$EndComp
-$Comp
-L symbols:CAP C40
-U 1 1 5C681F5D
-P 8650 5150
-F 0 "C40" H 8670 5120 50  0000 L TNN
-F 1 "2.2u" H 8675 5170 30  0000 L BNN
-F 2 "Capacitor_SMD:C_0603_1608Metric_Pad1.05x0.95mm_HandSolder" H 8650 5150 60  0001 C CNN
-F 3 "~" H 8650 5150 60  0000 C CNN
-	1    8650 5150
-	0    -1   -1   0
+	-1   0    0    1
 $EndComp
 Wire Wire Line
@@
 Wire Wire Line
 	1100 5200 1100 5450
-$Comp
-L symbols:CAP C32
-U 1 1 5C697450
-P 1600 5650
-F 0 "C32" H 1620 5620 50  0000 L TNN
-F 1 "2.2u" H 1625 5670 30  0000 L BNN
-F 2 "Capacitor_SMD:C_0603_1608Metric_Pad1.05x0.95mm_HandSolder" H 1600 5650 60  0001 C CNN
-F 3 "~" H 1600 5650 60  0000 C CNN
-	1    1600 5650
-	0    -1   -1   0
-$EndComp
 Wire Wire Line
 	1600 5550 1600 5450
@@
 	1800 5600 1800 5550
 Connection ~ 1800 5550
-$Comp
-L power:GND #PWR035
-U 1 1 5C6AF054
-P 1600 6050
-F 0 "#PWR035" H 1600 5800 50  0001 C CNN
-F 1 "GND" H 1605 5877 50  0000 C CNN
-F 2 "" H 1600 6050 50  0001 C CNN
-F 3 "" H 1600 6050 50  0001 C CNN
-	1    1600 6050
-	1    0    0    -1
-$EndComp
 Wire Wire Line
 	1600 5950 1800 5950
@@
 	1100 5450 1600 5450
 $Comp
-L symbols:CAP C38
+L Device:C_Small C38
 U 1 1 5C6BF0EB
 P 7550 5200
@@
 F 3 "~" H 7550 5200 60  0000 C CNN
 	1    7550 5200
-	0    -1   -1   0
+	-1   0    0    1
 $EndComp
 Wire Wire Line
@@
 Wire Wire Line
 	7700 4950 7750 4950
-$Comp
-L power:GND #PWR048
-U 1 1 5C6C9CA2
-P 7550 5350
-F 0 "#PWR048" H 7550 5100 50  0001 C CNN
-F 1 "GND" H 7555 5177 50  0000 C CNN
-F 2 "" H 7550 5350 50  0001 C CNN
-F 3 "" H 7550 5350 50  0001 C CNN
-	1    7550 5350
-	1    0    0    -1
-$EndComp
 Wire Wire Line
 	7550 5350 7550 5300
@@
 	7550 4750 7550 4950
 Connection ~ 7550 4950
-$Comp
-L power:GND #PWR049
-U 1 1 5C6D5457
-P 8050 5600
-F 0 "#PWR049" H 8050 5350 50  0001 C CNN
-F 1 "GND" H 8055 5427 50  0000 C CNN
-F 2 "" H 8050 5600 50  0001 C CNN
-F 3 "" H 8050 5600 50  0001 C CNN
-	1    8050 5600
-	1    0    0    -1
-$EndComp
 Wire Wire Line
 	8050 5600 8050 5450
@@
 	7050 3000 6850 3000
 $Comp
-L symbols:CAP C36
+L Device:C_Small C36
 U 1 1 5C6E6B78
 P 6850 3200
@@
 F 3 "~" H 6850 3200 60  0000 C CNN
 	1    6850 3200
-	0    -1   -1   0
-$EndComp
-$Comp
-L symbols:CAP C37
+	-1   0    0    1
+$EndComp
+$Comp
+L Device:C_Small C37
 U 1 1 5C6E6B7E
 P 7050 3200
@@
 F 3 "~" H 7050 3200 60  0000 C CNN
 	1    7050 3200
-	0    -1   -1   0
+	-1   0    0    1
 $EndComp
 Wire Wire Line
@@
 Connection ~ 7050 3000
 $Comp
-L symbols:CAP C35
+L Device:C_Small C35
 U 1 1 5C6E6B89
 P 5950 3250
@@
 F 3 "~" H 5950 3250 60  0000 C CNN
 	1    5950 3250
-	0    -1   -1   0
+	-1   0    0    1
 $EndComp
 Wire Wire Line
@@
 	6100 3000 6150 3000
 $Comp
-L power:GND #PWR044
-U 1 1 5C6E6B95
-P 5950 3450
-F 0 "#PWR044" H 5950 3200 50  0001 C CNN
-F 1 "GND" H 5955 3277 50  0000 C CNN
-F 2 "" H 5950 3450 50  0001 C CNN
-F 3 "" H 5950 3450 50  0001 C CNN
-	1    5950 3450
-	1    0    0    -1
-$EndComp
-$Comp
-L symbols:USB_5V #PWR036
+L audio_iface_rev2-rescue:USB_5V-symbols #PWR036
 U 1 1 5C6E6B9C
 P 2050 2850
+AR Path="/5C6E6B9C" Ref="#PWR036"  Part="1"
+AR Path="/524EE3EB/5C6E6B9C" Ref="#PWR036"  Part="1"
 F 0 "#PWR036" H 2050 2810 30  0001 C CNN
 F 1 "USB_5V" H 2050 2960 30  0000 C CNN
@@
 $EndComp
 Connection ~ 5950 3000
-$Comp
-L power:GND #PWR045
-U 1 1 5C6E6BA4
-P 6450 3650
-F 0 "#PWR045" H 6450 3400 50  0001 C CNN
-F 1 "GND" H 6455 3477 50  0000 C CNN
-F 2 "" H 6450 3650 50  0001 C CNN
-F 3 "" H 6450 3650 50  0001 C CNN
-	1    6450 3650
-	1    0    0    -1
-$EndComp
 Wire Wire Line
 	6450 3650 6450 3500
@@
 Connection ~ 6850 3500
 $Comp
-L symbols:RES R12
+L Device:R_Small R12
 U 1 1 5C72514F
 P 2400 3000
-F 0 "R12" H 2470 2965 50  0000 L TNN
-F 1 "0R" H 2400 3055 30  0000 C BNN
+F 0 "R12" V 2450 3050 50  0000 L TNN
+F 1 "0R" V 2350 3100 30  0000 C BNN
 F 2 "Resistor_SMD:R_0402_1005Metric" H 2400 3000 60  0001 C CNN
 F 3 "~" H 2400 3000 60  0000 C CNN
 	1    2400 3000
-	1    0    0    -1
+	0    -1   -1   0
 $EndComp
 $Comp
@@
 	2050 2850 2050 3000
 Wire Wire Line
-	2050 3000 2250 3000
-Wire Wire Line
-	2550 3000 2650 3000
+	2050 3000 2300 3000
+Wire Wire Line
+	2500 3000 2650 3000
 Wire Wire Line
 	2650 3000 2650 2850
@@
 	3000 3000 2650 3000
 Connection ~ 2650 3000
-$Comp
-L power:GND #PWR039
-U 1 1 5C750C65
-P 2650 3200
-F 0 "#PWR039" H 2650 2950 50  0001 C CNN
-F 1 "GND" H 2655 3027 50  0000 C CNN
-F 2 "" H 2650 3200 50  0001 C CNN
-F 3 "" H 2650 3200 50  0001 C CNN
-	1    2650 3200
-	1    0    0    -1
-$EndComp
 Wire Wire Line
 	2650 3200 2650 3100
@@
 	1    0    0    -1
 $EndComp
+$Comp
+L power:GNDD #PWR0102
+U 1 1 5D88F8FD
+P 2650 3200
+F 0 "#PWR0102" H 2650 2950 50  0001 C CNN
+F 1 "GNDD" H 2654 3045 50  0000 C CNN
+F 2 "" H 2650 3200 50  0001 C CNN
+F 3 "" H 2650 3200 50  0001 C CNN
+	1    2650 3200
+	1    0    0    -1
+$EndComp
+$Comp
+L power:GNDD #PWR0103
+U 1 1 5D891CE9
+P 1600 6050
+F 0 "#PWR0103" H 1600 5800 50  0001 C CNN
+F 1 "GNDD" H 1604 5895 50  0000 C CNN
+F 2 "" H 1600 6050 50  0001 C CNN
+F 3 "" H 1600 6050 50  0001 C CNN
+	1    1600 6050
+	1    0    0    -1
+$EndComp
+$Comp
+L power:GNDD #PWR0104
+U 1 1 5D894357
+P 8050 5600
+F 0 "#PWR0104" H 8050 5350 50  0001 C CNN
+F 1 "GNDD" H 8050 5450 50  0000 C CNN
+F 2 "" H 8050 5600 50  0000 C CNN
+F 3 "" H 8050 5600 50  0000 C CNN
+	1    8050 5600
+	1    0    0    -1
+$EndComp
+$Comp
+L power:GNDD #PWR0105
+U 1 1 5D895D9A
+P 7550 5350
+F 0 "#PWR0105" H 7550 5100 50  0001 C CNN
+F 1 "GNDD" H 7550 5200 50  0000 C CNN
+F 2 "" H 7550 5350 50  0000 C CNN
+F 3 "" H 7550 5350 50  0000 C CNN
+	1    7550 5350
+	1    0    0    -1
+$EndComp
+$Comp
+L power:GNDD #PWR0106
+U 1 1 5D8961B9
+P 5950 3450
+F 0 "#PWR0106" H 5950 3200 50  0001 C CNN
+F 1 "GNDD" H 5950 3300 50  0000 C CNN
+F 2 "" H 5950 3450 50  0000 C CNN
+F 3 "" H 5950 3450 50  0000 C CNN
+	1    5950 3450
+	1    0    0    -1
+$EndComp
+$Comp
+L power:GNDD #PWR0107
+U 1 1 5D897D71
+P 6450 3650
+F 0 "#PWR0107" H 6450 3400 50  0001 C CNN
+F 1 "GNDD" H 6450 3500 50  0000 C CNN
+F 2 "" H 6450 3650 50  0000 C CNN
+F 3 "" H 6450 3650 50  0000 C CNN
+	1    6450 3650
+	1    0    0    -1
+$EndComp
+Wire Wire Line
+	4700 4750 5100 4750
+$Comp
+L Device:C_Small C32
+U 1 1 5C697450
+P 1600 5650
+F 0 "C32" H 1620 5620 50  0000 L TNN
+F 1 "2.2u" H 1625 5670 30  0000 L BNN
+F 2 "Capacitor_SMD:C_0603_1608Metric_Pad1.05x0.95mm_HandSolder" H 1600 5650 60  0001 C CNN
+F 3 "~" H 1600 5650 60  0000 C CNN
+	1    1600 5650
+	-1   0    0    1
+$EndComp
+$Comp
+L Device:C_Small C40
+U 1 1 5C681F5D
+P 8650 5150
+F 0 "C40" H 8670 5120 50  0000 L TNN
+F 1 "2.2u" H 8675 5170 30  0000 L BNN
+F 2 "Capacitor_SMD:C_0603_1608Metric_Pad1.05x0.95mm_HandSolder" H 8650 5150 60  0001 C CNN
+F 3 "~" H 8650 5150 60  0000 C CNN
+	1    8650 5150
+	-1   0    0    1
+$EndComp
 $EndSCHEMATC
