File: hw/rev2/audio_in.sch (KiCad schematic (older format))
At the start: 45 parts, among them U201 LT6241, U202 LTC6242

Commit message: Lots of things: --Added RGB LED on timer outputs --Input: Moved capacitively coupled feedback nodes from vgnd to gnd --Output: LTC6242 for filtering to amplifier --Power: 2-stage supply for analog: USB 5V boost to 6V, LDO to 5V   Digital still using LDO from USB 5V and not caring about anyone   Bonus! Can completely shut off analog portion of board --Layout and routing: All of it TODO: final checks on layout and LVS (vs simulation) HEAD2HEAD2HEAD! TODO: adjust silkscreen, add logo TODO: debate adding 12.288MHz dedicated crystal
Parts:
- removed C204: 10u 6.3V, ~, symbol CPOL
- removed R201: 3.9k, symbol RES
- removed R218, R219: 1k, ~, symbol RES
- removed R?: 10k, symbol RES
- added C2: 10u 6.3V, ~, symbol CAP
- added C20: 10p, ~, symbol CAP
- added C4: 100u 6.3V, ~, symbol CPOL
- added C69: 0.1u, ~, symbol CAP
- added TP2, TP3: TP, ~, symbol TP
- C12: renamed from C221; symbol CPOL -> CAP
- C3: renamed from C?; footprint SMD0402 -> ~
- R4, R5: renamed from R?; value 1k (1%) -> 100k (1%)
- R6: renamed from R207; value 90 (1%) -> 470 (1%)
- Rf1: renamed from Rf; value 1.20k (1%) -> 5.11k (1%)
- gave numbers to parts that had none: 4
- renumbered C216 to C10, C220 to C11, C212 to C13, C217 to C14, C213 to C15, C214 to C17, C215 to C18, C218 to C19, C219 to C21, C223 to C23, C222 to C24, C207 to C5, C209 to C6, C208 to C7, C211 to C8, C210 to C9, R221 to R10, R223 to R11, R222 to R12, R224 to R13, R226 to R14, R225 to R16, R229 to R17, R227 to R18, R228 to R19, R216 to R7, R217 to R8, R220 to R9, U201 to U1, U202 to U2
Connections:
- wire segments 118 -> 117

Commit message: Added extra oscillator JIC. Moved labels and made it pretty. Also fixed a missing capacitron
Parts:
- added C70: 0.01u, ~, symbol CAP
Connections:
- wire segments 117 -> 119
Changed lines of the file:
@@
 Sheet 2 6
 Title "Android DPOAE Interface"
-Date "3 may 2014"
+Date "6 may 2014"
 Rev "2a"
 Comp "Sana AudioPulse"
@@
 L OPAMP_QUAD U2
 U 2 1 523B17B7
-P 3250 3650
-F 0 "U2" H 3325 3500 60  0000 L CNN
-F 1 "LTC6242" H 3300 3800 60  0000 L CNN
-F 2 "~" H 3250 3650 60  0000 C CNN
-F 3 "~" H 3250 3650 60  0000 C CNN
-	2    3250 3650
+P 2750 3650
+F 0 "U2" H 2825 3500 60  0000 L CNN
+F 1 "LTC6242" H 2800 3800 60  0000 L CNN
+F 2 "~" H 2750 3650 60  0000 C CNN
+F 3 "~" H 2750 3650 60  0000 C CNN
+	2    2750 3650
 	1    0    0    -1
 $EndComp
@@
 	0    -1   -1   0
 $EndComp
-Text HLabel 2050 3750 0    60   Input ~ 0
+Text HLabel 1550 3750 0    60   Input ~ 0
 MIC_IN
 Text HLabel 8800 3550 2    60   Output ~ 0
@@
 MIC_DIFF_P
 $Comp
-L AGND_IN #PWR06
+L AGND_IN #PWR19
 U 1 1 523BB57F
 P 8100 2300
-F 0 "#PWR06" H 8100 2300 40  0001 C CNN
+F 0 "#PWR19" H 8100 2300 40  0001 C CNN
 F 1 "AGND_IN" H 8100 2230 50  0000 C CNN
 F 2 "" H 8100 2300 60  0000 C CNN
@@
 $EndComp
 $Comp
-L AGND_IN #PWR07
+L AGND_IN #PWR21
 U 1 1 523BB58F
 P 8600 2300
-F 0 "#PWR07" H 8600 2300 40  0001 C CNN
+F 0 "#PWR21" H 8600 2300 40  0001 C CNN
 F 1 "AGND_IN" H 8600 2230 50  0000 C CNN
 F 2 "" H 8600 2300 60  0000 C CNN
@@
 $EndComp
 $Comp
-L VCOM_VRT #PWR14
+L VCOM_VRT #PWR15
 U 1 1 523BBA77
 P 7200 4450
-F 0 "#PWR14" H 7200 4650 40  0001 C CNN
+F 0 "#PWR15" H 7200 4650 40  0001 C CNN
 F 1 "VCOM_VRT" H 7200 4600 40  0000 C CNN
 F 2 "" H 7200 4450 60  0000 C CNN
@@
 $EndComp
 $Comp
-L VCOM_VRT #PWR11
+L VCOM_VRT #PWR12
 U 1 1 523BBACF
 P 4600 4750
-F 0 "#PWR11" H 4600 4950 40  0001 C CNN
+F 0 "#PWR12" H 4600 4950 40  0001 C CNN
 F 1 "VCOM_VRT" H 4600 4900 40  0000 C CNN
 F 2 "" H 4600 4750 60  0000 C CNN
@@
 L RES R6
 U 1 1 5245ECF0
+P 2200 3250
+F 0 "R6" H 2270 3215 50  0000 L TNN
+F 1 "470 (1%)" H 2200 3305 30  0000 C BNN
+F 2 "" H 2200 3250 60  0000 C CNN
+F 3 "" H 2200 3250 60  0000 C CNN
+	1    2200 3250
+	1    0    0    -1
+$EndComp
+$Comp
+L RES Rf1
+U 1 1 5245ECF6
 P 2700 3250
-F 0 "R6" H 2770 3215 50  0000 L TNN
-F 1 "470 (1%)" H 2700 3305 30  0000 C BNN
+F 0 "Rf1" H 2770 3215 50  0000 L TNN
+F 1 "5.11k (1%)" H 2700 3305 30  0000 C BNN
 F 2 "" H 2700 3250 60  0000 C CNN
 F 3 "" H 2700 3250 60  0000 C CNN
 	1    2700 3250
-	1    0    0    -1
-$EndComp
-$Comp
-L RES Rf1
-U 1 1 5245ECF6
-P 3200 3250
-F 0 "Rf1" H 3270 3215 50  0000 L TNN
-F 1 "5.11k (1%)" H 3200 3305 30  0000 C BNN
-F 2 "" H 3200 3250 60  0000 C CNN
-F 3 "" H 3200 3250 60  0000 C CNN
-	1    3200 3250
 	1    0    0    -1
 $EndComp
@@
 $EndComp
 $Comp
-L AGND_IN #PWR08
+L AGND_IN #PWR17
 U 1 1 524EBECC
 P 7400 2300
-F 0 "#PWR08" H 7400 2300 40  0001 C CNN
+F 0 "#PWR17" H 7400 2300 40  0001 C CNN
 F 1 "AGND_IN" H 7400 2230 50  0000 C CNN
 F 2 "" H 7400 2300 60  0000 C CNN
@@
 $EndComp
 $Comp
-L +5VA #PWR09
+L +5VA #PWR16
 U 1 1 524E7127
 P 7400 1500
-F 0 "#PWR09" H 7400 1630 20  0001 C CNN
+F 0 "#PWR16" H 7400 1630 20  0001 C CNN
 F 1 "+5VA" H 7400 1600 30  0000 C CNN
 F 2 "" H 7400 1500 60  0000 C CNN
@@
 $EndComp
 $Comp
-L +5VA #PWR010
+L +5VA #PWR18
 U 1 1 524E713E
 P 8100 1500
-F 0 "#PWR010" H 8100 1630 20  0001 C CNN
+F 0 "#PWR18" H 8100 1630 20  0001 C CNN
 F 1 "+5VA" H 8100 1600 30  0000 C CNN
 F 2 "" H 8100 1500 60  0000 C CNN
@@
 $EndComp
 $Comp
-L +5VA #PWR011
+L +5VA #PWR20
 U 1 1 524E7144
 P 8600 1500
-F 0 "#PWR011" H 8600 1630 20  0001 C CNN
+F 0 "#PWR20" H 8600 1630 20  0001 C CNN
 F 1 "+5VA" H 8600 1600 30  0000 C CNN
 F 2 "" H 8600 1500 60  0000 C CNN
@@
 $EndComp
 $Comp
-L AGND_IN #PWR012
+L AGND_IN #PWR8
 U 1 1 534E82DB
 P 2500 5450
-F 0 "#PWR012" H 2500 5450 40  0001 C CNN
+F 0 "#PWR8" H 2500 5450 40  0001 C CNN
 F 1 "AGND_IN" H 2500 5380 50  0000 C CNN
 F 2 "" H 2500 5450 60  0000 C CNN
@@
 $EndComp
 $Comp
-L +5VA #PWR013
+L +5VA #PWR7
 U 1 1 534E85DE
 P 2500 4350
-F 0 "#PWR013" H 2500 4480 20  0001 C CNN
+F 0 "#PWR7" H 2500 4480 20  0001 C CNN
 F 1 "+5VA" H 2500 4450 30  0000 C CNN
 F 2 "" H 2500 4350 60  0000 C CNN
@@
 L CAP C3
 U 1 1 534E87C8
-P 3200 3000
-F 0 "C3" H 3220 2970 50  0000 L TNN
-F 1 "10p" H 3225 3020 30  0000 L BNN
-F 2 "~" H 3200 3100 60  0000 C CNN
-F 3 "~" H 3200 3000 60  0000 C CNN
-	1    3200 3000
+P 2700 3000
+F 0 "C3" H 2720 2970 50  0000 L TNN
+F 1 "10p" H 2725 3020 30  0000 L BNN
+F 2 "~" H 2700 3100 60  0000 C CNN
+F 3 "~" H 2700 3000 60  0000 C CNN
+	1    2700 3000
 	1    0    0    -1
 $EndComp
@@
 L RES R15
 U 1 1 534E8F70
-P 7700 3300
-F 0 "R15" H 7770 3265 50  0000 L TNN
-F 1 "220k" H 7700 3355 30  0000 C BNN
-F 2 "~" H 7700 3300 60  0000 C CNN
-F 3 "~" H 7700 3300 60  0000 C CNN
-	1    7700 3300
+P 3600 3400
+F 0 "R15" H 3670 3365 50  0000 L TNN
+F 1 "220k" H 3600 3455 30  0000 C BNN
+F 2 "~" H 3600 3400 60  0000 C CNN
+F 3 "~" H 3600 3400 60  0000 C CNN
+	1    3600 3400
 	0    -1   -1   0
 $EndComp
 $Comp
-L VCOM_VRT #PWR17
+L VCOM_VRT #PWR9
 U 1 1 534E8F7D
-P 7700 3050
-F 0 "#PWR17" H 7700 3250 40  0001 C CNN
-F 1 "VCOM_VRT" H 7700 3200 40  0000 C CNN
-F 2 "" H 7700 3050 60  0000 C CNN
-F 3 "" H 7700 3050 60  0000 C CNN
-	1    7700 3050
+P 3600 3150
+F 0 "#PWR9" H 3600 3350 40  0001 C CNN
+F 1 "VCOM_VRT" H 3600 3300 40  0000 C CNN
+F 2 "" H 3600 3150 60  0000 C CNN
+F 3 "" H 3600 3150 60  0000 C CNN
+	1    3600 3150
 	1    0    0    -1
 $EndComp
@@
 $EndComp
 $Comp
-L VCOM_VRT #PWR12
+L VCOM_VRT #PWR13
 U 1 1 5357FD42
 P 5700 5900
-F 0 "#PWR12" H 5700 6100 40  0001 C CNN
+F 0 "#PWR13" H 5700 6100 40  0001 C CNN
 F 1 "VCOM_VRT" H 5700 6050 40  0000 C CNN
 F 2 "~" H 5700 5900 60  0000 C CNN
@@
 Connection ~ 3900 4750
 Wire Wire Line
-	3900 4900 3900 4750
+	3900 4750 3900 4900
 Wire Wire Line
 	6000 5050 6000 6000
@@
 Connection ~ 7500 4050
 Wire Wire Line
-	7400 4050 7500 4050
+	7500 4050 7400 4050
 Connection ~ 7100 4050
 Wire Wire Line
@@
 Connection ~ 7700 3550
 Wire Wire Line
-	7700 3450 7700 3550
-Wire Wire Line
-	7700 3050 7700 3150
+	7700 3550 7700 3450
+Wire Wire Line
+	3600 3150 3600 3250
 Wire Wire Line
 	6650 3550 6850 3550
 Wire Wire Line
-	3300 3000 3650 3000
-Wire Wire Line
-	3100 3000 2950 3000
+	2800 3000 3150 3000
+Wire Wire Line
+	2600 3000 2450 3000
 Wire Wire Line
 	3700 4500 3700 4750
@@
 Connection ~ 6000 6000
 Wire Wire Line
-	3350 3250 3650 3250
+	2850 3250 3150 3250
 Wire Notes Line
 	8300 4800 8300 4550
@@
 Connection ~ 7150 2200
 Wire Wire Line
-	7000 2000 7000 2200
+	7000 2200 7000 2000
 Connection ~ 7300 2200
 Wire Wire Line
-	7150 2000 7150 2200
+	7150 2200 7150 2000
 Connection ~ 6850 1600
 Wire Wire Line
@@
 Connection ~ 7150 1600
 Wire Wire Line
-	7000 1800 7000 1600
+	7000 1600 7000 1800
 Connection ~ 7300 1600
 Wire Wire Line
-	7150 1800 7150 1600
+	7150 1600 7150 1800
 Connection ~ 7400 2200
 Wire Wire Line
@@
 Connection ~ 4100 4750
 Wire Wire Line
-	4100 4900 4100 4750
+	4100 4750 4100 4900
 Connection ~ 8550 6000
 Wire Wire Line
@@
 	6850 5500 7300 5500
 Wire Wire Line
-	2050 3750 3050 3750
-Connection ~ 3650 3250
-Connection ~ 3650 3650
-Wire Wire Line
-	2000 3250 2150 3250
-Wire Wire Line
-	2000 3350 2000 3250
+	1550 3750 2550 3750
+Connection ~ 3150 3250
+Connection ~ 3150 3650
+Wire Wire Line
+	1500 3250 1650 3250
+Wire Wire Line
+	1500 3350 1500 3250
+Wire Wire Line
+	1850 3250 2050 3250
+Connection ~ 2450 3250
+Wire Wire Line
+	3150 3000 3150 3650
 Wire Wire Line
 	2350 3250 2550 3250
-Connection ~ 2950 3250
-Wire Wire Line
-	3650 3000 3650 3650
-Wire Wire Line
-	2850 3250 3050 3250
-Wire Wire Line
-	2950 3000 2950 3550
-Wire Wire Line
-	2950 3550 3050 3550
+Wire Wire Line
+	2450 3000 2450 3550
+Wire Wire Line
+	2450 3550 2550 3550
 Connection ~ 8700 4350
 Connection ~ 8700 3550
@@
 	4050 3650 4150 3650
 Wire Wire Line
-	3550 3650 3750 3650
+	3050 3650 3300 3650
 Connection ~ 4350 4750
 Wire Wire Line
-	4350 4900 4350 4750
+	4350 4750 4350 4900
 Connection ~ 3700 4750
 Wire Wire Line
@@
 Connection ~ 4350 5250
 Wire Wire Line
-	4350 5100 4350 5250
+	4350 5250 4350 5100
 Wire Wire Line
 	4600 5250 4600 5100
@@
 L CAP C2
 U 1 1 53580DA8
-P 2250 3250
-F 0 "C2" H 2280 3220 50  0000 L TNN
-F 1 "10u 6.3V" H 2280 3270 30  0000 L BNN
-F 2 "~" H 2250 3250 60  0000 C CNN
-F 3 "~" H 2250 3250 60  0000 C CNN
-	1    2250 3250
+P 1750 3250
+F 0 "C2" H 1780 3220 50  0000 L TNN
+F 1 "10u 6.3V" H 1780 3270 30  0000 L BNN
+F 2 "~" H 1750 3250 60  0000 C CNN
+F 3 "~" H 1750 3250 60  0000 C CNN
+	1    1750 3250
 	-1   0    0    1
 $EndComp
 $Comp
-L AGND_IN #PWR014
+L AGND_IN #PWR10
 U 1 1 5359DFBD
 P 4200 5450
-F 0 "#PWR014" H 4200 5450 40  0001 C CNN
+F 0 "#PWR10" H 4200 5450 40  0001 C CNN
 F 1 "AGND_IN" H 4200 5380 50  0000 C CNN
 F 2 "" H 4200 5450 60  0000 C CNN
@@
 Connection ~ 2500 5350
 $Comp
-L AGND_IN #PWR015
+L AGND_IN #PWR11
 U 1 1 535F1A3A
 P 4500 4100
-F 0 "#PWR015" H 4500 4100 40  0001 C CNN
+F 0 "#PWR11" H 4500 4100 40  0001 C CNN
 F 1 "AGND_IN" H 4500 4030 50  0000 C CNN
 F 2 "" H 4500 4100 60  0000 C CNN
@@
 $EndComp
 $Comp
-L AGND_IN #PWR016
+L AGND_IN #PWR14
 U 1 1 535F1A56
 P 6100 4100
-F 0 "#PWR016" H 6100 4100 40  0001 C CNN
+F 0 "#PWR14" H 6100 4100 40  0001 C CNN
 F 1 "AGND_IN" H 6100 4030 50  0000 C CNN
 F 2 "" H 6100 4100 60  0000 C CNN
@@
 $EndComp
 $Comp
-L AGND_IN #PWR017
+L AGND_IN #PWR6
 U 1 1 535F1C48
-P 2000 3350
-F 0 "#PWR017" H 2000 3350 40  0001 C CNN
-F 1 "AGND_IN" H 2000 3280 50  0000 C CNN
-F 2 "" H 2000 3350 60  0000 C CNN
-F 3 "" H 2000 3350 60  0000 C CNN
-	1    2000 3350
-	1    0    0    -1
-$EndComp
+P 1500 3350
+F 0 "#PWR6" H 1500 3350 40  0001 C CNN
+F 1 "AGND_IN" H 1500 3280 50  0000 C CNN
+F 2 "" H 1500 3350 60  0000 C CNN
+F 3 "" H 1500 3350 60  0000 C CNN
+	1    1500 3350
+	1    0    0    -1
+$EndComp
+$Comp
+L CAP C70
+U 1 1 53685897
+P 3400 3650
+F 0 "C70" H 3420 3620 50  0000 L TNN
+F 1 "0.01u" H 3425 3670 30  0000 L BNN
+F 2 "~" H 3400 3750 60  0000 C CNN
+F 3 "~" H 3400 3650 60  0000 C CNN
+	1    3400 3650
+	1    0    0    -1
+$EndComp
+Wire Wire Line
+	3500 3650 3750 3650
+Wire Wire Line
+	3600 3650 3600 3550
+Connection ~ 3600 3650
 $EndSCHEMATC

Commit message: Rev 2a sent off for manufacturing: Slot added instead of drill hole at audio IO end Drill added near center Fixed huge error in HP amp schematic/layout Got rid of more labels Got rid of redundant UART port. Not sure how that happened twice... Got rid of DC blocking before CODEC inputs
Parts:
- removed C16: 1u, ~, symbol CAP
Connections:
- wire segments 119 -> 117
Changed lines of the file:
@@
 Sheet 2 6
 Title "Android DPOAE Interface"
-Date "6 may 2014"
-Rev "2a"
+Date "29 jun 2014"
+Rev "2b"
 Comp "Sana AudioPulse"
 Comment1 "Ben Nahill <bnahill@gmail.com>"
@@
 $EndComp
 $Comp
-L CAP C16
-U 1 1 534E8B5E
-P 6950 3550
-F 0 "C16" H 6970 3520 50  0000 L TNN
-F 1 "1u" H 6975 3570 30  0000 L BNN
-F 2 "~" H 6950 3550 60  0000 C CNN
-F 3 "~" H 6950 3550 60  0000 C CNN
-	1    6950 3550
-	1    0    0    -1
-$EndComp
-$Comp
 L RES R15
 U 1 1 534E8F70
@@
 Wire Wire Line
 	7700 3750 7500 3750
-Connection ~ 7700 3550
-Wire Wire Line
-	7700 3550 7700 3450
 Wire Wire Line
 	3600 3150 3600 3250
-Wire Wire Line
-	6650 3550 6850 3550
 Wire Wire Line
 	2800 3000 3150 3000
@@
 	6050 3650 6150 3650
 Wire Wire Line
-	7050 3550 8200 3550
+	6650 3550 8200 3550
 Wire Wire Line
 	6050 3450 6050 3250

Commit message: Started board upgrade to 4 layers and better signal isolation
Parts:
- C10, C11, C7, C9: footprint (none) -> lib:SMD0603
- C12, C14, C21, C5: footprint ~ -> lib:SMD0805
- C13, C15, C17, C18, C23, C24, C6, C8, R10, R13, R16, R17, R18, R19, R4, R5, R6, R7, R8, R9, Rf1: footprint (none) -> lib:SMD0402
- C19, C20, C22, C3, C69, C70, R11, R12, R14, R15: footprint ~ -> lib:SMD0402
- C2: footprint ~ -> lib:SMD0603
- C4: footprint ~ -> lib:SMD1411_POL
- TP2, TP3: footprint ~ -> lib:TP_HOLE
- U1: footprint ~ -> lib:LT_DFN8_DUAL
- U2: footprint ~ -> lib:LT_DFN16_QUAD

Commit message: More routing
Parts:
- added TP13: TP, lib:TP_HOLE, symbol TP
Connections:
- wire segments 117 -> 118
Changed lines of the file:
@@
 MIC_DIFF_P
 $Comp
-L AGND_IN #PWR011
+L AGND_IN #PWR24
 U 1 1 523BB57F
 P 8100 2300
-F 0 "#PWR011" H 8100 2300 40  0001 C CNN
+F 0 "#PWR24" H 8100 2300 40  0001 C CNN
 F 1 "AGND_IN" H 8100 2230 50  0000 C CNN
 F 2 "" H 8100 2300 60  0000 C CNN
@@
 $EndComp
 $Comp
-L AGND_IN #PWR012
+L AGND_IN #PWR26
 U 1 1 523BB58F
 P 8600 2300
-F 0 "#PWR012" H 8600 2300 40  0001 C CNN
+F 0 "#PWR26" H 8600 2300 40  0001 C CNN
 F 1 "AGND_IN" H 8600 2230 50  0000 C CNN
 F 2 "" H 8600 2300 60  0000 C CNN
@@
 $EndComp
 $Comp
-L AGND_IN #PWR013
+L AGND_IN #PWR22
 U 1 1 524EBECC
 P 7400 2300
-F 0 "#PWR013" H 7400 2300 40  0001 C CNN
+F 0 "#PWR22" H 7400 2300 40  0001 C CNN
 F 1 "AGND_IN" H 7400 2230 50  0000 C CNN
 F 2 "" H 7400 2300 60  0000 C CNN
@@
 $EndComp
 $Comp
-L +5VA #PWR014
+L +5VA #PWR21
 U 1 1 524E7127
 P 7400 1500
-F 0 "#PWR014" H 7400 1630 20  0001 C CNN
+F 0 "#PWR21" H 7400 1630 20  0001 C CNN
 F 1 "+5VA" H 7400 1600 30  0000 C CNN
 F 2 "" H 7400 1500 60  0000 C CNN
@@
 $EndComp
 $Comp
-L +5VA #PWR015
+L +5VA #PWR23
 U 1 1 524E713E
 P 8100 1500
-F 0 "#PWR015" H 8100 1630 20  0001 C CNN
+F 0 "#PWR23" H 8100 1630 20  0001 C CNN
 F 1 "+5VA" H 8100 1600 30  0000 C CNN
 F 2 "" H 8100 1500 60  0000 C CNN
@@
 $EndComp
 $Comp
-L +5VA #PWR016
+L +5VA #PWR25
 U 1 1 524E7144
 P 8600 1500
-F 0 "#PWR016" H 8600 1630 20  0001 C CNN
+F 0 "#PWR25" H 8600 1630 20  0001 C CNN
 F 1 "+5VA" H 8600 1600 30  0000 C CNN
 F 2 "" H 8600 1500 60  0000 C CNN
@@
 $EndComp
 $Comp
-L AGND_IN #PWR017
+L AGND_IN #PWR13
 U 1 1 534E82DB
 P 2500 5450
-F 0 "#PWR017" H 2500 5450 40  0001 C CNN
+F 0 "#PWR13" H 2500 5450 40  0001 C CNN
 F 1 "AGND_IN" H 2500 5380 50  0000 C CNN
 F 2 "" H 2500 5450 60  0000 C CNN
@@
 $EndComp
 $Comp
-L +5VA #PWR018
+L +5VA #PWR12
 U 1 1 534E85DE
 P 2500 4350
-F 0 "#PWR018" H 2500 4480 20  0001 C CNN
+F 0 "#PWR12" H 2500 4480 20  0001 C CNN
 F 1 "+5VA" H 2500 4450 30  0000 C CNN
 F 2 "" H 2500 4350 60  0000 C CNN
@@
 	4600 4750 4600 4900
 Wire Wire Line
-	3600 4750 4600 4750
+	3600 4750 5000 4750
 Connection ~ 4350 5250
 Wire Wire Line
@@
 $EndComp
 $Comp
-L AGND_IN #PWR019
+L AGND_IN #PWR15
 U 1 1 5359DFBD
 P 4200 5450
-F 0 "#PWR019" H 4200 5450 40  0001 C CNN
+F 0 "#PWR15" H 4200 5450 40  0001 C CNN
 F 1 "AGND_IN" H 4200 5380 50  0000 C CNN
 F 2 "" H 4200 5450 60  0000 C CNN
@@
 Connection ~ 2500 5350
 $Comp
-L AGND_IN #PWR020
+L AGND_IN #PWR16
 U 1 1 535F1A3A
 P 4500 4100
-F 0 "#PWR020" H 4500 4100 40  0001 C CNN
+F 0 "#PWR16" H 4500 4100 40  0001 C CNN
 F 1 "AGND_IN" H 4500 4030 50  0000 C CNN
 F 2 "" H 4500 4100 60  0000 C CNN
@@
 $EndComp
 $Comp
-L AGND_IN #PWR021
+L AGND_IN #PWR19
 U 1 1 535F1A56
 P 6100 4100
-F 0 "#PWR021" H 6100 4100 40  0001 C CNN
+F 0 "#PWR19" H 6100 4100 40  0001 C CNN
 F 1 "AGND_IN" H 6100 4030 50  0000 C CNN
 F 2 "" H 6100 4100 60  0000 C CNN
@@
 $EndComp
 $Comp
-L AGND_IN #PWR022
+L AGND_IN #PWR11
 U 1 1 535F1C48
 P 1500 3350
-F 0 "#PWR022" H 1500 3350 40  0001 C CNN
+F 0 "#PWR11" H 1500 3350 40  0001 C CNN
 F 1 "AGND_IN" H 1500 3280 50  0000 C CNN
 F 2 "" H 1500 3350 60  0000 C CNN
@@
 	3600 3650 3600 3550
 Connection ~ 3600 3650
+$Comp
+L TP TP13
+U 1 1 57EC7B95
+P 5000 4500
+F 0 "TP13" H 5000 4400 60  0000 C CNN
+F 1 "TP" H 5000 4600 60  0000 C CNN
+F 2 "lib:TP_HOLE" H 5000 4500 60  0001 C CNN
+F 3 "~" H 5000 4500 60  0000 C CNN
+	1    5000 4500
+	0    -1   -1   0
+$EndComp
+Wire Wire Line
+	5000 4750 5000 4600
+Connection ~ 4600 4750
 $EndSCHEMATC
