File: hw/rev2/audio_in.sch (KiCad schematic (older format))
At the start: 46 parts, among them U1 LT6241, U2 LTC6242

Commit message: Simplified input processing, reduced amp count by 2
Parts:
- removed C10: 1n, lib:SMD0603, symbol CAP
- removed C11: 33n, lib:SMD0603, symbol CAP
- removed C12, C14: 10u 6.3V, lib:SMD0805, symbol CAP
- removed C21: 10u 6.3V, lib:SMD0805, symbol CPOL
- removed C23, C24: 10n, lib:SMD0402, symbol CAP
- removed R10: 4.53k (1%), lib:SMD0402, symbol RES
- removed R11, R14: 220 (1%), lib:SMD0402, symbol RES
- removed R12: 250k, lib:SMD0402, symbol RES
- removed R17: 22, lib:SMD0402, symbol RES
- removed R9: 1.4k (1%), lib:SMD0402, symbol RES
- removed U1: LT6241, lib:LT_DFN8_DUAL, symbol OPAMP_DUAL
- added C21: 1u 6.3V, lib:SMD0402, symbol CAP
- added R2, R3: 0, lib:SMD0402, symbol RES
- added TP15, TP4: TP, lib:TP_HOLE, symbol TP
- C7, C9: footprint lib:SMD0603 -> lib:SMD0402
Connections:
- net labels removed: EXT_IN
- wire segments 118 -> 92
Other:
- note added: "2nd-order Sallen-Key Chebyshev low-pass"
- note removed: "4th-order Sallen-Key Chebyshev low-pass"

Commit message: Lots of layout and grounding changes. DRC good
Parts:
- removed C4: 100u 6.3V, lib:SMD1411_POL, symbol CPOL
- removed U2: LTC6242, lib:LT_DFN16_QUAD, symbol OPAMP_QUAD
- added U1: OPAMP_QUAD, lib:LT_DFN16_QUAD, symbol OPAMP_QUAD
Connections:
- wire segments 92 -> 90
Changed lines of the file:
@@
 $EndDescr
-$Comp
-L OPAMP_QUAD U2
-U 1 1 523B0E67
-P 4750 3550
-F 0 "U2" H 4825 3400 60  0000 L CNN
-F 1 "LTC6242" H 4800 3700 60  0000 L CNN
-F 2 "lib:LT_DFN16_QUAD" H 4750 3550 60  0001 C CNN
-F 3 "~" H 4750 3550 60  0000 C CNN
-	1    4750 3550
-	1    0    0    -1
-$EndComp
-$Comp
-L OPAMP_QUAD U2
-U 4 1 523B0E7A
-P 7750 4350
-F 0 "U2" H 7825 4200 60  0000 L CNN
-F 1 "LTC6242" H 7800 4500 60  0000 L CNN
-F 2 "lib:LT_DFN16_QUAD" H 7750 4350 60  0001 C CNN
-F 3 "~" H 7750 4350 60  0000 C CNN
-	4    7750 4350
-	1    0    0    -1
-$EndComp
-$Comp
-L OPAMP_QUAD U2
-U 5 1 523B0E80
-P 8600 1850
-F 0 "U2" H 8675 1700 60  0000 L CNN
-F 1 "LTC6242" H 8650 2000 60  0000 L CNN
-F 2 "lib:LT_DFN16_QUAD" H 8600 1850 60  0001 C CNN
-F 3 "~" H 8600 1850 60  0000 C CNN
-	5    8600 1850
-	1    0    0    -1
-$EndComp
 $Comp
 L CAP C8
@@
 F 3 "" H 4750 3100 60  0000 C CNN
 	1    4750 3100
-	1    0    0    -1
-$EndComp
-$Comp
-L OPAMP_QUAD U2
-U 2 1 523B17B7
-P 2750 3650
-F 0 "U2" H 2825 3500 60  0000 L CNN
-F 1 "LTC6242" H 2800 3800 60  0000 L CNN
-F 2 "lib:LT_DFN16_QUAD" H 2750 3650 60  0001 C CNN
-F 3 "~" H 2750 3650 60  0000 C CNN
-	2    2750 3650
 	1    0    0    -1
 $EndComp
@@
 MIC_DIFF_P
 $Comp
-L AGND_IN #PWR08
-U 1 1 523BB58F
-P 8600 2300
-F 0 "#PWR08" H 8600 2300 40  0001 C CNN
-F 1 "AGND_IN" H 8600 2230 50  0000 C CNN
-F 2 "" H 8600 2300 60  0000 C CNN
-F 3 "" H 8600 2300 60  0000 C CNN
-	1    8600 2300
-	1    0    0    -1
-$EndComp
-$Comp
 L VCOM_VRT #PWR15
 U 1 1 523BBA77
@@
 	1    0    0    -1
 $EndComp
-$Comp
-L OPAMP_QUAD U2
-U 3 1 5248471B
-P 3300 4750
-F 0 "U2" H 3375 4600 60  0000 L CNN
-F 1 "LTC6242" H 3350 4900 60  0000 L CNN
-F 2 "lib:LT_DFN16_QUAD" H 3300 4750 60  0001 C CNN
-F 3 "~" H 3300 4750 60  0000 C CNN
-	3    3300 4750
-	1    0    0    -1
-$EndComp
 Text HLabel 8650 5400 2    60   Output ~ 0
 EXT_DIFF_N
@@
 	0    1    1    0
 $EndComp
-$Comp
-L AGND_IN #PWR09
-U 1 1 524EBECC
-P 7400 2300
-F 0 "#PWR09" H 7400 2300 40  0001 C CNN
-F 1 "AGND_IN" H 7400 2230 50  0000 C CNN
-F 2 "" H 7400 2300 60  0000 C CNN
-F 3 "" H 7400 2300 60  0000 C CNN
-	1    7400 2300
-	1    0    0    -1
-$EndComp
 Text Notes 6950 4950 0    40   ~ 0
 Values for unity gain
@@
 $EndComp
 $Comp
-L +5VA #PWR010
+L +5VA #PWR08
 U 1 1 524E7127
 P 7400 1500
-F 0 "#PWR010" H 7400 1630 20  0001 C CNN
+F 0 "#PWR08" H 7400 1630 20  0001 C CNN
 F 1 "+5VA" H 7400 1600 30  0000 C CNN
 F 2 "" H 7400 1500 60  0000 C CNN
@@
 $EndComp
 $Comp
-L +5VA #PWR011
+L +5VA #PWR09
 U 1 1 524E7144
-P 8600 1500
-F 0 "#PWR011" H 8600 1630 20  0001 C CNN
-F 1 "+5VA" H 8600 1600 30  0000 C CNN
-F 2 "" H 8600 1500 60  0000 C CNN
-F 3 "" H 8600 1500 60  0000 C CNN
-	1    8600 1500
+P 8250 1500
+F 0 "#PWR09" H 8250 1630 20  0001 C CNN
+F 1 "+5VA" H 8250 1600 30  0000 C CNN
+F 2 "" H 8250 1500 60  0000 C CNN
+F 3 "" H 8250 1500 60  0000 C CNN
+	1    8250 1500
 	1    0    0    -1
 $EndComp
@@
 $EndComp
 $Comp
-L AGND_IN #PWR012
-U 1 1 534E82DB
-P 2500 5450
-F 0 "#PWR012" H 2500 5450 40  0001 C CNN
-F 1 "AGND_IN" H 2500 5380 50  0000 C CNN
-F 2 "" H 2500 5450 60  0000 C CNN
-F 3 "" H 2500 5450 60  0000 C CNN
-	1    2500 5450
-	1    0    0    -1
-$EndComp
-$Comp
-L +5VA #PWR013
+L +5VA #PWR010
 U 1 1 534E85DE
 P 2500 4350
-F 0 "#PWR013" H 2500 4480 20  0001 C CNN
+F 0 "#PWR010" H 2500 4480 20  0001 C CNN
 F 1 "+5VA" H 2500 4450 30  0000 C CNN
 F 2 "" H 2500 4350 60  0000 C CNN
@@
 	0    -1   -1   0
 $EndComp
-$Comp
-L CPOL C4
-U 1 1 53580671
-P 3900 5000
-F 0 "C4" H 3930 4970 50  0000 L TNN
-F 1 "100u 6.3V" H 3930 5020 30  0000 L BNN
-F 2 "lib:SMD1411_POL" H 3900 5000 60  0001 C CNN
-F 3 "~" H 3900 5000 60  0000 C CNN
-	1    3900 5000
-	0    1    1    0
-$EndComp
-Connection ~ 4100 5250
-Wire Wire Line
-	3900 5100 3900 5250
-Connection ~ 3900 4750
-Wire Wire Line
-	3900 4750 3900 4900
 Connection ~ 7500 4050
 Wire Wire Line
@@
 	4600 5250 4600 5100
 Wire Wire Line
-	3900 5250 4600 5250
-Wire Wire Line
-	8600 2200 8600 2300
-Wire Wire Line
-	8600 1500 8600 1650
+	4100 5250 4600 5250
 $Comp
 L CAP C2
@@
 	-1   0    0    1
 $EndComp
-$Comp
-L AGND_IN #PWR014
-U 1 1 5359DFBD
-P 4200 5450
-F 0 "#PWR014" H 4200 5450 40  0001 C CNN
-F 1 "AGND_IN" H 4200 5380 50  0000 C CNN
-F 2 "" H 4200 5450 60  0000 C CNN
-F 3 "" H 4200 5450 60  0000 C CNN
-	1    4200 5450
-	1    0    0    -1
-$EndComp
 Wire Wire Line
 	4200 5450 4200 5250
@@
 Connection ~ 2500 5350
 $Comp
-L AGND_IN #PWR015
-U 1 1 535F1A3A
-P 4500 4100
-F 0 "#PWR015" H 4500 4100 40  0001 C CNN
-F 1 "AGND_IN" H 4500 4030 50  0000 C CNN
-F 2 "" H 4500 4100 60  0000 C CNN
-F 3 "" H 4500 4100 60  0000 C CNN
-	1    4500 4100
-	1    0    0    -1
-$EndComp
-$Comp
-L AGND_IN #PWR016
-U 1 1 535F1C48
-P 1500 3350
-F 0 "#PWR016" H 1500 3350 40  0001 C CNN
-F 1 "AGND_IN" H 1500 3280 50  0000 C CNN
-F 2 "" H 1500 3350 60  0000 C CNN
-F 3 "" H 1500 3350 60  0000 C CNN
-	1    1500 3350
-	1    0    0    -1
-$EndComp
-$Comp
 L CAP C70
 U 1 1 53685897
@@
 Wire Wire Line
 	8700 3550 8700 3350
+Wire Wire Line
+	8250 1500 8250 1700
+Wire Wire Line
+	8250 2300 8250 2250
+$Comp
+L OPAMP_QUAD U1
+U 1 1 58297954
+P 4750 3550
+F 0 "U1" H 4825 3400 60  0000 L CNN
+F 1 "OPAMP_QUAD" H 4800 3700 60  0000 L CNN
+F 2 "lib:LT_DFN16_QUAD" H 4750 3550 60  0001 C CNN
+F 3 "" H 4750 3550 60  0000 C CNN
+	1    4750 3550
+	1    0    0    -1
+$EndComp
+$Comp
+L OPAMP_QUAD U1
+U 2 1 58297A08
+P 2750 3650
+F 0 "U1" H 2825 3500 60  0000 L CNN
+F 1 "OPAMP_QUAD" H 2800 3800 60  0000 L CNN
+F 2 "lib:LT_DFN16_QUAD" H 2750 3650 60  0001 C CNN
+F 3 "" H 2750 3650 60  0000 C CNN
+	2    2750 3650
+	1    0    0    -1
+$EndComp
+$Comp
+L OPAMP_QUAD U1
+U 3 1 58297AFB
+P 3300 4750
+F 0 "U1" H 3375 4600 60  0000 L CNN
+F 1 "OPAMP_QUAD" H 3350 4900 60  0000 L CNN
+F 2 "lib:LT_DFN16_QUAD" H 3300 4750 60  0001 C CNN
+F 3 "" H 3300 4750 60  0000 C CNN
+	3    3300 4750
+	1    0    0    -1
+$EndComp
+$Comp
+L OPAMP_QUAD U1
+U 4 1 58297C51
+P 7750 4350
+F 0 "U1" H 7825 4200 60  0000 L CNN
+F 1 "OPAMP_QUAD" H 7800 4500 60  0000 L CNN
+F 2 "lib:LT_DFN16_QUAD" H 7750 4350 60  0001 C CNN
+F 3 "" H 7750 4350 60  0000 C CNN
+	4    7750 4350
+	1    0    0    -1
+$EndComp
+$Comp
+L OPAMP_QUAD U1
+U 5 1 58297D4A
+P 8250 1900
+F 0 "U1" H 8325 1750 60  0000 L CNN
+F 1 "OPAMP_QUAD" H 8300 2050 60  0000 L CNN
+F 2 "lib:LT_DFN16_QUAD" H 8250 1900 60  0001 C CNN
+F 3 "" H 8250 1900 60  0000 C CNN
+	5    8250 1900
+	1    0    0    -1
+$EndComp
+$Comp
+L AGND_IN #PWR011
+U 1 1 582AF8E7
+P 4200 5450
+F 0 "#PWR011" H 4200 5450 40  0001 C CNN
+F 1 "AGND_IN" H 4200 5380 50  0000 C CNN
+F 2 "" H 4200 5450 60  0000 C CNN
+F 3 "" H 4200 5450 60  0000 C CNN
+	1    4200 5450
+	1    0    0    -1
+$EndComp
+$Comp
+L AGND_IN #PWR012
+U 1 1 582AFB46
+P 2500 5450
+F 0 "#PWR012" H 2500 5450 40  0001 C CNN
+F 1 "AGND_IN" H 2500 5380 50  0000 C CNN
+F 2 "" H 2500 5450 60  0000 C CNN
+F 3 "" H 2500 5450 60  0000 C CNN
+	1    2500 5450
+	1    0    0    -1
+$EndComp
+$Comp
+L AGND_IN #PWR013
+U 1 1 582AFBCC
+P 1500 3350
+F 0 "#PWR013" H 1500 3350 40  0001 C CNN
+F 1 "AGND_IN" H 1500 3280 50  0000 C CNN
+F 2 "" H 1500 3350 60  0000 C CNN
+F 3 "" H 1500 3350 60  0000 C CNN
+	1    1500 3350
+	1    0    0    -1
+$EndComp
+$Comp
+L AGND_IN #PWR014
+U 1 1 582AFD9A
+P 4500 4100
+F 0 "#PWR014" H 4500 4100 40  0001 C CNN
+F 1 "AGND_IN" H 4500 4030 50  0000 C CNN
+F 2 "" H 4500 4100 60  0000 C CNN
+F 3 "" H 4500 4100 60  0000 C CNN
+	1    4500 4100
+	1    0    0    -1
+$EndComp
+$Comp
+L AGND_IN #PWR015
+U 1 1 582AFE20
+P 7400 2300
+F 0 "#PWR015" H 7400 2300 40  0001 C CNN
+F 1 "AGND_IN" H 7400 2230 50  0000 C CNN
+F 2 "" H 7400 2300 60  0000 C CNN
+F 3 "" H 7400 2300 60  0000 C CNN
+	1    7400 2300
+	1    0    0    -1
+$EndComp
+$Comp
+L AGND_IN #PWR016
+U 1 1 582AFEA6
+P 8250 2300
+F 0 "#PWR016" H 8250 2300 40  0001 C CNN
+F 1 "AGND_IN" H 8250 2230 50  0000 C CNN
+F 2 "" H 8250 2300 60  0000 C CNN
+F 3 "" H 8250 2300 60  0000 C CNN
+	1    8250 2300
+	1    0    0    -1
+$EndComp
 $EndSCHEMATC

Commit message: Submitted new S70 PCB
Parts:
- added C4: 1u, lib:SMD0402, symbol CAP
- added R9: 220k, lib:SMD0402, symbol RES
Connections:
- wire segments 90 -> 93
Changed lines of the file:
@@
 LIBS:contrib
 LIBS:valves
-LIBS:audio_iface_rev2-cache
 EELAYER 25 0
 EELAYER END
@@
 MIC_DIFF_P
 $Comp
-L VCOM_VRT #PWR15
+L VCOM_VRT #PWR16
 U 1 1 523BBA77
 P 7200 4450
-F 0 "#PWR15" H 7200 4650 40  0001 C CNN
+F 0 "#PWR16" H 7200 4650 40  0001 C CNN
 F 1 "VCOM_VRT" H 7200 4600 40  0000 C CNN
 F 2 "" H 7200 4450 60  0000 C CNN
@@
 $EndComp
 $Comp
-L +5VA #PWR08
+L +5VA #PWR17
 U 1 1 524E7127
 P 7400 1500
-F 0 "#PWR08" H 7400 1630 20  0001 C CNN
+F 0 "#PWR17" H 7400 1630 20  0001 C CNN
 F 1 "+5VA" H 7400 1600 30  0000 C CNN
 F 2 "" H 7400 1500 60  0000 C CNN
@@
 $EndComp
 $Comp
-L +5VA #PWR09
+L +5VA #PWR20
 U 1 1 524E7144
 P 8250 1500
-F 0 "#PWR09" H 8250 1630 20  0001 C CNN
+F 0 "#PWR20" H 8250 1630 20  0001 C CNN
 F 1 "+5VA" H 8250 1600 30  0000 C CNN
 F 2 "" H 8250 1500 60  0000 C CNN
@@
 $EndComp
 $Comp
-L +5VA #PWR010
+L +5VA #PWR9
 U 1 1 534E85DE
 P 2500 4350
-F 0 "#PWR010" H 2500 4480 20  0001 C CNN
+F 0 "#PWR9" H 2500 4480 20  0001 C CNN
 F 1 "+5VA" H 2500 4450 30  0000 C CNN
 F 2 "" H 2500 4350 60  0000 C CNN
@@
 	4450 3650 4550 3650
 Wire Wire Line
-	5050 3550 8200 3550
-Wire Wire Line
 	4450 3250 5200 3250
 Wire Wire Line
@@
 Connection ~ 4600 4750
 $Comp
-L VCOM_VRT #PWR18
+L VCOM_VRT #PWR19
 U 1 1 5828A548
 P 7900 5350
-F 0 "#PWR18" H 7900 5550 40  0001 C CNN
+F 0 "#PWR19" H 7900 5550 40  0001 C CNN
 F 1 "VCOM_VRT" H 7900 5500 40  0000 C CNN
 F 2 "" H 7900 5350 60  0000 C CNN
@@
 $EndComp
 $Comp
-L AGND_IN #PWR011
+L AGND_IN #PWR12
 U 1 1 582AF8E7
 P 4200 5450
-F 0 "#PWR011" H 4200 5450 40  0001 C CNN
+F 0 "#PWR12" H 4200 5450 40  0001 C CNN
 F 1 "AGND_IN" H 4200 5380 50  0000 C CNN
 F 2 "" H 4200 5450 60  0000 C CNN
@@
 $EndComp
 $Comp
-L AGND_IN #PWR012
+L AGND_IN #PWR10
 U 1 1 582AFB46
 P 2500 5450
-F 0 "#PWR012" H 2500 5450 40  0001 C CNN
+F 0 "#PWR10" H 2500 5450 40  0001 C CNN
 F 1 "AGND_IN" H 2500 5380 50  0000 C CNN
 F 2 "" H 2500 5450 60  0000 C CNN
@@
 $EndComp
 $Comp
-L AGND_IN #PWR013
+L AGND_IN #PWR8
 U 1 1 582AFBCC
 P 1500 3350
-F 0 "#PWR013" H 1500 3350 40  0001 C CNN
+F 0 "#PWR8" H 1500 3350 40  0001 C CNN
 F 1 "AGND_IN" H 1500 3280 50  0000 C CNN
 F 2 "" H 1500 3350 60  0000 C CNN
@@
 $EndComp
 $Comp
-L AGND_IN #PWR014
+L AGND_IN #PWR13
 U 1 1 582AFD9A
 P 4500 4100
-F 0 "#PWR014" H 4500 4100 40  0001 C CNN
+F 0 "#PWR13" H 4500 4100 40  0001 C CNN
 F 1 "AGND_IN" H 4500 4030 50  0000 C CNN
 F 2 "" H 4500 4100 60  0000 C CNN
@@
 $EndComp
 $Comp
-L AGND_IN #PWR015
+L AGND_IN #PWR18
 U 1 1 582AFE20
 P 7400 2300
-F 0 "#PWR015" H 7400 2300 40  0001 C CNN
+F 0 "#PWR18" H 7400 2300 40  0001 C CNN
 F 1 "AGND_IN" H 7400 2230 50  0000 C CNN
 F 2 "" H 7400 2300 60  0000 C CNN
@@
 $EndComp
 $Comp
-L AGND_IN #PWR016
+L AGND_IN #PWR21
 U 1 1 582AFEA6
 P 8250 2300
-F 0 "#PWR016" H 8250 2300 40  0001 C CNN
+F 0 "#PWR21" H 8250 2300 40  0001 C CNN
 F 1 "AGND_IN" H 8250 2230 50  0000 C CNN
 F 2 "" H 8250 2300 60  0000 C CNN
@@
 	1    0    0    -1
 $EndComp
+$Comp
+L CAP C4
+U 1 1 582BE3E0
+P 5450 3550
+F 0 "C4" H 5470 3520 50  0000 L TNN
+F 1 "1u" H 5475 3570 30  0000 L BNN
+F 2 "lib:SMD0402" H 5450 3550 60  0001 C CNN
+F 3 "" H 5450 3550 60  0000 C CNN
+	1    5450 3550
+	1    0    0    -1
+$EndComp
+$Comp
+L RES R9
+U 1 1 582BE489
+P 5650 3800
+F 0 "R9" H 5720 3765 50  0000 L TNN
+F 1 "220k" H 5650 3855 30  0000 C BNN
+F 2 "lib:SMD0402" H 5650 3800 60  0001 C CNN
+F 3 "" H 5650 3800 60  0000 C CNN
+	1    5650 3800
+	0    1    1    0
+$EndComp
+Wire Wire Line
+	5050 3550 5350 3550
+Wire Wire Line
+	5550 3550 8200 3550
+Wire Wire Line
+	5650 3650 5650 3550
+Connection ~ 5650 3550
+Wire Wire Line
+	5650 3950 5650 4050
+$Comp
+L AGND_IN #PWR15
+U 1 1 582BE840
+P 5650 4050
+F 0 "#PWR15" H 5650 4050 40  0001 C CNN
+F 1 "AGND_IN" H 5650 3980 50  0000 C CNN
+F 2 "" H 5650 4050 60  0000 C CNN
+F 3 "" H 5650 4050 60  0000 C CNN
+	1    5650 4050
+	1    0    0    -1
+$EndComp

Commit message: Fixed power connections for S70--submitted PCB
Parts:
- C19: footprint lib:SMD0402 -> lib:SMD1411_POL
- C2: footprint lib:SMD0603 -> lib:SMD0805
Changed lines of the file:
@@
 LIBS:contrib
 LIBS:valves
+LIBS:audio_iface_rev2-cache
 EELAYER 25 0
 EELAYER END
@@
 F 0 "C19" H 7330 1870 50  0000 L TNN
 F 1 "100u 6.3V" H 7330 1920 30  0000 L BNN
-F 2 "lib:SMD0402" H 7300 1900 60  0001 C CNN
+F 2 "lib:SMD1411_POL" H 7300 1900 60  0001 C CNN
 F 3 "~" H 7300 1900 60  0000 C CNN
 	1    7300 1900
@@
 F 0 "C2" H 1780 3220 50  0000 L TNN
 F 1 "10u 6.3V" H 1780 3270 30  0000 L BNN
-F 2 "lib:SMD0603" H 1750 3250 60  0001 C CNN
+F 2 "lib:SMD0805" H 1750 3250 60  0001 C CNN
 F 3 "~" H 1750 3250 60  0000 C CNN
 	1    1750 3250
