File: hw/rev2/audio_in.sch (KiCad schematic (older format))
At the start: 46 parts, among them U1 LT6241, U2 LTC6242

Commit message: Most of a schematic
Parts:
- C10, C11, C12, C13, C14, C15, C17, C18, C2, C20, C22, C23, C24, C3, C6, C69, C7, C70, C8, C9: symbol CAP -> symbols:CAP
- C19, C21, C4, C5: symbol CPOL -> symbols:CPOL
- R10, R11, R12, R13, R14, R15, R16, R17, R18, R19, R4, R5, R6, R7, R8, R9, Rf1: symbol RES -> symbols:RES
- TP13, TP2, TP3: symbol TP -> symbols:TP
- U1: symbol OPAMP_DUAL -> symbols:OPAMP_DUAL
- U2: symbol OPAMP_QUAD -> symbols:OPAMP_QUAD
