File: hw/rev2/codec.sch (KiCad schematic (older format))
At the start: 6 parts, among them U301 AK4621

Commit message: Lots of things: --Added RGB LED on timer outputs --Input: Moved capacitively coupled feedback nodes from vgnd to gnd --Output: LTC6242 for filtering to amplifier --Power: 2-stage supply for analog: USB 5V boost to 6V, LDO to 5V   Digital still using LDO from USB 5V and not caring about anyone   Bonus! Can completely shut off analog portion of board --Layout and routing: All of it TODO: final checks on layout and LVS (vs simulation) HEAD2HEAD2HEAD! TODO: adjust silkscreen, add logo TODO: debate adding 12.288MHz dedicated crystal
Parts:
- removed SB301: SB_2-1, ~, symbol SB_2-1
- renumbered C301 to C25, C302 to C26, C303 to C27, C304 to C28, U301 to U3
Connections:
- wire segments 51 -> 50
Changed lines of the file:
@@
 Sheet 3 6
 Title "Android DPOAE Interface"
-Date "22 apr 2014"
+Date "3 may 2014"
 Rev "2a"
 Comp "Sana AudioPulse"
@@
 $EndDescr
 $Comp
-L AK4621 U301
+L AK4621 U3
 U 1 1 523B94A4
 P 5100 3350
-F 0 "U301" H 5100 2300 60  0000 C CNN
+F 0 "U3" H 5100 2300 60  0000 C CNN
 F 1 "AK4621" H 5100 3900 60  0000 C CNN
 F 2 "" H 5100 3350 60  0000 C CNN
@@
 $EndComp
 $Comp
-L CAP C302
+L CAP C26
 U 1 1 523B94B1
 P 2700 3600
-F 0 "C302" H 2720 3570 50  0000 L TNN
+F 0 "C26" H 2720 3570 50  0000 L TNN
 F 1 "0.1u" H 2725 3620 30  0000 L BNN
 F 2 "" H 2700 3600 60  0000 C CNN
@@
 $EndComp
 $Comp
-L CAP C301
+L CAP C25
 U 1 1 523B94B7
 P 2550 3600
-F 0 "C301" H 2570 3570 50  0000 L TNN
+F 0 "C25" H 2570 3570 50  0000 L TNN
 F 1 "1u" H 2575 3620 30  0000 L BNN
 F 2 "" H 2550 3600 60  0000 C CNN
@@
 AOUTL-
 $Comp
-L DGND #PWR023
+L DGND #PWR018
 U 1 1 523B95EE
 P 7900 3400
-F 0 "#PWR023" H 7900 3400 40  0001 C CNN
+F 0 "#PWR018" H 7900 3400 40  0001 C CNN
 F 1 "DGND" H 7900 3330 40  0000 C CNN
 F 2 "" H 7900 3400 60  0000 C CNN
@@
 	7900 3300 7900 3400
 $Comp
-L CAP C304
+L CAP C28
 U 1 1 523B9668
 P 4200 2700
-F 0 "C304" H 4220 2670 50  0000 L TNN
+F 0 "C28" H 4220 2670 50  0000 L TNN
 F 1 "0.1u" H 4225 2720 30  0000 L BNN
 F 2 "" H 4200 2700 60  0000 C CNN
@@
 $EndComp
 $Comp
-L CAP C303
+L CAP C27
 U 1 1 523B9675
 P 4000 2700
-F 0 "C303" H 4020 2670 50  0000 L TNN
+F 0 "C27" H 4020 2670 50  0000 L TNN
 F 1 "10u" H 4025 2720 30  0000 L BNN
 F 2 "" H 4000 2700 60  0000 C CNN
@@
 	2450 3350 2450 3400
 $Comp
-L +3V #PWR024
+L +3V #PWR019
 U 1 1 524DAE69
 P 7700 3450
-F 0 "#PWR024" H 7700 3410 30  0001 C CNN
+F 0 "#PWR019" H 7700 3410 30  0001 C CNN
 F 1 "+3V" H 7700 3560 30  0000 C CNN
 F 2 "~" H 7700 3450 60  0000 C CNN
@@
 	5700 3800 6250 3800
 Wire Wire Line
-	5700 3900 8100 3900
+	5700 3900 8200 3900
 NoConn ~ 5700 4300
 NoConn ~ 4500 4300
 $Comp
-L +5V #PWR025
+L +5V #PWR020
 U 1 1 524DADF1
 P 7600 3550
-F 0 "#PWR025" H 7600 3640 20  0001 C CNN
+F 0 "#PWR020" H 7600 3640 20  0001 C CNN
 F 1 "+5V" H 7600 3640 30  0000 C CNN
 F 2 "" H 7600 3550 60  0000 C CNN
@@
 $EndComp
 $Comp
-L +5VA #PWR026
+L +5VA #PWR021
 U 1 1 524E470F
 P 2450 3350
-F 0 "#PWR026" H 2450 3480 20  0001 C CNN
+F 0 "#PWR021" H 2450 3480 20  0001 C CNN
 F 1 "+5VA" H 2450 3450 30  0000 C CNN
 F 2 "" H 2450 3350 60  0000 C CNN
@@
 $EndComp
 $Comp
-L +5VA #PWR027
+L +5VA #PWR022
 U 1 1 524E4726
 P 3450 3950
-F 0 "#PWR027" H 3450 4080 20  0001 C CNN
+F 0 "#PWR022" H 3450 4080 20  0001 C CNN
 F 1 "+5VA" H 3450 4050 30  0000 C CNN
 F 2 "" H 3450 3950 60  0000 C CNN
@@
 	3600 4150 3600 3700
 $Comp
-L AGND_OUT #PWR028
+L AGND_OUT #PWR023
 U 1 1 524E577E
 P 2800 3850
-F 0 "#PWR028" H 2800 3850 40  0001 C CNN
+F 0 "#PWR023" H 2800 3850 40  0001 C CNN
 F 1 "AGND_OUT" H 2800 3780 50  0000 C CNN
 F 2 "~" H 2800 3850 60  0000 C CNN
@@
 $EndComp
 $Comp
-L AGND_OUT #PWR029
+L AGND_OUT #PWR024
 U 1 1 524E579A
 P 4100 2900
-F 0 "#PWR029" H 4100 2900 40  0001 C CNN
+F 0 "#PWR024" H 4100 2900 40  0001 C CNN
 F 1 "AGND_OUT" H 4100 2830 50  0000 C CNN
 F 2 "~" H 4100 2900 60  0000 C CNN
@@
 $EndComp
 $Comp
-L AGND_OUT #PWR030
+L AGND_OUT #PWR025
 U 1 1 5257A82B
 P 3600 4150
-F 0 "#PWR030" H 3600 4150 40  0001 C CNN
+F 0 "#PWR025" H 3600 4150 40  0001 C CNN
 F 1 "AGND_OUT" H 3600 4080 50  0000 C CNN
 F 2 "~" H 3600 4150 60  0000 C CNN
@@
 SPI_MOSI
 $Comp
-L SB_2-1 SB301
-U 1 1 5257A840
-P 8200 3900
-F 0 "SB301" H 8200 3800 60  0000 L CNN
-F 1 "SB_2-1" H 8200 3950 60  0000 L CNN
-F 2 "~" H 8200 3900 60  0000 C CNN
-F 3 "~" H 8200 3900 60  0000 C CNN
-	1    8200 3900
-	1    0    0    -1
-$EndComp
-$Comp
-L DGND #PWR031
+L DGND #PWR026
 U 1 1 5257A84F
 P 8200 4150
-F 0 "#PWR031" H 8200 4150 40  0001 C CNN
+F 0 "#PWR026" H 8200 4150 40  0001 C CNN
 F 1 "DGND" H 8200 4080 40  0000 C CNN
 F 2 "" H 8200 4150 60  0000 C CNN
@@
 $EndComp
 Wire Wire Line
-	8200 4150 8200 4050
-$Comp
-L +3V #PWR032
-U 1 1 5257A89B
-P 8200 3650
-F 0 "#PWR032" H 8200 3610 30  0001 C CNN
-F 1 "+3V" H 8200 3760 30  0000 C CNN
-F 2 "~" H 8200 3650 60  0000 C CNN
-F 3 "~" H 8200 3650 60  0000 C CNN
-	1    8200 3650
-	1    0    0    -1
-$EndComp
-Wire Wire Line
-	8200 3650 8200 3750
-$Comp
-L DGND #PWR033
+	8200 3900 8200 4150
+$Comp
+L DGND #PWR027
 U 1 1 5257AAC8
 P 6750 3750
-F 0 "#PWR033" H 6750 3750 40  0001 C CNN
+F 0 "#PWR027" H 6750 3750 40  0001 C CNN
 F 1 "DGND" H 6750 3680 40  0000 C CNN
 F 2 "" H 6750 3750 60  0000 C CNN

Commit message: Started board upgrade to 4 layers and better signal isolation
Parts:
- C25, C26, C28: footprint (none) -> lib:SMD0402
- C27: footprint (none) -> lib:SMD0805
- U3: footprint (none) -> lib:AK4621_VSOP30
Connections:
- net labels added: GNDD
- net labels removed: DGND
Changed lines of the file:
@@
 LIBS:memory
 LIBS:xilinx
-LIBS:special
 LIBS:microcontrollers
 LIBS:dsp
@@
 LIBS:valves
 LIBS:audio_iface_rev2-cache
-EELAYER 27 0
+EELAYER 25 0
 EELAYER END
 $Descr A 11000 8500
@@
 F 0 "U3" H 5100 2300 60  0000 C CNN
 F 1 "AK4621" H 5100 3900 60  0000 C CNN
-F 2 "" H 5100 3350 60  0000 C CNN
+F 2 "lib:AK4621_VSOP30" H 5100 3350 60  0001 C CNN
 F 3 "" H 5100 3350 60  0000 C CNN
 	1    5100 3350
@@
 F 0 "C26" H 2720 3570 50  0000 L TNN
 F 1 "0.1u" H 2725 3620 30  0000 L BNN
-F 2 "" H 2700 3600 60  0000 C CNN
+F 2 "lib:SMD0402" H 2700 3600 60  0001 C CNN
 F 3 "" H 2700 3600 60  0000 C CNN
 	1    2700 3600
@@
 F 0 "C25" H 2570 3570 50  0000 L TNN
 F 1 "1u" H 2575 3620 30  0000 L BNN
-F 2 "" H 2550 3600 60  0000 C CNN
+F 2 "lib:SMD0402" H 2550 3600 60  0001 C CNN
 F 3 "" H 2550 3600 60  0000 C CNN
 	1    2550 3600
@@
 Text HLabel 6300 3200 2    60   Output ~ 0
 AOUTL-
-$Comp
-L DGND #PWR33
-U 1 1 523B95EE
-P 7900 3400
-F 0 "#PWR33" H 7900 3400 40  0001 C CNN
-F 1 "DGND" H 7900 3330 40  0000 C CNN
-F 2 "" H 7900 3400 60  0000 C CNN
-F 3 "" H 7900 3400 60  0000 C CNN
-	1    7900 3400
-	1    0    0    -1
-$EndComp
 Wire Wire Line
 	7900 3300 7900 3400
@@
 F 0 "C28" H 4220 2670 50  0000 L TNN
 F 1 "0.1u" H 4225 2720 30  0000 L BNN
-F 2 "" H 4200 2700 60  0000 C CNN
+F 2 "lib:SMD0402" H 4200 2700 60  0001 C CNN
 F 3 "" H 4200 2700 60  0000 C CNN
 	1    4200 2700
@@
 F 0 "C27" H 4020 2670 50  0000 L TNN
 F 1 "10u" H 4025 2720 30  0000 L BNN
-F 2 "" H 4000 2700 60  0000 C CNN
+F 2 "lib:SMD0805" H 4000 2700 60  0001 C CNN
 F 3 "" H 4000 2700 60  0000 C CNN
 	1    4000 2700
@@
 	2450 3350 2450 3400
 $Comp
-L +3V #PWR32
+L +3V #PWR023
 U 1 1 524DAE69
 P 7700 3450
-F 0 "#PWR32" H 7700 3410 30  0001 C CNN
+F 0 "#PWR023" H 7700 3410 30  0001 C CNN
 F 1 "+3V" H 7700 3560 30  0000 C CNN
 F 2 "~" H 7700 3450 60  0000 C CNN
@@
 NoConn ~ 4500 4300
 $Comp
-L +5V #PWR31
+L +5V #PWR024
 U 1 1 524DADF1
 P 7600 3550
-F 0 "#PWR31" H 7600 3640 20  0001 C CNN
+F 0 "#PWR024" H 7600 3640 20  0001 C CNN
 F 1 "+5V" H 7600 3640 30  0000 C CNN
 F 2 "" H 7600 3550 60  0000 C CNN
@@
 $EndComp
 $Comp
-L +5VA #PWR25
+L +5VA #PWR025
 U 1 1 524E470F
 P 2450 3350
-F 0 "#PWR25" H 2450 3480 20  0001 C CNN
+F 0 "#PWR025" H 2450 3480 20  0001 C CNN
 F 1 "+5VA" H 2450 3450 30  0000 C CNN
 F 2 "" H 2450 3350 60  0000 C CNN
@@
 $EndComp
 $Comp
-L +5VA #PWR27
+L +5VA #PWR026
 U 1 1 524E4726
 P 3450 3950
-F 0 "#PWR27" H 3450 4080 20  0001 C CNN
+F 0 "#PWR026" H 3450 4080 20  0001 C CNN
 F 1 "+5VA" H 3450 4050 30  0000 C CNN
 F 2 "" H 3450 3950 60  0000 C CNN
@@
 	3600 4150 3600 3700
 $Comp
-L AGND_OUT #PWR26
+L AGND_OUT #PWR027
 U 1 1 524E577E
 P 2800 3850
-F 0 "#PWR26" H 2800 3850 40  0001 C CNN
+F 0 "#PWR027" H 2800 3850 40  0001 C CNN
 F 1 "AGND_OUT" H 2800 3780 50  0000 C CNN
 F 2 "~" H 2800 3850 60  0000 C CNN
@@
 $EndComp
 $Comp
-L AGND_OUT #PWR29
+L AGND_OUT #PWR028
 U 1 1 524E579A
 P 4100 2900
-F 0 "#PWR29" H 4100 2900 40  0001 C CNN
+F 0 "#PWR028" H 4100 2900 40  0001 C CNN
 F 1 "AGND_OUT" H 4100 2830 50  0000 C CNN
 F 2 "~" H 4100 2900 60  0000 C CNN
@@
 $EndComp
 $Comp
-L AGND_OUT #PWR28
+L AGND_OUT #PWR029
 U 1 1 5257A82B
 P 3600 4150
-F 0 "#PWR28" H 3600 4150 40  0001 C CNN
+F 0 "#PWR029" H 3600 4150 40  0001 C CNN
 F 1 "AGND_OUT" H 3600 4080 50  0000 C CNN
 F 2 "~" H 3600 4150 60  0000 C CNN
@@
 Text HLabel 6900 4200 2    60   Input ~ 0
 SPI_MOSI
-$Comp
-L DGND #PWR34
-U 1 1 5257A84F
-P 8200 4150
-F 0 "#PWR34" H 8200 4150 40  0001 C CNN
-F 1 "DGND" H 8200 4080 40  0000 C CNN
-F 2 "" H 8200 4150 60  0000 C CNN
-F 3 "" H 8200 4150 60  0000 C CNN
-	1    8200 4150
-	1    0    0    -1
-$EndComp
 Wire Wire Line
 	8200 3900 8200 4150
-$Comp
-L DGND #PWR30
-U 1 1 5257AAC8
-P 6750 3750
-F 0 "#PWR30" H 6750 3750 40  0001 C CNN
-F 1 "DGND" H 6750 3680 40  0000 C CNN
-F 2 "" H 6750 3750 60  0000 C CNN
-F 3 "" H 6750 3750 60  0000 C CNN
-	1    6750 3750
-	1    0    0    -1
-$EndComp
 Wire Wire Line
 	6750 3750 6750 3600
@@
 	5700 3700 6750 3700
 Connection ~ 6750 3700
+$Comp
+L GNDD #PWR030
+U 1 1 57D656B3
+P 7900 3400
+F 0 "#PWR030" H 7900 3150 50  0001 C CNN
+F 1 "GNDD" H 7900 3250 50  0000 C CNN
+F 2 "" H 7900 3400 50  0000 C CNN
+F 3 "" H 7900 3400 50  0000 C CNN
+	1    7900 3400
+	1    0    0    -1
+$EndComp
+$Comp
+L GNDD #PWR031
+U 1 1 57D656EE
+P 8200 4150
+F 0 "#PWR031" H 8200 3900 50  0001 C CNN
+F 1 "GNDD" H 8200 4000 50  0000 C CNN
+F 2 "" H 8200 4150 50  0000 C CNN
+F 3 "" H 8200 4150 50  0000 C CNN
+	1    8200 4150
+	1    0    0    -1
+$EndComp
+$Comp
+L GNDD #PWR032
+U 1 1 57D65722
+P 6750 3750
+F 0 "#PWR032" H 6750 3500 50  0001 C CNN
+F 1 "GNDD" H 6750 3600 50  0000 C CNN
+F 2 "" H 6750 3750 50  0000 C CNN
+F 3 "" H 6750 3750 50  0000 C CNN
+	1    6750 3750
+	1    0    0    -1
+$EndComp
 $EndSCHEMATC
