File: hw/rev2/codec.sch (KiCad schematic (older format))
At the start: 5 parts, among them U3 AK4621

Commit message: Lots of layout and grounding changes. DRC good
Parts:
- added FB7: BLM18PG221SN1D, lib:SMD0805, symbol FB
- C25: value 1u -> 10u; footprint lib:SMD0402 -> lib:SMD0805
Connections:
- net labels added: AGND_IN
- net labels removed: AGND_OUT, GNDD
Changed lines of the file:
@@
 P 2550 3600
 F 0 "C25" H 2570 3570 50  0000 L TNN
-F 1 "1u" H 2575 3620 30  0000 L BNN
-F 2 "lib:SMD0402" H 2550 3600 60  0001 C CNN
+F 1 "10u" H 2575 3620 30  0000 L BNN
+F 2 "lib:SMD0805" H 2550 3600 60  0001 C CNN
 F 3 "" H 2550 3600 60  0000 C CNN
 	1    2550 3600
 	0    -1   -1   0
 $EndComp
-Wire Wire Line
-	3450 3600 4500 3600
-Wire Wire Line
-	6300 2900 5700 2900
-Wire Wire Line
-	5700 3000 6300 3000
-Wire Wire Line
-	6300 3100 5700 3100
-Wire Wire Line
-	5700 3200 6300 3200
-Wire Wire Line
-	4500 3100 3100 3100
-Wire Wire Line
-	3100 3000 4500 3000
-Wire Wire Line
-	5700 3300 7900 3300
-Wire Wire Line
-	2800 3500 2800 3850
-Wire Wire Line
-	2800 3500 4500 3500
-Wire Wire Line
-	2550 3800 2800 3800
-Wire Wire Line
-	2550 3800 2550 3700
-Connection ~ 2800 3800
-Wire Wire Line
-	2550 3500 2550 3400
-Wire Wire Line
-	2450 3400 4500 3400
-Wire Wire Line
-	2700 3400 2700 3500
-Connection ~ 2700 3400
-Wire Wire Line
-	2700 3700 2700 3800
-Connection ~ 2700 3800
-Connection ~ 2550 3400
 Text HLabel 3100 3200 0    60   Input ~ 0
 AINL+
@@
 Text HLabel 3100 3100 0    60   Input ~ 0
 AINR-
-Wire Wire Line
-	3100 3200 4500 3200
-Wire Wire Line
-	4500 3300 3100 3300
 Text HLabel 6300 2900 2    60   Output ~ 0
 AOUTR+
@@
 Text HLabel 6300 3200 2    60   Output ~ 0
 AOUTL-
-Wire Wire Line
-	7900 3300 7900 3400
 $Comp
 L CAP C28
@@
 	0    -1   -1   0
 $EndComp
-Wire Wire Line
-	4500 2900 4400 2900
-Wire Wire Line
-	4400 2900 4400 2500
-Wire Wire Line
-	4400 2500 4000 2500
-Wire Wire Line
-	4000 2500 4000 2600
-Wire Wire Line
-	4200 2600 4200 2500
-Connection ~ 4200 2500
-Wire Wire Line
-	4100 2900 4100 2850
-Wire Wire Line
-	4000 2850 4200 2850
-Wire Wire Line
-	4200 2850 4200 2800
-Wire Wire Line
-	4000 2850 4000 2800
-Connection ~ 4100 2850
 Text HLabel 4100 3800 0    60   Input ~ 0
 MCLK
@@
 Text HLabel 4100 4100 0    60   Output ~ 0
 SDTO
-Wire Wire Line
-	4100 3800 4500 3800
-Wire Wire Line
-	4500 3900 4100 3900
-Wire Wire Line
-	4100 4000 4500 4000
-Wire Wire Line
-	4500 4100 4100 4100
-Wire Wire Line
-	4100 4200 4500 4200
-Wire Wire Line
-	3600 3700 4500 3700
-Wire Wire Line
-	2450 3350 2450 3400
 $Comp
 L +3V #PWR017
@@
 	-1   0    0    1
 $EndComp
-Wire Wire Line
-	5700 3400 7700 3400
-Wire Wire Line
-	7700 3400 7700 3450
-Wire Wire Line
-	7600 3550 7600 3500
-Wire Wire Line
-	7600 3500 5700 3500
 Text Notes 3650 3700 0    40   ~ 0
 Serial Mode
 Text HLabel 6250 3800 2    60   Input ~ 0
 PDN
-Wire Wire Line
-	5700 4200 6900 4200
-Wire Wire Line
-	5700 4100 6900 4100
-Wire Wire Line
-	5700 4000 6900 4000
-Wire Wire Line
-	5700 3800 6250 3800
-Wire Wire Line
-	5700 3900 8200 3900
 NoConn ~ 5700 4300
 NoConn ~ 4500 4300
@@
 $Comp
 L +5VA #PWR019
-U 1 1 524E470F
-P 2450 3350
-F 0 "#PWR019" H 2450 3480 20  0001 C CNN
-F 1 "+5VA" H 2450 3450 30  0000 C CNN
-F 2 "" H 2450 3350 60  0000 C CNN
-F 3 "" H 2450 3350 60  0000 C CNN
-	1    2450 3350
-	1    0    0    -1
-$EndComp
-$Comp
-L +5VA #PWR020
 U 1 1 524E4726
-P 3450 3950
-F 0 "#PWR020" H 3450 4080 20  0001 C CNN
-F 1 "+5VA" H 3450 4050 30  0000 C CNN
-F 2 "" H 3450 3950 60  0000 C CNN
-F 3 "" H 3450 3950 60  0000 C CNN
-	1    3450 3950
+P 3450 4750
+F 0 "#PWR019" H 3450 4880 20  0001 C CNN
+F 1 "+5VA" H 3450 4850 30  0000 C CNN
+F 2 "" H 3450 4750 60  0000 C CNN
+F 3 "" H 3450 4750 60  0000 C CNN
+	1    3450 4750
 	-1   0    0    1
-$EndComp
-Wire Wire Line
-	3450 3600 3450 3950
-Wire Wire Line
-	3600 4150 3600 3700
-$Comp
-L AGND_OUT #PWR021
-U 1 1 524E577E
-P 2800 3850
-F 0 "#PWR021" H 2800 3850 40  0001 C CNN
-F 1 "AGND_OUT" H 2800 3780 50  0000 C CNN
-F 2 "~" H 2800 3850 60  0000 C CNN
-F 3 "~" H 2800 3850 60  0000 C CNN
-	1    2800 3850
-	1    0    0    -1
-$EndComp
-$Comp
-L AGND_OUT #PWR022
-U 1 1 524E579A
-P 4100 2900
-F 0 "#PWR022" H 4100 2900 40  0001 C CNN
-F 1 "AGND_OUT" H 4100 2830 50  0000 C CNN
-F 2 "~" H 4100 2900 60  0000 C CNN
-F 3 "~" H 4100 2900 60  0000 C CNN
-	1    4100 2900
-	1    0    0    -1
-$EndComp
-$Comp
-L AGND_OUT #PWR023
-U 1 1 5257A82B
-P 3600 4150
-F 0 "#PWR023" H 3600 4150 40  0001 C CNN
-F 1 "AGND_OUT" H 3600 4080 50  0000 C CNN
-F 2 "~" H 3600 4150 60  0000 C CNN
-F 3 "~" H 3600 4150 60  0000 C CNN
-	1    3600 4150
-	1    0    0    -1
 $EndComp
 Text HLabel 6900 4100 2    60   Input ~ 0
@@
 Text HLabel 6900 4200 2    60   Input ~ 0
 SPI_MOSI
+$Comp
+L AGND_IN #PWR020
+U 1 1 582ADE41
+P 7900 3400
+F 0 "#PWR020" H 7900 3400 40  0001 C CNN
+F 1 "AGND_IN" H 7900 3330 50  0000 C CNN
+F 2 "" H 7900 3400 60  0000 C CNN
+F 3 "" H 7900 3400 60  0000 C CNN
+	1    7900 3400
+	1    0    0    -1
+$EndComp
+$Comp
+L AGND_IN #PWR021
+U 1 1 582AE1DB
+P 2800 3850
+F 0 "#PWR021" H 2800 3850 40  0001 C CNN
+F 1 "AGND_IN" H 2800 3780 50  0000 C CNN
+F 2 "" H 2800 3850 60  0000 C CNN
+F 3 "" H 2800 3850 60  0000 C CNN
+	1    2800 3850
+	1    0    0    -1
+$EndComp
+$Comp
+L AGND_IN #PWR022
+U 1 1 582AE264
+P 4100 2900
+F 0 "#PWR022" H 4100 2900 40  0001 C CNN
+F 1 "AGND_IN" H 4100 2830 50  0000 C CNN
+F 2 "" H 4100 2900 60  0000 C CNN
+F 3 "" H 4100 2900 60  0000 C CNN
+	1    4100 2900
+	1    0    0    -1
+$EndComp
+$Comp
+L FB FB7
+U 1 1 582B4FC8
+P 3450 4500
+F 0 "FB7" H 3520 4465 50  0000 L TNN
+F 1 "BLM18PG221SN1D" H 3385 4575 30  0000 C BNN
+F 2 "lib:SMD0805" H 3430 4520 60  0001 C CNN
+F 3 "" H 3430 4520 60  0000 C CNN
+	1    3450 4500
+	0    1    1    0
+$EndComp
+Wire Wire Line
+	3450 3600 4500 3600
+Wire Wire Line
+	6300 2900 5700 2900
+Wire Wire Line
+	5700 3000 6300 3000
+Wire Wire Line
+	6300 3100 5700 3100
+Wire Wire Line
+	5700 3200 6300 3200
+Wire Wire Line
+	4500 3100 3100 3100
+Wire Wire Line
+	3100 3000 4500 3000
+Wire Wire Line
+	5700 3300 7900 3300
+Wire Wire Line
+	2800 3500 2800 3850
+Wire Wire Line
+	2800 3500 4500 3500
+Wire Wire Line
+	2550 3800 2800 3800
+Wire Wire Line
+	2550 3800 2550 3700
+Connection ~ 2800 3800
+Wire Wire Line
+	2550 3500 2550 3400
+Wire Wire Line
+	2700 3400 2700 3500
+Connection ~ 2700 3400
+Wire Wire Line
+	2700 3700 2700 3800
+Connection ~ 2700 3800
+Wire Wire Line
+	3100 3200 4500 3200
+Wire Wire Line
+	4500 3300 3100 3300
+Wire Wire Line
+	7900 3300 7900 3400
+Wire Wire Line
+	4500 2900 4400 2900
+Wire Wire Line
+	4400 2900 4400 2500
+Wire Wire Line
+	4400 2500 4000 2500
+Wire Wire Line
+	4000 2500 4000 2600
+Wire Wire Line
+	4200 2600 4200 2500
+Connection ~ 4200 2500
+Wire Wire Line
+	4100 2900 4100 2850
+Wire Wire Line
+	4000 2850 4200 2850
+Wire Wire Line
+	4200 2850 4200 2800
+Wire Wire Line
+	4000 2850 4000 2800
+Connection ~ 4100 2850
+Wire Wire Line
+	4100 3800 4500 3800
+Wire Wire Line
+	4500 3900 4100 3900
+Wire Wire Line
+	4100 4000 4500 4000
+Wire Wire Line
+	4500 4100 4100 4100
+Wire Wire Line
+	4100 4200 4500 4200
+Wire Wire Line
+	3600 3700 4500 3700
+Wire Wire Line
+	5700 3400 7700 3400
+Wire Wire Line
+	7700 3400 7700 3450
+Wire Wire Line
+	7600 3550 7600 3500
+Wire Wire Line
+	7600 3500 5700 3500
+Wire Wire Line
+	5700 4200 6900 4200
+Wire Wire Line
+	5700 4100 6900 4100
+Wire Wire Line
+	5700 4000 6900 4000
+Wire Wire Line
+	5700 3800 6250 3800
+Wire Wire Line
+	5700 3900 8200 3900
+Wire Wire Line
+	3450 3400 3450 4350
+Wire Wire Line
+	3600 4150 3600 3700
 Wire Wire Line
 	8200 3900 8200 4150
 Wire Wire Line
-	6750 3750 6750 3600
+	6750 3600 6750 3750
 Wire Wire Line
 	6750 3600 5700 3600
@@
 	5700 3700 6750 3700
 Connection ~ 6750 3700
-$Comp
-L GNDD #PWR024
-U 1 1 57D656B3
-P 7900 3400
-F 0 "#PWR024" H 7900 3150 50  0001 C CNN
-F 1 "GNDD" H 7900 3250 50  0000 C CNN
-F 2 "" H 7900 3400 50  0000 C CNN
-F 3 "" H 7900 3400 50  0000 C CNN
-	1    7900 3400
-	1    0    0    -1
-$EndComp
-$Comp
-L GNDD #PWR025
-U 1 1 57D656EE
+Wire Wire Line
+	3450 4750 3450 4650
+Wire Wire Line
+	2550 3400 4500 3400
+Connection ~ 3450 3400
+Connection ~ 3450 3600
+$Comp
+L AGND_IN #PWR024
+U 1 1 582B627B
+P 6750 3750
+F 0 "#PWR024" H 6750 3750 40  0001 C CNN
+F 1 "AGND_IN" H 6750 3680 50  0000 C CNN
+F 2 "" H 6750 3750 60  0000 C CNN
+F 3 "" H 6750 3750 60  0000 C CNN
+	1    6750 3750
+	1    0    0    -1
+$EndComp
+$Comp
+L AGND_IN #PWR025
+U 1 1 582B671C
 P 8200 4150
-F 0 "#PWR025" H 8200 3900 50  0001 C CNN
-F 1 "GNDD" H 8200 4000 50  0000 C CNN
-F 2 "" H 8200 4150 50  0000 C CNN
-F 3 "" H 8200 4150 50  0000 C CNN
+F 0 "#PWR025" H 8200 4150 40  0001 C CNN
+F 1 "AGND_IN" H 8200 4080 50  0000 C CNN
+F 2 "" H 8200 4150 60  0000 C CNN
+F 3 "" H 8200 4150 60  0000 C CNN
 	1    8200 4150
 	1    0    0    -1
 $EndComp
 $Comp
-L GNDD #PWR026
-U 1 1 57D65722
-P 6750 3750
-F 0 "#PWR026" H 6750 3500 50  0001 C CNN
-F 1 "GNDD" H 6750 3600 50  0000 C CNN
-F 2 "" H 6750 3750 50  0000 C CNN
-F 3 "" H 6750 3750 50  0000 C CNN
-	1    6750 3750
-	1    0    0    -1
-$EndComp
+L AGND_IN #PWR?
+U 1 1 582B6A9C
+P 3600 4150
+F 0 "#PWR?" H 3600 4150 40  0001 C CNN
+F 1 "AGND_IN" H 3600 4080 50  0000 C CNN
+F 2 "" H 3600 4150 60  0000 C CNN
+F 3 "" H 3600 4150 60  0000 C CNN
+	1    3600 4150
+	1    0    0    -1
+$EndComp

Commit message: Fixed power connections for S70--submitted PCB
Parts:
- added TP16, TP17, TP18: TP, lib:TP_HOLE, symbol TP
- FB7: footprint lib:SMD0805 -> lib:SMD0603
Connections:
- wire segments 50 -> 53
Changed lines of the file:
@@
 LIBS:contrib
 LIBS:valves
+LIBS:audio_iface_rev2-cache
 EELAYER 25 0
 EELAYER END
@@
 F 0 "FB7" H 3520 4465 50  0000 L TNN
 F 1 "BLM18PG221SN1D" H 3385 4575 30  0000 C BNN
-F 2 "lib:SMD0805" H 3430 4520 60  0001 C CNN
+F 2 "lib:SMD0603" H 3430 4520 60  0001 C CNN
 F 3 "" H 3430 4520 60  0000 C CNN
 	1    3450 4500
@@
 	4500 2900 4400 2900
 Wire Wire Line
-	4400 2900 4400 2500
-Wire Wire Line
-	4400 2500 4000 2500
+	4400 2500 4400 2900
+Wire Wire Line
+	4000 2500 4400 2500
 Wire Wire Line
 	4000 2500 4000 2600
@@
 	4100 3800 4500 3800
 Wire Wire Line
-	4500 3900 4100 3900
+	4100 3900 4500 3900
 Wire Wire Line
 	4100 4000 4500 4000
 Wire Wire Line
-	4500 4100 4100 4100
+	4100 4100 4500 4100
 Wire Wire Line
 	4100 4200 4500 4200
@@
 	1    0    0    -1
 $EndComp
+$Comp
+L TP TP16
+U 1 1 5848E57A
+P 4150 4600
+F 0 "TP16" H 4150 4500 60  0000 C CNN
+F 1 "TP" H 4150 4700 60  0000 C CNN
+F 2 "lib:TP_HOLE" H 4150 4600 60  0001 C CNN
+F 3 "~" H 4150 4600 60  0000 C CNN
+	1    4150 4600
+	0    1    1    0
+$EndComp
+Wire Wire Line
+	4150 4500 4150 3900
+Connection ~ 4150 3900
+$Comp
+L TP TP17
+U 1 1 5848E660
+P 4250 4850
+F 0 "TP17" H 4250 4750 60  0000 C CNN
+F 1 "TP" H 4250 4950 60  0000 C CNN
+F 2 "lib:TP_HOLE" H 4250 4850 60  0001 C CNN
+F 3 "~" H 4250 4850 60  0000 C CNN
+	1    4250 4850
+	0    1    1    0
+$EndComp
+$Comp
+L TP TP18
+U 1 1 5848E690
+P 4350 5100
+F 0 "TP18" H 4350 5000 60  0000 C CNN
+F 1 "TP" H 4350 5200 60  0000 C CNN
+F 2 "lib:TP_HOLE" H 4350 5100 60  0001 C CNN
+F 3 "~" H 4350 5100 60  0000 C CNN
+	1    4350 5100
+	0    1    1    0
+$EndComp
+Wire Wire Line
+	4250 4750 4250 4000
+Connection ~ 4250 4000
+Wire Wire Line
+	4350 5000 4350 4100
+Connection ~ 4350 4100
 $EndSCHEMATC

Commit message: Modified feedback values on PCB
Changed lines of the file:
@@
 SDTO
 $Comp
-L +3V #PWR28
+L +3V #PWR018
 U 1 1 524DAE69
 P 7700 3450
-F 0 "#PWR28" H 7700 3410 30  0001 C CNN
+F 0 "#PWR018" H 7700 3410 30  0001 C CNN
 F 1 "+3V" H 7700 3560 30  0000 C CNN
 F 2 "~" H 7700 3450 60  0000 C CNN
@@
 NoConn ~ 4500 4300
 $Comp
-L +5V #PWR27
+L +5V #PWR019
 U 1 1 524DADF1
 P 7600 3550
-F 0 "#PWR27" H 7600 3640 20  0001 C CNN
+F 0 "#PWR019" H 7600 3640 20  0001 C CNN
 F 1 "+5V" H 7600 3640 30  0000 C CNN
 F 2 "" H 7600 3550 60  0000 C CNN
@@
 $EndComp
 $Comp
-L +5VA #PWR23
+L +5VA #PWR020
 U 1 1 524E4726
 P 3450 4750
-F 0 "#PWR23" H 3450 4880 20  0001 C CNN
+F 0 "#PWR020" H 3450 4880 20  0001 C CNN
 F 1 "+5VA" H 3450 4850 30  0000 C CNN
 F 2 "" H 3450 4750 60  0000 C CNN
@@
 SPI_MOSI
 $Comp
-L AGND_IN #PWR29
+L AGND_IN #PWR021
 U 1 1 582ADE41
 P 7900 3400
-F 0 "#PWR29" H 7900 3400 40  0001 C CNN
+F 0 "#PWR021" H 7900 3400 40  0001 C CNN
 F 1 "AGND_IN" H 7900 3330 50  0000 C CNN
 F 2 "" H 7900 3400 60  0000 C CNN
@@
 $EndComp
 $Comp
-L AGND_IN #PWR22
+L AGND_IN #PWR022
 U 1 1 582AE1DB
 P 2800 3850
-F 0 "#PWR22" H 2800 3850 40  0001 C CNN
+F 0 "#PWR022" H 2800 3850 40  0001 C CNN
 F 1 "AGND_IN" H 2800 3780 50  0000 C CNN
 F 2 "" H 2800 3850 60  0000 C CNN
@@
 $EndComp
 $Comp
-L AGND_IN #PWR25
+L AGND_IN #PWR023
 U 1 1 582AE264
 P 4100 2900
-F 0 "#PWR25" H 4100 2900 40  0001 C CNN
+F 0 "#PWR023" H 4100 2900 40  0001 C CNN
 F 1 "AGND_IN" H 4100 2830 50  0000 C CNN
 F 2 "" H 4100 2900 60  0000 C CNN
@@
 	4500 2900 4400 2900
 Wire Wire Line
-	4400 2500 4400 2900
-Wire Wire Line
-	4000 2500 4400 2500
+	4400 2900 4400 2500
+Wire Wire Line
+	4400 2500 4000 2500
 Wire Wire Line
 	4000 2500 4000 2600
@@
 Connection ~ 3450 3600
 $Comp
-L AGND_IN #PWR26
+L AGND_IN #PWR024
 U 1 1 582B627B
 P 6750 3750
-F 0 "#PWR26" H 6750 3750 40  0001 C CNN
+F 0 "#PWR024" H 6750 3750 40  0001 C CNN
 F 1 "AGND_IN" H 6750 3680 50  0000 C CNN
 F 2 "" H 6750 3750 60  0000 C CNN
@@
 $EndComp
 $Comp
-L AGND_IN #PWR30
+L AGND_IN #PWR025
 U 1 1 582B671C
 P 8200 4150
-F 0 "#PWR30" H 8200 4150 40  0001 C CNN
+F 0 "#PWR025" H 8200 4150 40  0001 C CNN
 F 1 "AGND_IN" H 8200 4080 50  0000 C CNN
 F 2 "" H 8200 4150 60  0000 C CNN
@@
 $EndComp
 $Comp
-L AGND_IN #PWR24
+L AGND_IN #PWR026
 U 1 1 582B6A9C
 P 3600 4150
-F 0 "#PWR24" H 3600 4150 40  0001 C CNN
+F 0 "#PWR026" H 3600 4150 40  0001 C CNN
 F 1 "AGND_IN" H 3600 4080 50  0000 C CNN
 F 2 "" H 3600 4150 60  0000 C CNN

Commit message: Finished schematic and layout with STM32F7
Connections:
- net labels added: +3V3
- net labels removed: +3V
- wire segments 53 -> 55
Changed lines of the file:
@@
 Text HLabel 4100 4100 0    60   Output ~ 0
 SDTO
-$Comp
-L +3V #PWR28
-U 1 1 524DAE69
-P 7700 3450
-F 0 "#PWR28" H 7700 3410 30  0001 C CNN
-F 1 "+3V" H 7700 3560 30  0000 C CNN
-F 2 "~" H 7700 3450 60  0000 C CNN
-F 3 "~" H 7700 3450 60  0000 C CNN
-	1    7700 3450
-	-1   0    0    1
-$EndComp
 Text Notes 3650 3700 0    40   ~ 0
 Serial Mode
@@
 NoConn ~ 4500 4300
 $Comp
-L +5V #PWR27
+L +5V #PWR018
 U 1 1 524DADF1
 P 7600 3550
-F 0 "#PWR27" H 7600 3640 20  0001 C CNN
+F 0 "#PWR018" H 7600 3640 20  0001 C CNN
 F 1 "+5V" H 7600 3640 30  0000 C CNN
 F 2 "" H 7600 3550 60  0000 C CNN
@@
 $EndComp
 $Comp
-L +5VA #PWR23
+L +5VA #PWR019
 U 1 1 524E4726
 P 3450 4750
-F 0 "#PWR23" H 3450 4880 20  0001 C CNN
+F 0 "#PWR019" H 3450 4880 20  0001 C CNN
 F 1 "+5VA" H 3450 4850 30  0000 C CNN
 F 2 "" H 3450 4750 60  0000 C CNN
@@
 SPI_MOSI
 $Comp
-L AGND_IN #PWR29
+L AGND_IN #PWR020
 U 1 1 582ADE41
 P 7900 3400
-F 0 "#PWR29" H 7900 3400 40  0001 C CNN
+F 0 "#PWR020" H 7900 3400 40  0001 C CNN
 F 1 "AGND_IN" H 7900 3330 50  0000 C CNN
 F 2 "" H 7900 3400 60  0000 C CNN
@@
 $EndComp
 $Comp
-L AGND_IN #PWR22
+L AGND_IN #PWR021
 U 1 1 582AE1DB
 P 2800 3850
-F 0 "#PWR22" H 2800 3850 40  0001 C CNN
+F 0 "#PWR021" H 2800 3850 40  0001 C CNN
 F 1 "AGND_IN" H 2800 3780 50  0000 C CNN
 F 2 "" H 2800 3850 60  0000 C CNN
@@
 $EndComp
 $Comp
-L AGND_IN #PWR25
+L AGND_IN #PWR022
 U 1 1 582AE264
 P 4100 2900
-F 0 "#PWR25" H 4100 2900 40  0001 C CNN
+F 0 "#PWR022" H 4100 2900 40  0001 C CNN
 F 1 "AGND_IN" H 4100 2830 50  0000 C CNN
 F 2 "" H 4100 2900 60  0000 C CNN
@@
 	5700 3400 7700 3400
 Wire Wire Line
-	7700 3400 7700 3450
+	7700 3400 7700 3650
 Wire Wire Line
 	7600 3550 7600 3500
@@
 Connection ~ 3450 3600
 $Comp
-L AGND_IN #PWR26
+L AGND_IN #PWR023
 U 1 1 582B627B
 P 6750 3750
-F 0 "#PWR26" H 6750 3750 40  0001 C CNN
+F 0 "#PWR023" H 6750 3750 40  0001 C CNN
 F 1 "AGND_IN" H 6750 3680 50  0000 C CNN
 F 2 "" H 6750 3750 60  0000 C CNN
@@
 $EndComp
 $Comp
-L AGND_IN #PWR30
+L AGND_IN #PWR024
 U 1 1 582B671C
 P 8200 4150
-F 0 "#PWR30" H 8200 4150 40  0001 C CNN
+F 0 "#PWR024" H 8200 4150 40  0001 C CNN
 F 1 "AGND_IN" H 8200 4080 50  0000 C CNN
 F 2 "" H 8200 4150 60  0000 C CNN
@@
 $EndComp
 $Comp
-L AGND_IN #PWR24
+L AGND_IN #PWR025
 U 1 1 582B6A9C
 P 3600 4150
-F 0 "#PWR24" H 3600 4150 40  0001 C CNN
+F 0 "#PWR025" H 3600 4150 40  0001 C CNN
 F 1 "AGND_IN" H 3600 4080 50  0000 C CNN
 F 2 "" H 3600 4150 60  0000 C CNN
@@
 	4350 5000 4350 4100
 Connection ~ 4350 4100
+$Comp
+L +3V3 #PWR026
+U 1 1 58CFB0B9
+P 8300 3550
+F 0 "#PWR026" H 8300 3400 50  0001 C CNN
+F 1 "+3V3" H 8300 3690 50  0000 C CNN
+F 2 "" H 8300 3550 50  0000 C CNN
+F 3 "" H 8300 3550 50  0000 C CNN
+	1    8300 3550
+	1    0    0    -1
+$EndComp
+Wire Wire Line
+	7700 3650 8300 3650
+Wire Wire Line
+	8300 3650 8300 3550
 $EndSCHEMATC
