File: hw/rev2/codec.sch (KiCad schematic (older format))
At the start: 5 parts, among them U3 AK4621

Commit message: Most of a schematic
Parts:
- C25, C26, C27, C28: symbol CAP -> symbols:CAP
- U3: symbol AK4621 -> symbols:AK4621
Connections:
- wire segments 50 -> 57
Changed lines of the file:
@@
-EESchema Schematic File Version 2
-LIBS:symbols
-LIBS:power
-LIBS:device
-LIBS:transistors
-LIBS:conn
-LIBS:linear
-LIBS:regul
-LIBS:74xx
-LIBS:cmos4000
-LIBS:adc-dac
-LIBS:memory
-LIBS:xilinx
-LIBS:microcontrollers
-LIBS:dsp
-LIBS:microchip
-LIBS:analog_switches
-LIBS:motorola
-LIBS:texas
-LIBS:intel
-LIBS:audio
-LIBS:interface
-LIBS:digital-audio
-LIBS:philips
-LIBS:display
-LIBS:cypress
-LIBS:siliconi
-LIBS:opto
-LIBS:atmel
-LIBS:contrib
-LIBS:valves
+EESchema Schematic File Version 4
 LIBS:audio_iface_rev2-cache
-EELAYER 25 0
+EELAYER 26 0
 EELAYER END
 $Descr A 11000 8500
@@
 $EndDescr
 $Comp
-L AK4621 U3
+L symbols:AK4621 U3
 U 1 1 523B94A4
 P 5100 3350
@@
 $EndComp
 $Comp
-L CAP C26
+L symbols:CAP C26
 U 1 1 523B94B1
 P 2700 3600
@@
 $EndComp
 $Comp
-L CAP C25
+L symbols:CAP C25
 U 1 1 523B94B7
 P 2550 3600
@@
 	5700 3300 7900 3300
 Wire Wire Line
-	2800 3500 2800 3850
+	2800 3500 2800 3800
 Wire Wire Line
 	2800 3500 4500 3500
 Wire Wire Line
-	2550 3800 2800 3800
+	2550 3800 2700 3800
 Wire Wire Line
 	2550 3800 2550 3700
@@
 	2550 3500 2550 3400
 Wire Wire Line
-	2450 3400 4500 3400
+	2450 3400 2550 3400
 Wire Wire Line
 	2700 3400 2700 3500
@@
 	7900 3300 7900 3400
 $Comp
-L CAP C28
+L symbols:CAP C28
 U 1 1 523B9668
 P 4200 2700
@@
 $EndComp
 $Comp
-L CAP C27
+L symbols:CAP C27
 U 1 1 523B9675
 P 4000 2700
@@
 	4400 2900 4400 2500
 Wire Wire Line
-	4400 2500 4000 2500
+	4400 2500 4200 2500
 Wire Wire Line
 	4000 2500 4000 2600
@@
 	4100 2900 4100 2850
 Wire Wire Line
-	4000 2850 4200 2850
+	4000 2850 4100 2850
 Wire Wire Line
 	4200 2850 4200 2800
@@
 	2450 3350 2450 3400
 $Comp
-L +3V #PWR33
+L symbols:+3V #PWR33
 U 1 1 524DAE69
 P 7700 3450
@@
 NoConn ~ 4500 4300
 $Comp
-L +5V #PWR32
+L power:+5V #PWR32
 U 1 1 524DADF1
 P 7600 3550
@@
 $EndComp
 $Comp
-L +5VA #PWR26
+L power:+5VA #PWR26
 U 1 1 524E470F
 P 2450 3350
@@
 $EndComp
 $Comp
-L +5VA #PWR28
+L power:+5VA #PWR28
 U 1 1 524E4726
 P 3450 3950
@@
 	3600 4150 3600 3700
 $Comp
-L AGND_OUT #PWR27
+L symbols:AGND_OUT #PWR27
 U 1 1 524E577E
 P 2800 3850
@@
 $EndComp
 $Comp
-L AGND_OUT #PWR30
+L symbols:AGND_OUT #PWR30
 U 1 1 524E579A
 P 4100 2900
@@
 $EndComp
 $Comp
-L AGND_OUT #PWR29
+L symbols:AGND_OUT #PWR29
 U 1 1 5257A82B
 P 3600 4150
@@
 	8200 3900 8200 4150
 Wire Wire Line
-	6750 3750 6750 3600
+	6750 3750 6750 3700
 Wire Wire Line
 	6750 3600 5700 3600
@@
 Connection ~ 6750 3700
 $Comp
-L GNDD #PWR34
+L power:GNDD #PWR34
 U 1 1 57D656B3
 P 7900 3400
@@
 $EndComp
 $Comp
-L GNDD #PWR35
+L power:GNDD #PWR35
 U 1 1 57D656EE
 P 8200 4150
@@
 $EndComp
 $Comp
-L GNDD #PWR31
+L power:GNDD #PWR31
 U 1 1 57D65722
 P 6750 3750
@@
 	1    0    0    -1
 $EndComp
+Wire Wire Line
+	2800 3800 2800 3850
+Wire Wire Line
+	2700 3400 4500 3400
+Wire Wire Line
+	2700 3800 2800 3800
+Wire Wire Line
+	2550 3400 2700 3400
+Wire Wire Line
+	4200 2500 4000 2500
+Wire Wire Line
+	4100 2850 4200 2850
+Wire Wire Line
+	6750 3700 6750 3600
 $EndSCHEMATC
