File: hw/rev2/hp_amp.sch (KiCad schematic (older format))
At the start: 36 parts

Commit message: Lots of things: --Added RGB LED on timer outputs --Input: Moved capacitively coupled feedback nodes from vgnd to gnd --Output: LTC6242 for filtering to amplifier --Power: 2-stage supply for analog: USB 5V boost to 6V, LDO to 5V   Digital still using LDO from USB 5V and not caring about anyone   Bonus! Can completely shut off analog portion of board --Layout and routing: All of it TODO: final checks on layout and LVS (vs simulation) HEAD2HEAD2HEAD! TODO: adjust silkscreen, add logo TODO: debate adding 12.288MHz dedicated crystal
Parts:
- gave numbers to parts that had none: 32

Commit message: Rev 2a sent off for manufacturing: Slot added instead of drill hole at audio IO end Drill added near center Fixed huge error in HP amp schematic/layout Got rid of more labels Got rid of redundant UART port. Not sure how that happened twice... Got rid of DC blocking before CODEC inputs
Parts:
- added C72: 1u, ~, symbol CAP
Connections:
- wire segments 113 -> 115

Commit message: Started board upgrade to 4 layers and better signal isolation
Parts:
- C51, C52, C53, C54, C55, C56, C57, C58, C59, C60, C61, C62, C63, C64, C65, C67, C68, C72, R31, R32, R33, R34, R35, R36, R37, R38: footprint ~ -> lib:SMD0402
- C66: footprint ~ -> lib:SMD0805
- TP10, TP11, TP8, TP9: footprint ~ -> lib:TP_HOLE
- U7: footprint ~ -> lib:LT_DFN16_QUAD
- U8: footprint ~ -> lib:TPA8130A2-QFN20
