File: hw/rev2/hp_amp.sch (KiCad schematic (older format))
At the start: 33 parts, among them U7 LTC6242, U8 TPA6130A2

Commit message: Lots of layout and grounding changes. DRC good
Connections:
- net labels removed: GND
Changed lines of the file:
@@
-$EndComp
-$Comp
-L GND #PWR060
-U 1 1 534EFAAA
-P 2150 3100
-F 0 "#PWR060" H 2150 3100 30  0001 C CNN
-F 1 "GND" H 2150 3030 30  0001 C CNN
-F 2 "" H 2150 3100 60  0000 C CNN
-F 3 "" H 2150 3100 60  0000 C CNN
-	1    2150 3100
-	1    0    0    -1
 $EndComp
 $Comp
@@
 $EndComp
 $Comp
-L GND #PWR061
-U 1 1 534EFB3A
-P 2150 4100
-F 0 "#PWR061" H 2150 4100 30  0001 C CNN
-F 1 "GND" H 2150 4030 30  0001 C CNN
-F 2 "" H 2150 4100 60  0000 C CNN
-F 3 "" H 2150 4100 60  0000 C CNN
-	1    2150 4100
-	1    0    0    -1
-$EndComp
-$Comp
 L OPAMP_QUAD U7
 U 1 1 534EFB41
@@
 $EndComp
 $Comp
-L GND #PWR062
-U 1 1 534EFB6D
-P 2150 5100
-F 0 "#PWR062" H 2150 5100 30  0001 C CNN
-F 1 "GND" H 2150 5030 30  0001 C CNN
-F 2 "" H 2150 5100 60  0000 C CNN
-F 3 "" H 2150 5100 60  0000 C CNN
-	1    2150 5100
-	1    0    0    -1
-$EndComp
-$Comp
 L OPAMP_QUAD U7
 U 2 1 534EFB74
@@
 $EndComp
 $Comp
-L GND #PWR063
-U 1 1 534EFBA0
-P 2150 6100
-F 0 "#PWR063" H 2150 6100 30  0001 C CNN
-F 1 "GND" H 2150 6030 30  0001 C CNN
-F 2 "" H 2150 6100 60  0000 C CNN
-F 3 "" H 2150 6100 60  0000 C CNN
-	1    2150 6100
-	1    0    0    -1
-$EndComp
-$Comp
-L AGND_OUT #PWR064
-U 1 1 534FD9C3
-P 6350 5250
-F 0 "#PWR064" H 6350 5250 40  0001 C CNN
-F 1 "AGND_OUT" H 6350 5180 50  0000 C CNN
-F 2 "" H 6350 5250 60  0000 C CNN
-F 3 "" H 6350 5250 60  0000 C CNN
-	1    6350 5250
-	1    0    0    -1
-$EndComp
-$Comp
-L +5VA #PWR065
+L +5VA #PWR061
 U 1 1 534FDA74
 P 6550 4150
-F 0 "#PWR065" H 6550 4280 20  0001 C CNN
+F 0 "#PWR061" H 6550 4280 20  0001 C CNN
 F 1 "+5VA" H 6550 4250 30  0000 C CNN
 F 2 "" H 6550 4150 60  0000 C CNN
@@
 $EndComp
 $Comp
-L +5VA #PWR066
+L +5VA #PWR062
 U 1 1 534FDB27
 P 7200 3850
-F 0 "#PWR066" H 7200 3980 20  0001 C CNN
+F 0 "#PWR062" H 7200 3980 20  0001 C CNN
 F 1 "+5VA" H 7200 3950 30  0000 C CNN
 F 2 "" H 7200 3850 60  0000 C CNN
 F 3 "" H 7200 3850 60  0000 C CNN
 	1    7200 3850
-	1    0    0    -1
-$EndComp
-$Comp
-L AGND_OUT #PWR067
-U 1 1 534FDB2D
-P 7200 4300
-F 0 "#PWR067" H 7200 4300 40  0001 C CNN
-F 1 "AGND_OUT" H 7200 4230 50  0000 C CNN
-F 2 "" H 7200 4300 60  0000 C CNN
-F 3 "" H 7200 4300 60  0000 C CNN
-	1    7200 4300
 	1    0    0    -1
 $EndComp
@@
 HPL
 $Comp
-L +5VA #PWR068
+L +5VA #PWR063
 U 1 1 534FE1CA
 P 3050 6600
-F 0 "#PWR068" H 3050 6730 20  0001 C CNN
+F 0 "#PWR063" H 3050 6730 20  0001 C CNN
 F 1 "+5VA" H 3050 6700 30  0000 C CNN
 F 2 "" H 3050 6600 60  0000 C CNN
@@
 $EndComp
 $Comp
-L AGND_OUT #PWR069
+L AGND_OUT #PWR064
 U 1 1 534FE2F2
 P 3050 7700
-F 0 "#PWR069" H 3050 7700 40  0001 C CNN
+F 0 "#PWR064" H 3050 7700 40  0001 C CNN
 F 1 "AGND_OUT" H 3050 7630 50  0000 C CNN
 F 2 "" H 3050 7700 60  0000 C CNN
@@
 $EndComp
 $Comp
-L AGND_OUT #PWR070
-U 1 1 5356F02A
-P 4200 4950
-F 0 "#PWR070" H 4200 4950 40  0001 C CNN
-F 1 "AGND_OUT" H 4200 4880 50  0000 C CNN
-F 2 "~" H 4200 4950 60  0000 C CNN
-F 3 "~" H 4200 4950 60  0000 C CNN
-	1    4200 4950
-	1    0    0    -1
-$EndComp
-$Comp
 L CAP C65
 U 1 1 5356F2A6
@@
 $EndComp
 $Comp
-L +5VA #PWR071
+L +5VA #PWR065
 U 1 1 5356F633
 P 4700 3250
-F 0 "#PWR071" H 4700 3380 20  0001 C CNN
+F 0 "#PWR065" H 4700 3380 20  0001 C CNN
 F 1 "+5VA" H 4700 3350 30  0000 C CNN
 F 2 "" H 4700 3250 60  0000 C CNN
@@
 	5850 4150 5850 3650
 Connection ~ 5850 3650
+$Comp
+L AGND_OUT #PWR066
+U 1 1 582AD0F9
+P 6350 5250
+F 0 "#PWR066" H 6350 5250 40  0001 C CNN
+F 1 "AGND_OUT" H 6350 5180 50  0000 C CNN
+F 2 "" H 6350 5250 60  0000 C CNN
+F 3 "" H 6350 5250 60  0000 C CNN
+	1    6350 5250
+	1    0    0    -1
+$EndComp
+$Comp
+L AGND_OUT #PWR067
+U 1 1 582AD17A
+P 7200 4300
+F 0 "#PWR067" H 7200 4300 40  0001 C CNN
+F 1 "AGND_OUT" H 7200 4230 50  0000 C CNN
+F 2 "" H 7200 4300 60  0000 C CNN
+F 3 "" H 7200 4300 60  0000 C CNN
+	1    7200 4300
+	1    0    0    -1
+$EndComp
+$Comp
+L AGND_OUT #PWR068
+U 1 1 582AD1F4
+P 4200 4950
+F 0 "#PWR068" H 4200 4950 40  0001 C CNN
+F 1 "AGND_OUT" H 4200 4880 50  0000 C CNN
+F 2 "" H 4200 4950 60  0000 C CNN
+F 3 "" H 4200 4950 60  0000 C CNN
+	1    4200 4950
+	1    0    0    -1
+$EndComp
+$Comp
+L AGND_OUT #PWR069
+U 1 1 582AD26E
+P 2150 6100
+F 0 "#PWR069" H 2150 6100 40  0001 C CNN
+F 1 "AGND_OUT" H 2150 6030 50  0000 C CNN
+F 2 "" H 2150 6100 60  0000 C CNN
+F 3 "" H 2150 6100 60  0000 C CNN
+	1    2150 6100
+	1    0    0    -1
+$EndComp
+$Comp
+L AGND_OUT #PWR070
+U 1 1 582AD3C6
+P 2150 5100
+F 0 "#PWR070" H 2150 5100 40  0001 C CNN
+F 1 "AGND_OUT" H 2150 5030 50  0000 C CNN
+F 2 "" H 2150 5100 60  0000 C CNN
+F 3 "" H 2150 5100 60  0000 C CNN
+	1    2150 5100
+	1    0    0    -1
+$EndComp
+$Comp
+L AGND_OUT #PWR071
+U 1 1 582AD568
+P 2150 4100
+F 0 "#PWR071" H 2150 4100 40  0001 C CNN
+F 1 "AGND_OUT" H 2150 4030 50  0000 C CNN
+F 2 "" H 2150 4100 60  0000 C CNN
+F 3 "" H 2150 4100 60  0000 C CNN
+	1    2150 4100
+	1    0    0    -1
+$EndComp
+$Comp
+L AGND_OUT #PWR072
+U 1 1 582AD779
+P 2150 3100
+F 0 "#PWR072" H 2150 3100 40  0001 C CNN
+F 1 "AGND_OUT" H 2150 3030 50  0000 C CNN
+F 2 "" H 2150 3100 60  0000 C CNN
+F 3 "" H 2150 3100 60  0000 C CNN
+	1    2150 3100
+	1    0    0    -1
+$EndComp
 $EndSCHEMATC
