File: hw/rev2/audio_iface_rev2.kicad_pcb (KiCad board)
At the start: 4 copper layers, 66 x 24.8 mm, 153 parts, among them J1 COAX, J2 CONN_01X02, J3 USBMICROCONN, J4 CONN_01X02, J5 CONN_01X02, J6 COAX, J7 COAX, J9 CONN_01X02, P3 CONN_01X06, U1 LT6241, U2 LTC6242, U3 AK4621, U4 K20X7_QFP64, U5 TPS61252, U6 LP2992AILD-5.0, U7 LTC6242, U8 TPA6130A2, U9 MT29FXX01A, X1 XTAL, X2 ASFLM2-12.288MHZ

Commit message: Most of a schematic
Parts:
- removed C34, C39, C44, C64, C68: 10n, lib:SMD0402
- removed C35, C36: CAP, lib:SMD0402
- removed C37: 22u, lib:SMD1206_POL
- removed C38, C63, C67: 100n, lib:SMD0402
- removed C40: 100p, lib:SMD0402
- removed C41, C45: 10n 16V, lib:SMD0402
- removed C42: 2.2u, lib:SMD0402
- removed C43, C66: 10u, lib:SMD0805
- removed C46: 10n 6.3V, lib:SMD0402
- removed C47: 0.1u 6.3V, lib:SMD0402
- removed C48: 0.1u 6.3V, lib:SMD0603
- removed C49: 10u 6.3V, lib:SMD0805
- removed C50: 100u 6.3V, lib:SMD1411_POL
- removed C51, C52, C53, C54, C55, C56, C57, C58: 470p (5%), lib:SMD0402
- removed C59, C60, C61, C62, C65, C72, C73: 1u, lib:SMD0402
- removed C69: 0.1u, lib:SMD0402
- removed C70: 0.01u, lib:SMD0402
- removed J1, J6, J7: COAX, lib:SMA_EDGE
- removed J4, J5, J9: CONN_01X02, lib:HDR_2X1_50MIL
- removed L1: MLZ2012A1R5WT000, lib:SMD0805
- removed P3: CONN_01X06, lib:HDR_6X1_50MIL
- removed R10: 4.53k (1%), lib:SMD0402
- removed R11, R14: 220 (1%), lib:SMD0402
- removed R12: 250k, lib:SMD0402
- removed R13, R16: 10k (1%), lib:SMD0402
- removed R15: 220k, lib:SMD0402
- removed R17, R18, R19: 22, lib:SMD0402
- removed R20: 10k, lib:SMD0402
- removed R25, R26: RES, lib:SMD0402
- removed R27: 20k, lib:SMD0402
- removed R28: 1Meg, lib:SMD0402
- removed R29: 0R, lib:SMD0402
- removed R3: 22R, lib:SMD0402
- removed R30: 39, lib:SMD0402
- removed R31, R32, R33, R34, R35, R36, R37, R38: 6.8k (1%), lib:SMD0402
- removed R39: 100k, lib:SMD0402
- removed Rf1: 5.11k (1%), lib:SMD0402
- removed TP10, TP11, TP12, TP13, TP14: TP, lib:TP_HOLE
- removed U8: TPA6130A2, lib:TPA8130A2-QFN20
- removed U9: MT29FXX01A, MICRON_VFBGA63:MICRON_VFBGA63
- added D2: LS L29K-H1J2-1-Z, LEDs:LED_0603, F.Cu at (151.4, 58.3)
- C1, C23, C24: value 10n -> 2.2u; footprint lib:SMD0402 -> Capacitors_SMD:C_0603
- C10: value 1n -> 22u; footprint lib:SMD0603 -> Capacitors_SMD:C_1210
- C11: value 33n -> 100n; footprint lib:SMD0603 -> Capacitors_SMD:C_0402
- C12, C14: value 10u 6.3V -> 1u; footprint lib:SMD0805 -> Capacitors_SMD:C_0402
- C13: value 0.1u 6.3V -> 10u; footprint lib:SMD0402 -> Capacitors_SMD:C_0805; moved to F.Cu
- C15: value 0.1u 6.3V -> 0.1u; footprint lib:SMD0402 -> Capacitors_SMD:C_0402
- C16: footprint lib:SMD0402 -> Capacitors_SMD:C_0402; moved to F.Cu
- C17: value 1u 6.3V -> 0.1u; footprint lib:SMD0402 -> Capacitors_SMD:C_0402; moved to F.Cu
- C18: value 1u 6.3V -> 0.1u; footprint lib:SMD0402 -> Capacitors_SMD:C_0402
- C19: value 100u 6.3V -> 0.1u; footprint lib:SMD0402 -> Capacitors_SMD:C_0402
- C2: value 10u 6.3V -> 2.2u; footprint lib:SMD0603 -> Capacitors_SMD:C_0603
- C20: value 10p -> 0.1u; footprint lib:SMD0402 -> Capacitors_SMD:C_0402
- C21: value 10u 6.3V -> 2.2u; footprint lib:SMD0805 -> Capacitors_SMD:C_0603
- C22: value 10p -> 10u; footprint lib:SMD0402 -> Capacitors_SMD:C_0805
- C25: value 1u -> 10u; footprint lib:SMD0402 -> Capacitors_SMD:C_0805
- C26, C30, C8: value 0.1u -> 2.2u; footprint lib:SMD0402 -> Capacitors_SMD:C_0603
- C27, C75: value 10u -> 2.2u; footprint lib:SMD0805 -> Capacitors_SMD:C_0603
- C28: value 0.1u -> 10u; footprint lib:SMD0402 -> Capacitors_SMD:C_0805
- C29, C31: footprint lib:SMD0603 -> Capacitors_SMD:C_0603
- C3: value 10p -> 2.2u; footprint lib:SMD0402 -> Capacitors_SMD:C_0603
- C32, C33, C76: footprint lib:SMD0402 -> Capacitors_SMD:C_0402
- C4: value 100u 6.3V -> 2.2u; footprint lib:SMD1411_POL -> Capacitors_SMD:C_0603
- C5: value 10u 4V -> 2.2u; footprint lib:SMD0805 -> Capacitors_SMD:C_0603
- C6: value 1u -> 2.2u; footprint lib:SMD0402 -> Capacitors_SMD:C_0603
- C7: value 1n -> 100n; footprint lib:SMD0603 -> Capacitors_SMD:C_0402
- C71: value 10n -> 100n; footprint lib:SMD0402 -> Capacitors_SMD:C_0402
- C9: value 2n -> 22u; footprint lib:SMD0603 -> Capacitors_SMD:C_1210
- D1: value LTST-C19FD1WT -> LG L29K-F2J1-24-Z; footprint lib:LED-6PLCC -> LEDs:LED_0603
- FB1, FB2: footprint lib:SMD0805 -> Inductors_SMD:L_0805
- J2: value CONN_01X02 -> Screw_Terminal_01x02; footprint lib:HDR_2X1_50MIL -> TerminalBlocks_Phoenix:TerminalBlock_Phoenix_MPT-2.54mm_2pol
- J3: value USBMICROCONN -> USB_B_Micro; footprint lib:FCI_10118194 -> Connectors:USB_Micro-B_10103594-0001LF
- R1: value 3.9k (1%) -> 100k; footprint lib:SMD0402 -> Resistors_SMD:R_0402
- R2: value 22R -> 820; footprint lib:SMD0402 -> Resistors_SMD:R_0402
- R21, R22, R24: footprint lib:SMD0402 -> Resistors_SMD:R_0402
- R23: value 220 -> 7.5; footprint lib:SMD0402 -> Resistors_SMD:R_0402
- R4: value 100k (1%) -> 12k (1%); footprint lib:SMD0402 -> Resistors_SMD:R_0402
- R5: value 100k (1%) -> 2k; footprint lib:SMD0402 -> Resistors_SMD:R_0402
- R6: value 470 (1%) -> 2k; footprint lib:SMD0402 -> Resistors_SMD:R_0402
- R7: value 8.87k (1%) -> 100k; footprint lib:SMD0402 -> Resistors_SMD:R_0402
- R8: value 26.1k (1%) -> 100k; footprint lib:SMD0402 -> Resistors_SMD:R_0402
- R9: value 1.4k (1%) -> 0R; footprint lib:SMD0402 -> Resistors_SMD:R_0402
- TP1, TP2, TP3, TP5, TP6, TP7, TP8, TP9: footprint lib:TP_HOLE -> Wire_Pads:SolderWirePad_single_1mmDrill
- TP4: value TP_PTE0 -> TP; footprint lib:TP_HOLE -> Wire_Pads:SolderWirePad_single_1mmDrill
- U1: value LT6241 -> STM32H743VITx; footprint lib:LT_DFN8_DUAL -> Housings_QFP:LQFP-100_14x14mm_Pitch0.5mm
- U2: value LTC6242 -> USB3300-EZK; footprint lib:LT_DFN16_QUAD -> Housings_DFN_QFN:QFN-32-1EP_5x5mm_Pitch0.5mm
- U3: value AK4621 -> ADAU1772; footprint lib:AK4621_VSOP30 -> Housings_DFN_QFN:QFN-40-1EP_6x6mm_Pitch0.5mm
- U4: value K20X7_QFP64 -> LP5907MFX-3.3; footprint lib:FREESCALE_QFP64 -> TO_SOT_Packages_SMD:SOT-23-5
- U5: value TPS61252 -> LP5907MFX-1.8; footprint lib:TPS61252_QFN8 -> TO_SOT_Packages_SMD:SOT-23-5
- U6: value LP2992AILD-5.0 -> LP5907MFX-3.3; footprint lib:TI_WSON6 -> TO_SOT_Packages_SMD:SOT-23-5
- U7: value LTC6242 -> USBLC6-2SC6; footprint lib:LT_DFN16_QUAD -> TO_SOT_Packages_SMD:SOT-23-6
- X1: value XTAL -> DSC6011JE1A-024.0000; footprint lib:TXC_7A -> Oscillators:Oscillator_SMD_SeikoEpson_SG210-4pin_2.5x2.0mm
- X2: value ASFLM2-12.288MHZ -> DSC6011CI2A-012.2880; footprint lib:ASFLM -> Oscillators:Oscillator_SMD_EuroQuartz_XO32-4pin_3.2x2.5mm
- moved U7 107.8 mm to (93.8, 88.2)
- moved U2 91.1 mm to (117.5, 98.0), turned to 0 degrees
- moved J3 66.5 mm to (87.7, 89.0)
- moved FB1 63.1 mm to (93.9, 90.7)
- moved FB2 62.4 mm to (93.9, 92.7), turned to 0 degrees
- moved C30 62.3 mm to (96.9, 90.3), turned to 0 degrees
- moved C13 61.9 mm to (148.2, 58.6), turned to 0 degrees
- moved C76 60.1 mm to (97.1, 87.9)
- moved TP1 60.1 mm to (96.7, 92.2)
- moved U1 57.4 mm to (129.7, 83.5)
- moved C1 57.0 mm to (157.2, 58.3), turned to 0 degrees
- moved C75 56.4 mm to (97.5, 86.7), turned to 0 degrees
- moved C9 53.7 mm to (173.6, 41.3), turned to 0 degrees
- moved R21 52.8 mm to (180.5, 40.4), turned to 0 degrees
- moved C7 49.1 mm to (176.3, 47.6), turned to 0 degrees
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Connections:
- C1 pad 1: AGND_IN -> GNDD
- C1 pad 2: /Audio In/MIC_IN -> +1V8
- C10 pad 1: AGND_IN -> /Microcontroller/MIC1_IN
- C11 pad 1: Net-(C11-Pad1) -> AGND
- C12 pad 2: VCOM_VRT -> GNDD
- C13 pad 1: +5VA -> +1V8
- C13 pad 2: AGND_IN -> GNDD
- C14 pad 1: /Audio In/EXT_IN -> +1V8
- C14 pad 2: Net-(C14-Pad2) -> GNDD
- C15 pad 1: +5VA -> +1V8
- C15 pad 2: AGND_IN -> GNDD
- C16 pad 1: AGND_IN -> AGND
- C16 pad 2: +3V -> +3V3A
- C17 pad 1: +5VA -> AGND
- C17 pad 2: AGND_IN -> +3V3A
- C18 pad 1: +5VA -> AGND
- C18 pad 2: AGND_IN -> +3V3A
- C19 pad 1: +5VA -> AGND
- C19 pad 2: AGND_IN -> +3V3A
- C2 pad 1: Net-(C2-Pad1) -> GNDD
- C2 pad 2: AGND_IN -> +1V8
- C20 pad 1: Net-(C11-Pad2) -> AGND
- C20 pad 2: Net-(C20-Pad2) -> +3V3A
- C21 pad 1: +5VA -> GND
- C21 pad 2: AGND_IN -> +5V
- C22 pad 1: Net-(C20-Pad2) -> AGND
- C22 pad 2: Net-(C22-Pad2) -> +3V3A
- C23 pad 1: VCOM_VRT -> AGND
- C23 pad 2: /CODEC/AINR- -> +3V3A
- C24 pad 1: /CODEC/AINL+ -> GND
- C24 pad 2: /CODEC/AINL- -> +5V
- C25 pad 1: AGND_IN -> GND
- C25 pad 2: +5VA -> +1V8
- C26 pad 1: AGND_IN -> GND
- C26 pad 2: +5VA -> +1V8
- C27 pad 1: AGND_IN -> GND
- C27 pad 2: Net-(C27-Pad2) -> +5V
- C28 pad 1: AGND_IN -> GND
- C28 pad 2: Net-(C27-Pad2) -> +3V3
- C29 pad 1: AGND_IN -> GND
- C29 pad 2: USB_5V -> +3V3
- C3 pad 1: Net-(C3-Pad1) -> GNDD
- C3 pad 2: Net-(C3-Pad2) -> +1V8
- C30 pad 1: AGND_IN -> Net-(C30-Pad1)
- C30 pad 2: USB_5V -> GNDD
- C31 pad 1: AGND_IN -> GNDD
- C31 pad 2: +3V -> +1V8
- C32 pad 1: AGND_IN -> GNDD
- C32 pad 2: +3V -> +1V8
- C33 pad 1: AGND_IN -> GNDD
- C33 pad 2: +3V -> +1V8
- C4 pad 1: VCOM_VRT -> GNDD
- C4 pad 2: AGND_IN -> Net-(C4-Pad2)
- C5 pad 1: VCOM_VRT -> GNDD
- C5 pad 2: AGND_IN -> +1V8
- C6 pad 1: VCOM_VRT -> GNDD
- C6 pad 2: AGND_IN -> Net-(C6-Pad2)
- C7 pad 1: AGND_IN -> GNDD
- C7 pad 2: Net-(C7-Pad2) -> +1V8
- C71 pad 1: AGND_IN -> GNDD
- C71 pad 2: +3V -> /Microcontroller/MCLK
- C75 pad 1: Net-(C75-Pad1) -> /Microcontroller/USB_VBUS
- C75 pad 2: AGND_IN -> GNDD
- C76 pad 2: AGND_IN -> GNDD
- C8 pad 1: VCOM_VRT -> Net-(C11-Pad2)
- C8 pad 2: AGND_IN -> AGND
- C9 pad 1: Net-(C9-Pad1) -> /Microcontroller/MIC0_IN
- FB1 pad 2: AGND_IN -> GNDD
- FB2 pad 2: Net-(C75-Pad1) -> /Microcontroller/USB_VBUS
- J2 pad 1: AGND_IN -> +5V
- J2 pad 2: /Audio In/EXT_IN -> GND
- J3 pad 1: Net-(C75-Pad1) -> /Microcontroller/USB_VBUS
- J3 pad 2: Net-(J3-Pad2) -> /Microcontroller/USB_D-
- J3 pad 3: Net-(J3-Pad3) -> /Microcontroller/USB_D+
- J3 pad 4: Net-(J3-Pad4) -> /Microcontroller/USB_ID
- R1 pad 1: /Audio In/MIC_IN -> Net-(R1-Pad1)
- R1 pad 2: +5VA -> GNDD
- R2 pad 1: Net-(J3-Pad2) -> Net-(R2-Pad1)
- R2 pad 2: /Microcontroller/USB_D- -> /Microcontroller/USB_VBUS
- R23 pad 1: Net-(D1-PadA3) -> Net-(D1-Pad2)
- R24 pad 1: Net-(D1-PadA2) -> Net-(D2-Pad2)
- R4 pad 1: Net-(C69-Pad2) -> GNDD
- R4 pad 2: +5VA -> Net-(R4-Pad2)
- R5 pad 1: AGND_IN -> /Microcontroller/MIC1_IN
- R5 pad 2: Net-(C69-Pad2) -> Net-(C12-Pad1)
- R6 pad 1: Net-(C2-Pad1) -> /Microcontroller/MIC0_IN
- R6 pad 2: Net-(C3-Pad1) -> Net-(C12-Pad1)
- R7 pad 1: Net-(C70-Pad2) -> GNDD
- R7 pad 2: Net-(C9-Pad1) -> /Microcontroller/CODEC_~PD
- R8 pad 1: Net-(C9-Pad1) -> GND
- R8 pad 2: Net-(C7-Pad2) -> /Microcontroller/ANALOG_EN
- R9 pad 1: Net-(C9-Pad2) -> USB_5V
- R9 pad 2: Net-(C11-Pad1) -> +5V
- TP1 pad 1: Net-(J3-Pad4) -> /Microcontroller/USB_ID
- TP2 pad 1: /CODEC/AINL- -> /Microcontroller/MCLK
- TP3 pad 1: /CODEC/AINL+ -> /Microcontroller/CODEC_SDI
- TP4 pad 1: Net-(TP4-Pad1) -> /Microcontroller/CODEC_SDO
- TP5 pad 1: +5VA -> /Microcontroller/CODEC_BCLK
- TP6 pad 1: +6V -> /Microcontroller/CODEC_LRCLK
- TP7 pad 1: AGND_IN -> +1V8
- TP8 pad 1: Net-(C55-Pad2) -> +3V3
- TP9 pad 1: Net-(C56-Pad2) -> GND
- U3 pad 1: Net-(C27-Pad2) -> /Microcontroller/I2C_SDA
- U3 pad 10: /Microcontroller/CODEC_MCLK -> +3V3A
- U3 pad 11: /Microcontroller/CODEC_LRCK -> AGND
- U3 pad 12: /CODEC/BICK -> Net-(C11-Pad2)
- U3 pad 13: /Microcontroller/CODEC_SDIN -> Net-(C11-Pad2)
- U3 pad 14: /Microcontroller/CODEC_SDO -> Net-(C10-Pad2)
- U3 pad 15: (no net) -> Net-(C11-Pad2)
- U3 pad 17: /Microcontroller/SPI1_SOUT -> Net-(C11-Pad2)
- U3 pad 18: /Microcontroller/SPI1_SCK -> (no net)
- U3 pad 19: /Microcontroller/SPI1_CS_CODEC -> +3V3A
- U3 pad 2: VCOM_VRT -> /Microcontroller/I2C_SCL
- U3 pad 20: AGND_IN -> AGND
- U3 pad 21: /Microcontroller/CODEC_PDN -> (no net)
- U3 pad 22: AGND_IN -> (no net)
- U3 pad 23: AGND_IN -> AGND
- U3 pad 24: (no net) -> +3V3A
- U3 pad 25: +3V -> (no net)
- U3 pad 26: AGND_IN -> (no net)
- U3 pad 27: /CODEC/AOUTL- -> /Microcontroller/CODEC_~PD
- U3 pad 28: /CODEC/AOUTL+ -> (no net)
- U3 pad 29: /CODEC/AOUTR- -> +1V8
- U3 pad 3: /CODEC/AINR- -> GNDD
- U3 pad 30: /CODEC/AOUTR+ -> GNDD
- U3 pad 4: /CODEC/AINL+ -> GNDD
- U3 pad 5: /CODEC/AINL- -> GNDD
- U3 pad 6: +5VA -> Net-(C12-Pad1)
- U3 pad 7: AGND_IN -> (no net)
- U3 pad 8: +5VA -> Net-(C11-Pad2)
- U3 pad 9: AGND_IN -> Net-(C9-Pad2)
- U4 pad 1: Net-(TP4-Pad1) -> +5V
- U4 pad 2: (no net) -> AGND
- U4 pad 3: +3V -> /Microcontroller/ANALOG_EN
- U4 pad 4: AGND_IN -> (no net)
- U4 pad 5: /Microcontroller/USB_D+ -> +3V3A
- U5 pad 1: AGND_IN -> +5V
- U5 pad 2: +6V -> GND
- U5 pad 3: Net-(C40-Pad1) -> +5V
- U5 pad 4: Net-(R27-Pad2) -> (no net)
- U5 pad 5: (no net) -> +1V8
- U6 pad 1: Net-(C45-Pad2) -> +5V
- U6 pad 2: AGND_IN -> GND
- U6 pad 3: +6V -> +5V
- U6 pad 4: +6V -> (no net)
- U6 pad 5: (no net) -> +3V3
- X1 pad 1: Net-(C36-Pad1) -> +1V8
- X1 pad 2: Net-(C35-Pad1) -> GNDD
- X2 pad 1: Net-(U4-Pad41) -> (no net)
- X2 pad 2: AGND_IN -> GNDD
- X2 pad 3: /Microcontroller/CODEC_MCLK -> /Microcontroller/MCLK
- X2 pad 4: +3V -> +1V8
Routing:
- net AGND_IN: track 199.8 -> 0.00 mm, vias 64 -> 0
- net +3V: track 110.7 -> 0.00 mm, vias 11 -> 0
- net +5VA: track 94.8 -> 0.00 mm, vias 15 -> 0
- net /Microcontroller/I2C_SCL: track 44.5 -> 0.00 mm, vias 2 -> 0
- net /Microcontroller/I2C_SDA: track 43.6 -> 0.00 mm
- net /Microcontroller/HP_~SD: track 42.0 -> 0.00 mm, vias 2 -> 0
- net VCOM_VRT: track 37.8 -> 0.00 mm
- net /Microcontroller/SPI1_SCK: track 33.3 -> 0.00 mm, vias 3 -> 0
- net /Microcontroller/CODEC_MCLK: track 32.8 -> 0.00 mm, vias 3 -> 0
- net /Microcontroller/SPI1_SOUT: track 29.2 -> 0.00 mm, vias 3 -> 0
- net /Microcontroller/SPI1_CS_CODEC: track 27.7 -> 0.00 mm, vias 2 -> 0
- net Net-(C11-Pad2): track 24.7 -> 0.00 mm, vias 2 -> 0
- net /Microcontroller/CODEC_LRCK: track 24.7 -> 0.00 mm, vias 2 -> 0
- net /Microcontroller/USB_D6: track 0.00 -> 24.6 mm
- net /Microcontroller/CODEC_SDIN: track 24.4 -> 0.00 mm, vias 2 -> 0
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- removed copper zone on B.Cu, net (none)
- removed copper zone on Inner1.Cu, net +5VA
- removed copper zone on B.Cu, net AGND_IN
- removed copper zone on F.Cu, net AGND_IN
- removed copper zone on Inner2.Cu, net AGND_IN
- removed copper zone on Inner1.Cu, net USB_5V
Other:
- board outline removed
- board text removed: "+"
- board text removed: "+ -"
- board text removed: "-"
- board text removed: "3"
- board text removed: "5V"
- board text removed: "6V"
- board text removed: "AGND"
- board text removed: "AudioPulse rev3b 2016"
- board text removed: "BRN"
- board text removed: "C"
- board text removed: "EXT"
- board text removed: "G"
- board text removed: "GND"
- board text removed: "I"
- board text removed: "ID"
- board text removed: "L"
- board text removed: "L+"
- board text removed: "L-"
- board text removed: "MIC"
- board text removed: "O"
- board text removed: "PGA"
- board text removed: "R"
- board text removed: "T R"
- board text removed: "VCOM"

Commit message: Schematic roughly complete
Parts:
- removed C71: 100n, Capacitors_SMD:C_0402
- removed C75: 2.2u, Capacitors_SMD:C_0603
- removed C76: 0.1u, Capacitors_SMD:C_0402
- removed R21, R22: 10k, Resistors_SMD:R_0402
- removed R23, R24: 7.5, Resistors_SMD:R_0402
- added C34: 2.2u, Capacitors_SMD:C_0603, F.Cu at (156.8, 68.6)
- added C35: 2.2u, Capacitors_SMD:C_0603, F.Cu at (170.5, 60.2)
- added C36: 10u, Capacitors_SMD:C_0805, F.Cu at (157.1, 67.1)
- added C37: 2.2u, Capacitors_SMD:C_0603, F.Cu at (163.9, 67.5)
- added C38: 2.2u, Capacitors_SMD:C_0603, F.Cu at (166.7, 65.6)
- added C39: 10u, Capacitors_SMD:C_0805, F.Cu at (160.7, 67.7)
- added C40: 2.2u, Capacitors_SMD:C_0603, F.Cu at (170.5, 61.5)
- added J1: USB_B_Micro, Connectors:USB_Micro-B_10103594-0001LF, F.Cu at (123.1, 86.6)
- added J4: Screw_Terminal_01x02, TerminalBlocks_Phoenix:TerminalBlock_Phoenix_MPT-2.54mm_2pol, F.Cu at (157.1, 62.8)
- added R10: 100k, Resistors_SMD:R_0402, F.Cu at (151.0, 66.6)
- added R11: 100k, Resistors_SMD:R_0402, F.Cu at (168.6, 68.1)
- added R12: 0R, Resistors_SMD:R_0402, F.Cu at (163.3, 68.7)
- added R3: 100k, Resistors_SMD:R_0402, F.Cu at (141.4, 75.2)
- C10, C9: value 22u -> 2.2u; footprint Capacitors_SMD:C_1210 -> Capacitors_SMD:C_0603
- C11: value 100n -> 1u
- C12: value 1u -> 0.1u
- C13, C22, C28: value 10u -> 100n; footprint Capacitors_SMD:C_0805 -> Capacitors_SMD:C_0402
- C14, C32: value 1u -> 2.2u; footprint Capacitors_SMD:C_0402 -> Capacitors_SMD:C_0603
- C15, C16: value 0.1u -> 22u; footprint Capacitors_SMD:C_0402 -> Capacitors_SMD:C_1210
- C17: value 0.1u -> 100n
- C18, C20: value 0.1u -> 1u
- C19, C33: value 0.1u -> 10u; footprint Capacitors_SMD:C_0402 -> Capacitors_SMD:C_0805
- C21, C24, C27, C29, C3, C30: value 2.2u -> 0.1u; footprint Capacitors_SMD:C_0603 -> Capacitors_SMD:C_0402
- C23: value 2.2u -> 4.7u; footprint Capacitors_SMD:C_0603 -> Capacitors_SMD:C_0805
- C25: value 10u -> 0.1u; footprint Capacitors_SMD:C_0805 -> Capacitors_SMD:C_0402
- C26, C31: value 2.2u -> 100n; footprint Capacitors_SMD:C_0603 -> Capacitors_SMD:C_0402
- C7: value 100n -> 2.2u; footprint Capacitors_SMD:C_0402 -> Capacitors_SMD:C_0603
- J2: value Screw_Terminal_01x02 -> Conn_01x08; footprint TerminalBlocks_Phoenix:TerminalBlock_Phoenix_MPT-2.54mm_2pol -> Pin_Headers:Pin_Header_Straight_1x08_Pitch1.27mm
- J3: value USB_B_Micro -> Amphenol 20021122; footprint Connectors:USB_Micro-B_10103594-0001LF -> Pin_Headers:Pin_Header_Straight_2x05_Pitch1.27mm
- R1: value 100k -> 7.5
- R2: value 820 -> 7.5
- R4: value 12k (1%) -> 10k
- R5: value 2k -> 10k
- R6: value 2k -> 820
- R7: value 100k -> 12k (1%)
- R8: value 100k -> 2k
- R9: value 0R -> 2k
- U1: value STM32H743VITx -> USBLC6-2SC6; footprint Housings_QFP:LQFP-100_14x14mm_Pitch0.5mm -> TO_SOT_Packages_SMD:SOT-23-6
- U2: value USB3300-EZK -> STM32H743VITx; footprint Housings_DFN_QFN:QFN-32-1EP_5x5mm_Pitch0.5mm -> Housings_QFP:LQFP-100_14x14mm_Pitch0.5mm
- U3: value ADAU1772 -> USB3300-EZK; footprint Housings_DFN_QFN:QFN-40-1EP_6x6mm_Pitch0.5mm -> Housings_DFN_QFN:QFN-32-1EP_5x5mm_Pitch0.5mm
- U4: value LP5907MFX-3.3 -> ADAU1772; footprint TO_SOT_Packages_SMD:SOT-23-5 -> Housings_DFN_QFN:QFN-40-1EP_6x6mm_Pitch0.5mm
- U5: value LP5907MFX-1.8 -> LP5907MFX-3.3
- U6: value LP5907MFX-3.3 -> LP5907MFX-1.8
- U7: value USBLC6-2SC6 -> LP5907MFX-3.3; footprint TO_SOT_Packages_SMD:SOT-23-6 -> TO_SOT_Packages_SMD:SOT-23-5
- moved U7 78.2 mm to (167.2, 61.3)
- moved C2 64.0 mm to (124.1, 91.7)
- moved C19 62.5 mm to (117.5, 78.3)
- moved C14 62.1 mm to (124.2, 79.4)
- moved C23 61.9 mm to (121.0, 78.3)
- moved J2 60.5 mm to (117.3, 84.3)
- moved C9 60.1 mm to (127.1, 79.4)
- moved C3 57.8 mm to (131.7, 85.0)
- moved C31 56.5 mm to (132.4, 79.2)
- moved D1 56.4 mm to (124.3, 78.0)
- moved C7 56.2 mm to (129.9, 79.4)
- moved J3 55.3 mm to (135.2, 60.7), turned to 0 degrees
- moved R1 55.3 mm to (132.4, 77.9)
- moved R7 51.1 mm to (139.3, 78.1)
- moved R5 49.1 mm to (143.5, 73.8)
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Connections:
- C1 pad 1: GNDD -> Net-(C1-Pad1)
- C1 pad 2: +1V8 -> GNDD
- C10 pad 1: /Microcontroller/MIC1_IN -> GNDD
- C10 pad 2: Net-(C10-Pad2) -> +1V8
- C11 pad 1: AGND -> GNDD
- C11 pad 2: Net-(C11-Pad2) -> +1V8
- C12 pad 1: Net-(C12-Pad1) -> GNDD
- C12 pad 2: GNDD -> +1V8
- C13 pad 1: +1V8 -> GNDD
- C13 pad 2: GNDD -> +1V8
- C14 pad 1: +1V8 -> Net-(C14-Pad1)
- C14 pad 2: GNDD -> AGND
- C15 pad 1: +1V8 -> /MIC0
- C15 pad 2: GNDD -> Net-(C15-Pad2)
- C16 pad 1: AGND -> /MIC1
- C16 pad 2: +3V3A -> Net-(C16-Pad2)
- C17 pad 2: +3V3A -> Net-(C14-Pad1)
- C18 pad 1: AGND -> Net-(C18-Pad1)
- C18 pad 2: +3V3A -> GNDD
- C19 pad 1: AGND -> +1V8
- C19 pad 2: +3V3A -> GNDD
- C2 pad 1: GNDD -> /Microcontroller/USB_VBUS
- C2 pad 2: +1V8 -> GNDD
- C20 pad 1: AGND -> +1V8
- C20 pad 2: +3V3A -> GNDD
- C21 pad 1: GND -> +1V8
- C21 pad 2: +5V -> GNDD
- C22 pad 1: AGND -> GNDD
- C22 pad 2: +3V3A -> Net-(C22-Pad2)
- C23 pad 1: AGND -> GNDD
- C23 pad 2: +3V3A -> Net-(C22-Pad2)
- C24 pad 1: GND -> AGND
- C24 pad 2: +5V -> +3V3A
- C25 pad 1: GND -> AGND
- C25 pad 2: +1V8 -> +3V3A
- C26 pad 1: GND -> GNDD
- C26 pad 2: +1V8 -> Net-(C26-Pad2)
- C27 pad 1: GND -> AGND
- C27 pad 2: +5V -> +3V3A
- C28 pad 1: GND -> GNDD
- C28 pad 2: +3V3 -> Net-(C26-Pad2)
- C29 pad 1: GND -> AGND
- C29 pad 2: +3V3 -> +3V3A
- C3 pad 1: GNDD -> USB_5V
- C3 pad 2: +1V8 -> GNDD
- C30 pad 1: Net-(C30-Pad1) -> AGND
- C30 pad 2: GNDD -> +3V3A
- C31 pad 2: +1V8 -> /Microcontroller/MCLK
- C32 pad 1: GNDD -> GND
- C32 pad 2: +1V8 -> +5V
- C33 pad 1: GNDD -> AGND
- C33 pad 2: +1V8 -> +3V3A
- C4 pad 2: Net-(C4-Pad2) -> +1V8
- C6 pad 2: Net-(C6-Pad2) -> +1V8
- C7 pad 2: +1V8 -> Net-(C7-Pad2)
- C8 pad 1: Net-(C11-Pad2) -> GNDD
- C8 pad 2: AGND -> +1V8
- C9 pad 1: /Microcontroller/MIC0_IN -> GNDD
- J2 pad 1: +5V -> /MIC0
- J2 pad 2: GND -> GNDD
- J3 pad 1: /Microcontroller/USB_VBUS -> +1V8
- J3 pad 2: /Microcontroller/USB_D- -> /Microcontroller/SWDIO
- J3 pad 3: /Microcontroller/USB_D+ -> GNDD
- J3 pad 4: /Microcontroller/USB_ID -> /Microcontroller/SWCLK
- J3 pad 5: Net-(FB1-Pad1) -> GNDD
- J3 pad 6: Net-(C30-Pad1) -> /Microcontroller/SWO
- R1 pad 1: Net-(R1-Pad1) -> Net-(D1-Pad2)
- R1 pad 2: GNDD -> Net-(R1-Pad2)
- R2 pad 1: Net-(R2-Pad1) -> Net-(D2-Pad2)
- R2 pad 2: /Microcontroller/USB_VBUS -> Net-(R2-Pad2)
- R4 pad 1: GNDD -> /Microcontroller/I2C_SDA
- R4 pad 2: Net-(R4-Pad2) -> +3V
- R5 pad 1: /Microcontroller/MIC1_IN -> /Microcontroller/I2C_SCL
- R5 pad 2: Net-(C12-Pad1) -> +3V
- R6 pad 1: /Microcontroller/MIC0_IN -> Net-(R6-Pad1)
- R6 pad 2: Net-(C12-Pad1) -> /Microcontroller/USB_VBUS
- R7 pad 2: /Microcontroller/CODEC_~PD -> Net-(R7-Pad2)
- R8 pad 1: GND -> /MIC1
- R8 pad 2: /Microcontroller/ANALOG_EN -> Net-(C18-Pad1)
- R9 pad 1: USB_5V -> /MIC0
- R9 pad 2: +5V -> Net-(C18-Pad1)
- U1 pad 1: (no net) -> /Microcontroller/USB_D-
- U1 pad 2: /Microcontroller/CODEC_SDI -> Net-(FB1-Pad1)
- U1 pad 3: /Microcontroller/CODEC_LRCLK -> /Microcontroller/USB_D+
- U1 pad 4: /Microcontroller/CODEC_BCLK -> /Microcontroller/USB_D+
- U1 pad 5: /Microcontroller/CODEC_SDO -> /Microcontroller/USB_VBUS
- U1 pad 6: +1V8 -> /Microcontroller/USB_D-
- U2 pad 1: GNDD -> (no net)
- U2 pad 10: (no net) -> GNDD
- U2 pad 11: /Microcontroller/USB_NXT -> +1V8
- U2 pad 12: /Microcontroller/USB_DIR -> (no net)
- U2 pad 13: /Microcontroller/USB_STP -> (no net)
- U2 pad 14: /Microcontroller/USB_CLKOUT -> /Microcontroller/~RESET
- U2 pad 15: +1V8 -> /Microcontroller/USB_STP
- U2 pad 16: +3V3 -> (no net)
- U2 pad 17: /Microcontroller/USB_D7 -> /Microcontroller/USB_DIR
- U2 pad 18: /Microcontroller/USB_D6 -> /Microcontroller/USB_NXT
- U2 pad 19: /Microcontroller/USB_D5 -> GNDD
- U2 pad 2: GNDD -> /Microcontroller/CODEC_SDI
- U2 pad 20: /Microcontroller/USB_D4 -> +1V8
- U2 pad 21: /Microcontroller/USB_D3 -> +1V8
- U2 pad 22: /Microcontroller/USB_D2 -> (no net)
- U2 pad 23: /Microcontroller/USB_D1 -> (no net)
- U2 pad 24: /Microcontroller/USB_D0 -> (no net)
- U2 pad 25: +3V3 -> /Microcontroller/USB_D0
- U2 pad 26: +1V8 -> GNDD
- U2 pad 27: (no net) -> +1V8
- U2 pad 28: Net-(U2-Pad28) -> (no net)
- U2 pad 29: +1V8 -> /Microcontroller/USB_CLKOUT
- U2 pad 3: (no net) -> /Microcontroller/CODEC_LRCLK
- U2 pad 30: +3V3 -> (no net)
- U2 pad 31: GNDD -> (no net)
- U2 pad 32: Net-(R4-Pad2) -> (no net)
- U2 pad 33: GNDD -> (no net)
- U2 pad 4: Net-(R2-Pad1) -> /Microcontroller/CODEC_BCLK
- U2 pad 5: /Microcontroller/USB_ID -> /Microcontroller/CODEC_SDO
- U2 pad 6: +3V3 -> +1V8
- U2 pad 7: /Microcontroller/USB_D- -> (no net)
- U2 pad 8: /Microcontroller/USB_D+ -> (no net)
- U3 pad 1: /Microcontroller/I2C_SDA -> GNDD
- U3 pad 10: +3V3A -> (no net)
- U3 pad 11: AGND -> /Microcontroller/USB_NXT
- U3 pad 12: Net-(C11-Pad2) -> /Microcontroller/USB_DIR
- U3 pad 13: Net-(C11-Pad2) -> /Microcontroller/USB_STP
- U3 pad 14: Net-(C10-Pad2) -> /Microcontroller/USB_CLKOUT
- U3 pad 15: Net-(C11-Pad2) -> Net-(C26-Pad2)
- U3 pad 16: (no net) -> +3V3
- U3 pad 17: Net-(C11-Pad2) -> /Microcontroller/USB_D7
- U3 pad 18: (no net) -> /Microcontroller/USB_D6
- U3 pad 19: +3V3A -> /Microcontroller/USB_D5
- U3 pad 2: /Microcontroller/I2C_SCL -> GNDD
- U3 pad 20: AGND -> /Microcontroller/USB_D4
- U3 pad 21: (no net) -> /Microcontroller/USB_D3
- U3 pad 22: (no net) -> /Microcontroller/USB_D2
- U3 pad 23: AGND -> /Microcontroller/USB_D1
- U3 pad 24: +3V3A -> /Microcontroller/USB_D0
- U3 pad 25: (no net) -> +3V3
- U3 pad 26: (no net) -> Net-(C26-Pad2)
- U3 pad 27: /Microcontroller/CODEC_~PD -> (no net)
- U3 pad 28: (no net) -> Net-(U3-Pad28)
- U3 pad 29: +1V8 -> Net-(C22-Pad2)
- U3 pad 3: GNDD -> (no net)
- U3 pad 30: GNDD -> +3V3
- U3 pad 31: /Microcontroller/CODEC_LRCLK -> +3V3
- U3 pad 32: /Microcontroller/CODEC_BCLK -> Net-(R7-Pad2)
- U3 pad 33: /Microcontroller/CODEC_SDO -> GNDD
- U3 pad 4: GNDD -> Net-(R6-Pad1)
- U3 pad 5: GNDD -> /Microcontroller/USB_ID
- U3 pad 6: Net-(C12-Pad1) -> +3V3
- U3 pad 7: (no net) -> /Microcontroller/USB_D-
- U3 pad 8: Net-(C11-Pad2) -> /Microcontroller/USB_D+
- U3 pad 9: Net-(C9-Pad2) -> (no net)
- U4 pad 1: +5V -> /Microcontroller/I2C_SDA
- U4 pad 2: AGND -> /Microcontroller/I2C_SCL
- U4 pad 3: /Microcontroller/ANALOG_EN -> GNDD
- U4 pad 4: (no net) -> GNDD
- U4 pad 5: +3V3A -> GNDD
- U5 pad 2: GND -> AGND
- U5 pad 3: +5V -> /Microcontroller/ANALOG_EN
- U5 pad 5: +1V8 -> +3V3A
- U6 pad 5: +3V3 -> +1V8
- U7 pad 1: /Microcontroller/USB_D- -> +5V
- U7 pad 2: Net-(FB1-Pad1) -> GND
- U7 pad 3: /Microcontroller/USB_D+ -> +5V
- U7 pad 4: /Microcontroller/USB_D+ -> (no net)
- U7 pad 5: /Microcontroller/USB_VBUS -> +3V3
- X1 pad 3: Net-(U2-Pad28) -> Net-(U3-Pad28)
Routing:
- net /Microcontroller/USB_D6: track 24.6 -> 0.00 mm
- net /Microcontroller/USB_D5: track 22.3 -> 0.00 mm
- net /Microcontroller/USB_D4: track 17.7 -> 0.00 mm
- net /Microcontroller/USB_D3: track 17.0 -> 0.00 mm

Commit message: Placement!
Parts:
- U4: footprint Housings_DFN_QFN:QFN-40-1EP_6x6mm_Pitch0.5mm -> lib:QFN-40-1EP_6x6mm_Pitch0.5mm
- moved C32 77.8 mm to (96.0, 87.0)
- moved C35 76.9 mm to (96.0, 79.0)
- moved R11 75.1 mm to (96.5, 88.8)
- moved TP9 73.5 mm to (97.8, 93.7)
- moved C38 72.8 mm to (96.0, 83.1)
- moved J4 72.6 mm to (91.0, 93.0)
- moved C40 71.9 mm to (102.2, 83.8), turned to 90 degrees
- moved U7 71.5 mm to (99.4, 84.1)
- moved U5 67.9 mm to (99.4, 87.9)
- moved C33 67.2 mm to (104.2, 87.8), turned to 90 degrees
- moved U6 66.4 mm to (99.6, 80.0)
- moved R12 64.7 mm to (99.2, 77.2), turned to 270 degrees
- moved TP8 64.5 mm to (106.9, 82.4)
- moved TP7 63.5 mm to (110.2, 80.8)
- moved C37 62.5 mm to (102.6, 79.8), turned to 90 degrees
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Connections:
- C13 pad 2: +1V8 -> /Microcontroller/1V8_USB
- C26 pad 2: Net-(C26-Pad2) -> /Microcontroller/1V8_USB
- C28 pad 2: Net-(C26-Pad2) -> /Microcontroller/1V8_USB
- C31 pad 2: /Microcontroller/MCLK -> +1V8
- J1 pad 2: /Microcontroller/USB_D- -> Net-(J1-Pad2)
- J1 pad 3: /Microcontroller/USB_D+ -> Net-(J1-Pad3)
- J2 pad 5: /HP_LP -> /HP_LN
- J2 pad 6: /HP_LN -> /HP_LP
- J2 pad 7: /HP_RP -> /HP_RN
- J2 pad 8: /HP_RN -> /HP_RP
- U1 pad 1: /Microcontroller/USB_D- -> Net-(J1-Pad2)
- U1 pad 3: /Microcontroller/USB_D+ -> Net-(J1-Pad3)
- U1 pad 4: /Microcontroller/USB_D+ -> /Microcontroller/USB_D_P
- U1 pad 6: /Microcontroller/USB_D- -> /Microcontroller/USB_D_N
- U3 pad 15: Net-(C26-Pad2) -> /Microcontroller/1V8_USB
- U3 pad 26: Net-(C26-Pad2) -> /Microcontroller/1V8_USB
- U3 pad 7: /Microcontroller/USB_D- -> /Microcontroller/USB_D_N
- U3 pad 8: /Microcontroller/USB_D+ -> /Microcontroller/USB_D_P
- U4 pad 41: (no net) -> GNDD
- X1 pad 1: +1V8 -> /Microcontroller/1V8_USB
- X1 pad 4: +1V8 -> /Microcontroller/1V8_USB
Routing:
- net GNDD: track 0.00 -> 44.0 mm, vias 0 -> 22
- net /Microcontroller/I2C_SCL: track 0.00 -> 43.9 mm, vias 0 -> 2
- net /Microcontroller/I2C_SDA: track 0.00 -> 41.4 mm, vias 0 -> 2
- net /Microcontroller/USB_NXT: track 0.00 -> 36.9 mm, vias 0 -> 2
- net /Microcontroller/USB_D0: track 0.00 -> 36.8 mm, vias 0 -> 2
- net /Microcontroller/USB_CLKOUT: track 0.00 -> 36.7 mm, vias 0 -> 2
- net /Microcontroller/MCLK: track 0.00 -> 35.8 mm
- net /Microcontroller/USB_DIR: track 0.00 -> 35.5 mm, vias 0 -> 2
- net /Microcontroller/ANALOG_EN: track 0.00 -> 35.0 mm, vias 0 -> 2
- net /Microcontroller/USB_D2: track 0.00 -> 34.3 mm, vias 0 -> 2
- net /Microcontroller/USB_D1: track 0.00 -> 34.2 mm, vias 0 -> 2
- net +1V8: track 0.00 -> 34.0 mm, vias 0 -> 10
- net /Microcontroller/USB_STP: track 0.00 -> 33.7 mm, vias 0 -> 2
- net /Microcontroller/USB_D5: track 0.00 -> 33.1 mm, vias 0 -> 2
- net /Microcontroller/USB_D4: track 0.00 -> 32.9 mm, vias 0 -> 2
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- added copper zone on Inner1.Cu, net +1V8
- added copper zone on Inner1.Cu, net +3V3A
- added copper zone on Inner2.Cu, net AGND
- added copper zone on Inner2.Cu, net GND
- added copper zone on Inner2.Cu, net GNDD
Other:
- board outline added: 57.4 x 42.8 mm

Commit message: Much more routing
Parts:
- added G***: LOGO, ear:LOGO, F.Cu at (100.6, 99.3)
- C1, C10, C14, C2, C32, C34, C35, C37, C38, C4, C40, C5, C6, C7, C8, C9: footprint Capacitors_SMD:C_0603 -> Capacitor_SMD:C_0603_1608Metric_Pad1.05x0.95mm_HandSolder
- C11, C12, C13, C17, C18, C20, C21, C22, C24, C25, C26, C27, C28, C29, C30, C31: footprint Capacitors_SMD:C_0402 -> Capacitor_SMD:C_0402_1005Metric
- C15, C16: footprint Capacitors_SMD:C_1210 -> Capacitor_SMD:C_1210_3225Metric
- C19, C23, C33, C36, C39: footprint Capacitors_SMD:C_0805 -> Capacitor_SMD:C_0805_2012Metric_Pad1.15x1.40mm_HandSolder
- D1, D2: footprint LEDs:LED_0603 -> LED_SMD:LED_0603_1608Metric_Pad1.05x0.95mm_HandSolder
- FB1, FB2: footprint Inductors_SMD:L_0805 -> Inductor_SMD:L_0805_2012Metric_Pad1.15x1.40mm_HandSolder
- J1: footprint Connectors:USB_Micro-B_10103594-0001LF -> Connector_USB:USB_Micro-B_Molex-105017-0001
- J2: footprint Pin_Headers:Pin_Header_Straight_1x08_Pitch1.27mm -> Connector_PinHeader_1.27mm:PinHeader_1x08_P1.27mm_Vertical
- J3: footprint Pin_Headers:Pin_Header_Straight_2x05_Pitch1.27mm -> Connector_PinHeader_1.27mm:PinHeader_2x05_P1.27mm_Vertical
- J4: footprint TerminalBlocks_Phoenix:TerminalBlock_Phoenix_MPT-2.54mm_2pol -> Connector_PinHeader_2.54mm:PinHeader_1x02_P2.54mm_Vertical
- R1, R10, R11, R12, R2, R3, R4, R5, R6, R7, R8, R9: footprint Resistors_SMD:R_0402 -> Resistor_SMD:R_0402_1005Metric
- U1: footprint TO_SOT_Packages_SMD:SOT-23-6 -> Package_TO_SOT_SMD:SOT-23-6
- U2: footprint Housings_QFP:LQFP-100_14x14mm_Pitch0.5mm -> Package_QFP:LQFP-100_14x14mm_P0.5mm
- U3: footprint Housings_DFN_QFN:QFN-32-1EP_5x5mm_Pitch0.5mm -> Package_DFN_QFN:QFN-32-1EP_5x5mm_P0.5mm_EP3.1x3.1mm_ThermalVias
- U4: footprint lib:QFN-40-1EP_6x6mm_Pitch0.5mm -> Package_DFN_QFN:QFN-40-1EP_6x6mm_P0.5mm_EP4.6x4.6mm_ThermalVias
- U5, U6, U7: footprint TO_SOT_Packages_SMD:SOT-23-5 -> Package_TO_SOT_SMD:SOT-23-5
- X1: footprint Oscillators:Oscillator_SMD_SeikoEpson_SG210-4pin_2.5x2.0mm -> Oscillator:Oscillator_SMD_SeikoEpson_SG210-4Pin_2.5x2.0mm_HandSoldering
- X2: footprint Oscillators:Oscillator_SMD_EuroQuartz_XO32-4pin_3.2x2.5mm -> Oscillator:Oscillator_SMD_EuroQuartz_XO32-4Pin_3.2x2.5mm_HandSoldering
- moved TP1 18.8 mm to (100.3, 69.6)
- moved C31 1.14 mm to (135.9, 65.8)
- moved C12 0.67 mm to (143.0, 81.4)
- moved C13 0.60 mm to (108.6, 65.5)
- moved C3 0.53 mm to (98.5, 77.1)
- moved TP3 0.51 mm to (133.1, 90.7)
- moved C27 0.48 mm to (113.3, 98.7)
- moved TP4 0.44 mm to (126.0, 90.7)
- moved TP5 0.41 mm to (136.7, 90.7)
- moved C7 0.38 mm to (143.4, 71.7)
- moved C16 0.38 mm to (115.8, 102.8)
- moved C24 0.35 mm to (123.8, 98.1)
- moved C32 0.34 mm to (95.7, 87.0)
- moved R12 0.33 mm to (99.5, 77.1)
- moved R7 0.32 mm to (103.0, 70.1)
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Connections:
- J3 pad 7: (no net) -> Net-(J3-Pad7)
- J3 pad 8: (no net) -> Net-(J3-Pad8)
- U2 pad 1: (no net) -> Net-(U2-Pad1)
- U2 pad 12: (no net) -> Net-(U2-Pad12)
- U2 pad 13: (no net) -> Net-(U2-Pad13)
- U2 pad 16: (no net) -> Net-(U2-Pad16)
- U2 pad 22: (no net) -> Net-(U2-Pad22)
- U2 pad 23: (no net) -> Net-(U2-Pad23)
- U2 pad 24: (no net) -> Net-(U2-Pad24)
- U2 pad 28: (no net) -> Net-(U2-Pad28)
- U2 pad 30: (no net) -> Net-(U2-Pad30)
- U2 pad 31: (no net) -> Net-(U2-Pad31)
- U2 pad 32: (no net) -> Net-(U2-Pad32)
- U2 pad 33: (no net) -> Net-(U2-Pad33)
- U2 pad 36: (no net) -> Net-(U2-Pad36)
- U2 pad 37: (no net) -> Net-(U2-Pad37)
- U2 pad 38: (no net) -> Net-(U2-Pad38)
- U2 pad 39: (no net) -> Net-(U2-Pad39)
- U2 pad 40: (no net) -> Net-(U2-Pad40)
- U2 pad 41: (no net) -> Net-(U2-Pad41)
- U2 pad 42: (no net) -> Net-(U2-Pad42)
- U2 pad 43: (no net) -> Net-(U2-Pad43)
- U2 pad 44: (no net) -> Net-(U2-Pad44)
- U2 pad 45: (no net) -> Net-(U2-Pad45)
- U2 pad 53: (no net) -> Net-(U2-Pad53)
- U2 pad 54: (no net) -> Net-(U2-Pad54)
- U2 pad 55: (no net) -> Net-(U2-Pad55)
- U2 pad 56: (no net) -> Net-(U2-Pad56)
- U2 pad 57: (no net) -> Net-(U2-Pad57)
- U2 pad 58: (no net) -> Net-(U2-Pad58)
- U2 pad 61: (no net) -> Net-(U2-Pad61)
- U2 pad 62: (no net) -> Net-(U2-Pad62)
- U2 pad 63: (no net) -> Net-(U2-Pad63)
- U2 pad 64: (no net) -> Net-(U2-Pad64)
- U2 pad 65: (no net) -> Net-(U2-Pad65)
- U2 pad 67: (no net) -> Net-(U2-Pad67)
- U2 pad 68: (no net) -> Net-(U2-Pad68)
- U2 pad 69: (no net) -> Net-(U2-Pad69)
- U2 pad 7: (no net) -> /Microcontroller/CODEC_~PD
- U2 pad 70: (no net) -> Net-(U2-Pad70)
- U2 pad 71: (no net) -> Net-(U2-Pad71)
- U2 pad 77: (no net) -> Net-(U2-Pad77)
- U2 pad 78: (no net) -> Net-(U2-Pad78)
- U2 pad 79: (no net) -> Net-(U2-Pad79)
- U2 pad 8: (no net) -> Net-(U2-Pad8)
- U2 pad 80: (no net) -> Net-(U2-Pad80)
- U2 pad 81: (no net) -> Net-(U2-Pad81)
- U2 pad 82: (no net) -> Net-(U2-Pad82)
- U2 pad 83: (no net) -> Net-(U2-Pad83)
- U2 pad 84: (no net) -> Net-(U2-Pad84)
- U2 pad 85: (no net) -> Net-(U2-Pad85)
- U2 pad 86: (no net) -> Net-(U2-Pad86)
- U2 pad 87: (no net) -> Net-(U2-Pad87)
- U2 pad 88: (no net) -> Net-(U2-Pad88)
- U2 pad 9: (no net) -> Net-(U2-Pad9)
- U2 pad 90: (no net) -> Net-(U2-Pad90)
- U2 pad 92: (no net) -> /Microcontroller/USB_RESET
- U2 pad 95: (no net) -> Net-(U2-Pad95)
- U2 pad 96: (no net) -> Net-(U2-Pad96)
- U3 pad 10: (no net) -> Net-(U3-Pad10)
- U3 pad 27: (no net) -> Net-(U3-Pad27)
- U3 pad 3: (no net) -> Net-(U3-Pad3)
- U3 pad 9: (no net) -> /Microcontroller/USB_RESET
- U4 pad 16: (no net) -> Net-(U4-Pad16)
- U4 pad 18: (no net) -> Net-(U4-Pad18)
- U4 pad 28: (no net) -> Net-(U4-Pad28)
- U4 pad 35: (no net) -> Net-(U4-Pad35)
- U4 pad 36: (no net) -> Net-(U4-Pad36)
- U4 pad 37: (no net) -> Net-(U4-Pad37)
- U4 pad 38: (no net) -> Net-(U4-Pad38)
- U4 pad 7: (no net) -> Net-(U4-Pad7)
- U5 pad 4: (no net) -> Net-(U5-Pad4)
- U6 pad 4: (no net) -> Net-(U6-Pad4)
- U7 pad 4: (no net) -> Net-(U7-Pad4)
- X2 pad 1: (no net) -> /Microcontroller/MCLK_EN
Routing:
- net +1V8: track 34.0 -> 144.1 mm, vias 10 -> 19
- net /Microcontroller/~RESET: track 0.00 -> 39.0 mm, vias 0 -> 2
- net GNDD: track 44.0 -> 72.1 mm, vias 22 -> 27
- net /Microcontroller/USB_RESET: track 0.00 -> 21.8 mm, vias 0 -> 2
- net /Microcontroller/CODEC_BCLK: track 12.2 -> 29.9 mm, vias 2 -> 3
- net /Microcontroller/CODEC_~PD: track 1.39 -> 16.1 mm, vias 0 -> 2
- net /Microcontroller/CODEC_SDI: track 11.7 -> 22.7 mm, vias 0 -> 1
- net /Microcontroller/CODEC_LRCLK: track 10.9 -> 20.2 mm, vias 0 -> 1
- net GND: track 17.3 -> 23.4 mm, vias 7 -> 9
- net AGND: track 12.9 -> 18.7 mm, vias 7 -> 9
- net /Microcontroller/CODEC_SDO: track 12.9 -> 17.2 mm, vias 2 -> 3
- net /Microcontroller/USB_ID: track 17.2 -> 20.3 mm
- net +3V3: track 20.8 -> 23.7 mm
- net /Microcontroller/1V8_USB: track 9.59 -> 10.9 mm
- net Net-(C18-Pad1): track 11.3 -> 12.4 mm
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